Commit message: add xarm6 with gripper

File: xarm_description/urdf/xarm6_robot.urdf.xacro (robot description, xacro)
@@ -8,5 +8,5 @@
   <!-- common stuff -->
   <xacro:include filename="$(find xarm_description)/urdf/common.gazebo.xacro" />
-  <!-- xarm6 -->
+  <!-- include xarm6 relative macros: -->
   <xacro:include filename="$(find xarm_description)/urdf/xarm6.urdf.xacro" />
   <xacro:include filename="$(find xarm_description)/urdf/xarm6.transmission.xacro" />

File: xarm_gripper/urdf/xarm_gripper.urdf.xacro (robot description, xacro)
@@ -1,14 +1,15 @@
 <?xml version="1.0"?>
-<robot xmlns:xacro="http://ros.org/wiki/xacro">
+<robot xmlns:xacro="http://ros.org/wiki/xacro" name="xarm_gripper">
 <!--
   Author: Jason Peng <jason@ufactory.cc>
 -->
-  <xacro:macro name="xarm_gripper_urdf" params="prefix">
-    <material name="White">
-      <color rgba="1.0 1.0 1.0 1.0"/>
-    </material>
-    <material name="Silver">
-      <color rgba="0.753 0.753 0.753 1.0"/>
-    </material>
+  <xacro:macro name="xarm_gripper_urdf" params="prefix:='' attach_to:='' rpy:='0 0 0' xyz:='0 0 0' ">
+  <xacro:unless value="${attach_to == ''}">
+    <joint name="${prefix}gripper_fix" type="fixed">
+      <parent link="${attach_to}"/>
+      <child link="${prefix}xarm_gripper_base_link"/>
+      <origin xyz="${xyz}" rpy="${rpy}"/>
+    </joint>
+  </xacro:unless>
   <link
     name="${prefix}xarm_gripper_base_link">
@@ -40,5 +41,7 @@
           rgba="0.89804 0.91765 0.92941 1" />
       </material> -->
-      <material name="White" />
+      <material name="White">
+        <color rgba="1.0 1.0 1.0 1.0"/>
+      </material>
     </visual>
     <collision>
@@ -76,5 +79,7 @@
           filename="package://xarm_gripper/meshes/left_outer_knuckle.STL" />
       </geometry>
-      <material name="Silver" />
+      <material name="Silver">
+        <color rgba="0.753 0.753 0.753 1.0"/>
+      </material>
     </visual>
     <collision>
@@ -130,5 +135,7 @@
           filename="package://xarm_gripper/meshes/left_finger.STL" />
       </geometry>
-      <material name="Silver" />
+      <material name="Silver">
+        <color rgba="0.753 0.753 0.753 1.0"/>
+      </material>
     </visual>
     <collision>
@@ -185,5 +192,7 @@
           filename="package://xarm_gripper/meshes/left_inner_knuckle.STL" />
       </geometry>
-      <material name="Silver" />
+      <material name="Silver">
+        <color rgba="0.753 0.753 0.753 1.0"/>
+      </material>
     </visual>
     <collision>
@@ -240,5 +249,7 @@
           filename="package://xarm_gripper/meshes/right_outer_knuckle.STL" />
       </geometry>
-      <material name="Silver" />
+      <material name="Silver">
+        <color rgba="0.753 0.753 0.753 1.0"/>
+      </material>
     </visual>
     <collision>
@@ -295,5 +306,7 @@
           filename="package://xarm_gripper/meshes/right_finger.STL" />
       </geometry>
-      <material name="Silver" />
+      <material name="Silver">
+        <color rgba="0.753 0.753 0.753 1.0"/>
+      </material>
     </visual>
     <collision>
@@ -350,5 +363,7 @@
           filename="package://xarm_gripper/meshes/right_inner_knuckle.STL" />
       </geometry>
-      <material name="Silver" />
+      <material name="Silver">
+        <color rgba="0.753 0.753 0.753 1.0"/>
+      </material>
     </visual>
     <collision>

File: xarm_gripper/urdf/xarm_gripper_model.xacro (robot description, xacro)
@@ -2,7 +2,4 @@
 <robot xmlns:xacro="http://ros.org/wiki/xacro"
        name="xarm_gripper" >
-  <xacro:arg name="prefix" default=""/>
-  <xacro:arg name="ros_control_namespace" default="xarm"/>
-  <xacro:arg name="effort_control" default="false"/>
   <!-- common stuff -->
   <xacro:include filename="$(find xarm_description)/urdf/common.gazebo.xacro" />
@@ -11,13 +8,15 @@
   <xacro:include filename="$(find xarm_gripper)/urdf/xarm_gripper.transmission.xacro" />
   <xacro:include filename="$(find xarm_gripper)/urdf/xarm_gripper.gazebo.xacro" />
-  <!-- gazebo plugin -->
-  <xacro:gazebo_ros_control_plugin namespace="$(arg ros_control_namespace)"/>
-  <xacro:xarm_gripper_urdf prefix="$(arg prefix)"/>
-  <xacro:if value="$(arg effort_control)">
-    <xacro:xarm_gripper_transmission prefix="$(arg prefix)" hard_interface="EffortJointInterface" />
-  </xacro:if>
-  <xacro:unless value="$(arg effort_control)">
-    <xacro:xarm_gripper_transmission prefix="$(arg prefix)" hard_interface="PositionJointInterface" />
-  </xacro:unless>
-  <xacro:xarm_gripper_gazebo prefix="$(arg prefix)" />
+  <xacro:macro name="load_gripper" params="prefix:='' attach_to:='' ns:='xarm_gripper' xyz:='0 0 0' rpy:='0 0 0' effort_control:='false' ">
+    <!-- gazebo plugin -->
+    <xacro:gazebo_ros_control_plugin namespace="${ns}"/>
+    <xacro:xarm_gripper_urdf prefix="${prefix}" attach_to="${attach_to}" xyz="${xyz}" rpy="${rpy}" />
+    <xacro:if value="${effort_control}">
+      <xacro:xarm_gripper_transmission prefix="${prefix}" hard_interface="EffortJointInterface" />
+    </xacro:if>
+    <xacro:unless value="${effort_control}">
+      <xacro:xarm_gripper_transmission prefix="${prefix}" hard_interface="PositionJointInterface" />
+    </xacro:unless>
+    <xacro:xarm_gripper_gazebo prefix="${prefix}" />
+  </xacro:macro>
 </robot>

Commit message: support new xarm_api

File: xarm_description/urdf/xarm6_robot.urdf.xacro (robot description, xacro)
@@ -1,41 +1,10 @@
-<?xml version="1.0"?>
-<robot xmlns:xacro="http://ros.org/wiki/xacro"
-       name="xarm6" >
+<?xml version='1.0' encoding='utf-8'?>
+<robot xmlns:xacro="http://ros.org/wiki/xacro" name="xarm6">
   <xacro:arg name="prefix" default=""/>
-  <xacro:arg name="ros_control_namespace" default="xarm"/>
+  <xacro:arg name="ros_namespace" default="xarm"/>
   <xacro:arg name="limited" default="false"/>
   <xacro:arg name="effort_control" default="false"/>
-  <!-- common stuff -->
-  <xacro:include filename="$(find xarm_description)/urdf/common.gazebo.xacro" />
-  <!-- include xarm6 relative macros: -->
-  <xacro:include filename="$(find xarm_description)/urdf/xarm6.urdf.xacro" />
-  <xacro:include filename="$(find xarm_description)/urdf/xarm6.transmission.xacro" />
-  <xacro:include filename="$(find xarm_description)/urdf/xarm6.gazebo.xacro" />
-  <!-- gazebo_plugin -->
-  <xacro:gazebo_ros_control_plugin namespace="$(arg ros_control_namespace)"/>
-  <xacro:if value="$(arg limited)">
-    <xacro:xarm6_urdf prefix="$(arg prefix)"
-      joint1_lower_limit="${-pi*0.99}" joint1_upper_limit="${pi*0.99}"
-      joint2_lower_limit="${-2.18}" joint2_upper_limit="${2.18}"
-      joint3_lower_limit="${-pi*0.99}" joint3_upper_limit="${0.11}"
-      joint4_lower_limit="${-pi*0.99}" joint4_upper_limit="${pi*0.99}"
-      joint5_lower_limit="${-1.75}" joint5_upper_limit="${pi*0.99}"
-      joint6_lower_limit="${-pi*0.99}" joint6_upper_limit="${pi*0.99}"/>
-  </xacro:if>
-  <xacro:unless value="$(arg limited)">
-    <xacro:xarm6_urdf prefix="$(arg prefix)"/>
-  </xacro:unless>
-  <xacro:if value="$(arg effort_control)">
-    <xacro:xarm6_transmission prefix="$(arg prefix)" hard_interface="EffortJointInterface" />
-  </xacro:if>
-  <xacro:unless value="$(arg effort_control)">
-    <xacro:xarm6_transmission prefix="$(arg prefix)" hard_interface="PositionJointInterface" />
-  </xacro:unless>
-  <xacro:xarm6_gazebo prefix="$(arg prefix)" />
-  <link name="world" />
-  <joint name="world_joint" type="fixed">
-    <parent link="world" />
-    <child link = "$(arg prefix)link_base" />
-    <origin xyz="0.0 0.0 0.0" rpy="0.0 0.0 0.0" />
-  </joint>
+  <!-- load xarm6 robot -->
+  <xacro:include filename="$(find xarm_description)/urdf/xarm6_robot_macro.xacro" />
+  <xacro:xarm6_robot prefix="$(arg prefix)" namespace="$(arg ros_namespace)" limited="$(arg limited)" effort_control="$(arg effort_control)"/>
 </robot>

File: xarm_description/urdf/xarm6_with_gripper.xacro (robot description, xacro)
@@ -1,10 +1,14 @@
 <?xml version='1.0' encoding='utf-8'?>
-<robot xmlns:xacro="http://ros.org/wiki/xacro" name="xarm6_gripper">
+<robot xmlns:xacro="http://ros.org/wiki/xacro" name="xarm6_with_gripper">
+  <xacro:arg name="prefix" default=""/>
+  <xacro:arg name="ros_namespace" default="xarm"/>
+  <xacro:arg name="limited" default="false"/>
+  <xacro:arg name="effort_control" default="false"/>
   <!-- load xarm6 robot -->
-  <xacro:include filename="$(find xarm_description)/urdf/xarm6_robot.urdf.xacro" />
+  <xacro:include filename="$(find xarm_description)/urdf/xarm6_robot_macro.xacro" />
   <!-- Attach gripper -->
   <xacro:include filename="$(find xarm_gripper)/urdf/xarm_gripper_model.xacro" />
   <!-- <xacro:load_gripper attach_to="$(arg prefix)link6" /> -->
-  <!-- TODO: Re-construct xarm6_robot.urdf.xacro to only define macro, thus here can support passing argument like "prefix" -->
-  <xacro:load_gripper attach_to="link6" />
+  <xacro:xarm6_robot prefix="$(arg prefix)" namespace="$(arg ros_namespace)" limited="$(arg limited)" effort_control="$(arg effort_control)"/>
+  <xacro:load_gripper attach_to="$(arg prefix)link6" />
 </robot>

Commit message: new xarm7 and xarm5 models

File: xarm_description/urdf/xarm6_robot.urdf.xacro (robot description, xacro)
@@ -1,41 +1,10 @@
-<?xml version="1.0"?>
-<robot xmlns:xacro="http://ros.org/wiki/xacro"
-       name="xarm6" >
+<?xml version='1.0' encoding='utf-8'?>
+<robot xmlns:xacro="http://ros.org/wiki/xacro" name="xarm6">
   <xacro:arg name="prefix" default=""/>
-  <xacro:arg name="ros_control_namespace" default="xarm"/>
+  <xacro:arg name="ros_namespace" default="xarm"/>
   <xacro:arg name="limited" default="false"/>
   <xacro:arg name="effort_control" default="false"/>
-  <!-- common stuff -->
-  <xacro:include filename="$(find xarm_description)/urdf/common.gazebo.xacro" />
-  <!-- xarm6 -->
-  <xacro:include filename="$(find xarm_description)/urdf/xarm6.urdf.xacro" />
-  <xacro:include filename="$(find xarm_description)/urdf/xarm6.transmission.xacro" />
-  <xacro:include filename="$(find xarm_description)/urdf/xarm6.gazebo.xacro" />
-  <!-- arm -->
-  <xacro:gazebo_ros_control_plugin namespace="$(arg ros_control_namespace)"/>
-  <xacro:if value="$(arg limited)">
-    <xacro:xarm6_urdf prefix="$(arg prefix)"
-      joint1_lower_limit="${-pi*0.99}" joint1_upper_limit="${pi*0.99}"
-      joint2_lower_limit="${-2.18}" joint2_upper_limit="${2.18}"
-      joint3_lower_limit="${-pi*0.99}" joint3_upper_limit="${0.11}"
-      joint4_lower_limit="${-pi*0.99}" joint4_upper_limit="${pi*0.99}"
-      joint5_lower_limit="${-1.75}" joint5_upper_limit="${pi*0.99}"
-      joint6_lower_limit="${-pi*0.99}" joint6_upper_limit="${pi*0.99}"/>
-  </xacro:if>
-  <xacro:unless value="$(arg limited)">
-    <xacro:xarm6_urdf prefix="$(arg prefix)"/>
-  </xacro:unless>
-  <xacro:if value="$(arg effort_control)">
-    <xacro:xarm6_transmission prefix="$(arg prefix)" hard_interface="EffortJointInterface" />
-  </xacro:if>
-  <xacro:unless value="$(arg effort_control)">
-    <xacro:xarm6_transmission prefix="$(arg prefix)" hard_interface="PositionJointInterface" />
-  </xacro:unless>
-  <xacro:xarm6_gazebo prefix="$(arg prefix)" />
-  <link name="world" />
-  <joint name="world_joint" type="fixed">
-    <parent link="world" />
-    <child link = "$(arg prefix)link_base" />
-    <origin xyz="0.0 0.0 0.0" rpy="0.0 0.0 0.0" />
-  </joint>
+  <!-- load xarm6 robot -->
+  <xacro:include filename="$(find xarm_description)/urdf/xarm6_robot_macro.xacro" />
+  <xacro:xarm6_robot prefix="$(arg prefix)" namespace="$(arg ros_namespace)" limited="$(arg limited)" effort_control="$(arg effort_control)"/>
 </robot>
