Commit message: updated solid model

File: xarm_description/urdf/xarm5.urdf.xacro (robot description, xacro)
@@ -100,5 +100,5 @@
       <origin
         xyz="0 0 0.267"
-        rpy="-1.5708 0 0" />
+        rpy="0 0 0" />
       <parent
         link="${prefix}link_base" />
@@ -106,6 +106,6 @@
         link="${prefix}link1" />
       <axis
-        xyz="0 1 0" />
-      <limit
+        xyz="0 0 1" />
+     <limit
         lower="${joint1_lower_limit}"
         upper="${joint1_upper_limit}"
@@ -157,5 +157,5 @@
       <origin
         xyz="0 0 0"
-        rpy="0 0 0" />
+        rpy="-1.5708 0 0" />
       <parent
         link="${prefix}link1" />

File: xarm_description/urdf/xarm7.urdf.xacro (robot description, xacro)
@@ -22,296 +22,442 @@
       <color rgba="1.0 1.0 1.0 1.0"/>
     </material>
-    <link name="${prefix}link_base">
-      <visual>
-        <geometry>
-          <mesh filename="package://xarm_description/meshes/xarm7/visual/base.stl"/>
-        </geometry>
-        <origin xyz="0 0 0" rpy="0 0 0"/>
-        <material name="White" />
-      </visual>
-      <collision>
-        <geometry>
-          <mesh filename="package://xarm_description/meshes/xarm7/visual/base.stl"/>
-        </geometry>
-        <origin xyz="0 0 0" rpy="0 0 0"/>
-      </collision>
-      <inertial>
-        <origin xyz="0.00092 -0.00014 0.07508" rpy="0 0 0"/>
-        <mass value="2.28"/>
-      <inertia
-        ixx="0.0090315"
-        ixy="5.17E-06"
-        ixz="-0.00013262"
-        iyy="0.0084154"
-        iyz="-3.97E-06"
-        izz="0.0044873"/>
-      </inertial>
-    </link>
-    <link name="${prefix}link1">
-      <visual>
-        <geometry>
-          <mesh filename="package://xarm_description/meshes/xarm7/visual/link1.stl"/>
-        </geometry>
-        <origin xyz="0 0 -0.261" rpy="0 0 0"/>
-        <material name="White" />
-      </visual>
-      <collision>
-        <geometry>
-          <mesh filename="package://xarm_description/meshes/xarm7/visual/link1.stl"/>
-        </geometry>
-        <origin xyz="0 0 -0.261" rpy="0 0 0"/>
-      </collision>
-      <inertial>
-        <origin xyz="0.00017 0.02867 -0.00967" rpy="0 0 0"/>
-        <mass value="1.77"/>
-        <inertia
-          ixx="0.0039077"
-          ixy="2.49E-06"
-          ixz="-1.69E-06"
-          iyy="0.0035025"
-          iyz="-0.00054831"
-          izz="0.0024964"/>
-      </inertial>
-    </link>
-    <joint name="${prefix}joint1" type="revolute">
-      <parent link="${prefix}link_base"/>
-      <child  link="${prefix}link1"/>
-      <origin xyz="0 0 0.261" rpy="0 0 0"/>
-      <axis   xyz="0 0 1"/>
-      <limit
-        lower="${joint1_lower_limit}"
-        upper="${joint1_upper_limit}"
-        effort="50.0"
-        velocity="3.14"/>
-      <dynamics damping="1.0" friction="1.0"/>
-    </joint>
-    <link name="${prefix}link2">
-      <visual>
-        <geometry>
-          <mesh filename="package://xarm_description/meshes/xarm7/visual/link2.stl"/>
-        </geometry>
-        <origin xyz="0 0.261 0" rpy="1.5708 0 0"/>
-        <material name="White" />
-      </visual>
-      <collision>
-        <geometry>
-          <mesh filename="package://xarm_description/meshes/xarm7/visual/link2.stl"/>
-        </geometry>
-        <origin xyz="0 0.261 0" rpy="1.5708 0 0"/>
-      </collision>
-      <inertial>
-        <origin xyz="1E-05 -0.13885 0.0139" rpy="0 0 0"/>
-        <mass value="1.51"/>
-        <inertia
-          ixx="0.0071397"
-          ixy="3.02E-06"
-          ixz="-3.01E-05"
-          iyy="0.0026516"
-          iyz="0.001979"
-          izz="0.0061118"/>
-      </inertial>
-    </link>
-    <joint name="${prefix}joint2" type="revolute">
-      <parent link="${prefix}link1"/>
-      <child link="${prefix}link2"/>
-      <origin xyz="0 0 0" rpy="-1.5708 0 0" />
-      <axis xyz="0 0 1"/>
-      <limit
-        lower="${joint2_lower_limit}"
-        upper="${joint2_upper_limit}"
-        effort="50.0"
-        velocity="3.14"/>
-      <dynamics damping="1.0" friction="1.0"/>
-    </joint>
-    <link name="${prefix}link3">
-      <visual>
-        <geometry>
-          <mesh filename="package://xarm_description/meshes/xarm7/visual/link3.stl"/>
-        </geometry>
-        <origin xyz="0 0 -0.546" rpy="0 0 0"/>
-        <material name="White" />
-      </visual>
-      <collision>
-        <geometry>
-          <mesh filename="package://xarm_description/meshes/xarm7/visual/link3.stl"/>
-        </geometry>
-        <origin xyz="0 0 -0.546" rpy="0 0 0"/>
-      </collision>
-      <inertial>
-        <origin xyz="0.04387 0.02142 -0.00835" rpy="0 0 0"/>
-        <mass value="1.33"/>
-        <inertia
-          ixx="0.0023676"
-          ixy="0.00021885"
-          ixz="0.00049035"
-          iyy="0.0023241"
-          iyz="0.00025284"
-          izz="0.0018927"/>
-      </inertial>
-    </link>
-    <joint name="${prefix}joint3" type="revolute">
-      <parent link="${prefix}link2"/>
-      <child link="${prefix}link3"/>
-      <origin xyz="0 -0.285 0" rpy="1.5708 0 0"/>
-      <axis xyz="0 0 1"/>
-      <limit
-        lower="${joint3_lower_limit}"
-        upper="${joint3_upper_limit}"
-        effort="32.0"
-        velocity="3.14"/>
-      <dynamics damping="1.0" friction="1.0"/>
-    </joint>
-    <link name="${prefix}link4">
-      <visual>
-        <geometry>
-          <mesh filename="package://xarm_description/meshes/xarm7/visual/link4.stl"/>
-        </geometry>
-        <origin xyz="-0.050 0.546 0" rpy="1.5708 0 0"/>
-        <material name="White" />
-      </visual>
-      <collision>
-        <geometry>
-          <mesh filename="package://xarm_description/meshes/xarm7/visual/link4.stl"/>
-        </geometry>
-        <origin xyz="-0.050 0.546 0" rpy="1.5708 0 0"/>
-      </collision>
-      <inertial>
-        <origin xyz="0.07059 0.11905 0.01071" rpy="0 0 0"/>
-        <mass value="1.43"/>
-        <inertia
-          ixx="0.0046571"
-          ixy="0.0012392"
-          ixz="-0.00056448"
-          iyy="0.0028189"
-          iyz="-0.0011969"
-          izz="0.0046273"/>
-      </inertial>
-    </link>
-    <joint name="${prefix}joint4" type="revolute">
-      <parent link="${prefix}link3"/>
-      <child link="${prefix}link4"/>
-      <origin xyz="0.05 0 0" rpy="-1.5708 0 0"/>
-      <axis xyz="0 0 1"/>
-      <limit
-        lower="${joint4_lower_limit}"
-        upper="${joint4_upper_limit}"
-        effort="32.0"
-        velocity="3.14"/>
-      <dynamics damping="1.0" friction="1.0"/>
-    </joint>
-    <link name="${prefix}link5">
-      <visual>
-        <geometry>
-          <mesh filename="package://xarm_description/meshes/xarm7/visual/link5.stl"/>
-        </geometry>
-        <origin xyz="-0.1285 0 0.210" rpy="3.1416 0 0"/>
-        <material name="White" />
-      </visual>
-      <collision>
-        <geometry>
-          <mesh filename="package://xarm_description/meshes/xarm7/visual/link5.stl"/>
-        </geometry>
-        <origin xyz="-0.1285 0 -0.210" rpy="0 0 0"/>
-      </collision>
-      <inertial>
-        <origin xyz="-0.1285 0 0.210" rpy="3.1416 0 0"/>
-        <mass value="0.99"/>
-        <inertia
-          ixx="0.0042795"
-          ixy="-3.42E-06"
-          ixz="-1.61E-06"
-          iyy="0.004111"
-          iyz="0.00032311"
-          izz="0.00092663"/>
-      </inertial>
-    </link>
-    <joint name="${prefix}joint5" type="revolute">
-      <parent link="${prefix}link4"/>
-      <child link="${prefix}link5"/>
-      <origin xyz="0.0785 0.336 0" rpy="-1.5708 0 0"/>
-      <axis xyz="0 0 1"/>
-      <limit
-        lower="${joint5_lower_limit}"
-        upper="${joint5_upper_limit}"
-        effort="32.0"
-        velocity="3.14"/>
-      <dynamics damping="1.0" friction="1.0"/>
-    </joint>
-    <link name="${prefix}link6">
-      <visual>
-        <geometry>
-          <mesh filename="package://xarm_description/meshes/xarm7/visual/link6.stl"/>
-        </geometry>
-        <origin xyz="-0.1285 0.210 0" rpy="1.5708 0 0"/>
-        <material name="White" />
-      </visual>
-      <collision>
-        <geometry>
-          <mesh filename="package://xarm_description/meshes/xarm7/visual/link6.stl"/>
-        </geometry>
-        <origin xyz="-0.1285 0.210 0" rpy="1.5708 0 0"/>
-      </collision>
-      <inertial>
-        <origin xyz="0.06596 0.00669 0.00097" rpy="0 0 0"/>
-        <mass value="0.9" />
-        <inertia
-          ixx="0.0006881"
-          ixy="4.074E-05"
-          ixz="-4.565E-05"
-          iyy="0.0010127"
-          iyz="-3.39E-06"
-          izz="0.0011106"/>
-      </inertial>
-    </link>
-    <joint name="${prefix}joint6" type="revolute">
-      <parent link="${prefix}link5"/>
-      <child link="${prefix}link6"/>
-      <origin xyz="0 0 0" rpy="1.5708 0 0"/>
-      <axis xyz="0 0 1"/>
-      <limit
-        lower="${joint6_lower_limit}"
-        upper="${joint6_upper_limit}"
-        effort="20.0"
-        velocity="3.14"/>
-      <dynamics damping="1.0" friction="1.0"/>
-    </joint>
-    <link name="${prefix}link7">
-      <visual>
-        <geometry>
-          <mesh filename="package://xarm_description/meshes/xarm7/visual/link7.stl"/>
-        </geometry>
-        <origin xyz="-0.2015 0 0.1405" rpy="3.1416 0 0"/>
-        <material name="White" />
-      </visual>
-      <collision>
-        <geometry>
-          <mesh filename="package://xarm_description/meshes/xarm7/visual/link7.stl"/>
-        </geometry>
-        <origin xyz="-0.2015 0 0.1405" rpy="3.1416 0 0"/>
-      </collision>
-      <inertial>
-        <origin xyz="-3.5072E-05 9.5542E-06 -0.022065" rpy="0 0 0"/>
-        <mass value="0.236"/>
-        <inertia
-          ixx="0.00018795"
-          ixy="2.4125E-07"
-          ixz="1.7234E-07"
-          iyy="0.00018921"
-          iyz="-4.3124E-08"
-          izz="0.00022645"/>
-      </inertial>
-    </link>
-    <joint name="${prefix}joint7" type="revolute">
-      <parent link="${prefix}link6"/>
-      <child link="${prefix}link7"/>
-      <origin xyz="0.073 0.0695 0" rpy="-1.5708 0 0"/>
-      <axis xyz="0 0 1"/>
-      <limit
-        lower="${joint7_lower_limit}"
-        upper="${joint7_upper_limit}"
-        effort="20.0"
-        velocity="3.14"/>
-      <dynamics damping="1.0" friction="1.0"/>
-    </joint>
+    <material name="Silver">
+      <color rgba="0.753 0.753 0.753 1.0"/>
+    </material>
+    <link
+    name="${prefix}link_base">
+    <inertial>
+      <origin
+        xyz="-0.021131 -0.0016302 0.056488"
+        rpy="0 0 0" />
+      <mass
+        value="0.88556" />
+      <inertia
+        ixx="0.0030595"
+        ixy="0.00012259"
+        ixz="-0.00062705"
+        iyy="0.0037783"
+        iyz="0.00027023"
+        izz="0.0020125" />
+    </inertial>
+    <visual>
+      <origin
+        xyz="0 0 0"
+        rpy="0 0 0" />
+      <geometry>
+        <mesh
+          filename="package://xarm_description/meshes/xarm7/visual/link_base.STL" />
+      </geometry>
+      <material name="White" />
+    </visual>
+    <collision>
+      <origin
+        xyz="0 0 0"
+        rpy="0 0 0" />
+      <geometry>
+        <mesh
+          filename="package://xarm_description/meshes/xarm7/visual/link_base.STL" />
+      </geometry>
+    </collision>
+  </link>
+  <link
+    name="${prefix}link1">
+    <inertial>
+      <origin
+        xyz="-0.0042142 0.02821 -0.0087788"
+        rpy="0 0 0" />
+      <mass
+        value="0.42603" />
+      <inertia
+        ixx="0.0014243"
+        ixy="3.9946E-05"
+        ixz="4.7078E-06"
+        iyy="0.00123"
+        iyz="-0.00026073"
+        izz="0.00099229" />
+    </inertial>
+    <visual>
+      <origin
+        xyz="0 0 0"
+        rpy="0 0 0" />
+      <geometry>
+        <mesh
+          filename="package://xarm_description/meshes/xarm7/visual/link1.STL" />
+      </geometry>
+      <material name="White" />
+    </visual>
+    <collision>
+      <origin
+        xyz="0 0 0"
+        rpy="0 0 0" />
+      <geometry>
+        <mesh
+          filename="package://xarm_description/meshes/xarm7/visual/link1.STL" />
+      </geometry>
+    </collision>
+  </link>
+  <joint
+    name="${prefix}joint1"
+    type="revolute">
+    <origin
+      xyz="0 0 0.267"
+      rpy="0 0 0" />
+    <parent
+      link="${prefix}link_base" />
+    <child
+      link="${prefix}link1" />
+    <axis
+      xyz="0 0 1" />
+    <limit
+      lower="${joint1_lower_limit}"
+      upper="${joint1_upper_limit}"
+      effort="50"
+      velocity="3.14" />
+    <dynamics
+      damping="10"
+      friction="1" />
+  </joint>
+  <link
+    name="${prefix}link2">
+    <inertial>
+      <origin
+        xyz="-3.3178E-05 -0.12849 0.026337"
+        rpy="0 0 0" />
+      <mass
+        value="0.56095" />
+      <inertia
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
File: xarm_description/urdf/xarm7_robot.urdf.xacro (robot description, xacro)
@@ -1,42 +1,10 @@
-<?xml version="1.0"?>
-<robot xmlns:xacro="http://ros.org/wiki/xacro"
-       name="xarm7" >
+<?xml version='1.0' encoding='utf-8'?>
+<robot xmlns:xacro="http://ros.org/wiki/xacro" name="xarm7">
   <xacro:arg name="prefix" default=""/>
-  <xacro:arg name="ros_control_namespace" default="xarm"/>
+  <xacro:arg name="ros_namespace" default="xarm"/>
   <xacro:arg name="limited" default="false"/>
   <xacro:arg name="effort_control" default="false"/>
-  <!-- common stuff -->
-  <xacro:include filename="$(find xarm_description)/urdf/common.gazebo.xacro" />
-  <!-- xarm7 -->
-  <xacro:include filename="$(find xarm_description)/urdf/xarm7.urdf.xacro" />
-  <xacro:include filename="$(find xarm_description)/urdf/xarm7.transmission.xacro" />
-  <xacro:include filename="$(find xarm_description)/urdf/xarm7.gazebo.xacro" />
-  <!-- arm -->
-  <xacro:gazebo_ros_control_plugin namespace="$(arg ros_control_namespace)"/>
-  <xacro:if value="$(arg limited)">
-    <xacro:xarm7_urdf prefix="$(arg prefix)"
-      joint1_lower_limit="${-pi*0.99}" joint1_upper_limit="${pi*0.99}"
-      joint2_lower_limit="${-2.18}" joint2_upper_limit="${2.18}"
-      joint3_lower_limit="${-pi*0.99}" joint3_upper_limit="${pi*0.99}"
-      joint4_lower_limit="${-pi*0.99}" joint4_upper_limit="${0.11}"
-      joint5_lower_limit="${-pi*0.99}" joint5_upper_limit="${pi*0.99}"
-      joint6_lower_limit="${-1.75}" joint6_upper_limit="${pi*0.99}"
-      joint7_lower_limit="${-pi*0.99}" joint7_upper_limit="${pi*0.99}"/>
-  </xacro:if>
-  <xacro:unless value="$(arg limited)">
-    <xacro:xarm7_urdf prefix="$(arg prefix)"/>
-  </xacro:unless>
-  <xacro:if value="$(arg effort_control)">
-    <xacro:xarm7_transmission prefix="$(arg prefix)" hard_interface="EffortJointInterface" />
-  </xacro:if>
-  <xacro:unless value="$(arg effort_control)">
-    <xacro:xarm7_transmission prefix="$(arg prefix)" hard_interface="PositionJointInterface" />
-  </xacro:unless>
-  <xacro:xarm7_gazebo prefix="$(arg prefix)" />
-  <link name="world" />
-  <joint name="world_joint" type="fixed">
-    <parent link="world" />
-    <child link = "$(arg prefix)link_base" />
-    <origin xyz="0.0 0.0 0.0" rpy="0.0 0.0 0.0" />
-  </joint>
+  <!-- load xarm7 robot -->
+  <xacro:include filename="$(find xarm_description)/urdf/xarm7_robot_macro.xacro" />
+  <xacro:xarm7_robot prefix="$(arg prefix)" namespace="$(arg ros_namespace)" limited="$(arg limited)" effort_control="$(arg effort_control)"/>
 </robot>

Commit message: xarm5 model bug fix

File: xarm_description/urdf/xarm5.urdf.xacro (robot description, xacro)
@@ -100,5 +100,5 @@
       <origin
         xyz="0 0 0.267"
-        rpy="-1.5708 0 0" />
+        rpy="0 0 0" />
       <parent
         link="${prefix}link_base" />
@@ -106,6 +106,6 @@
         link="${prefix}link1" />
       <axis
-        xyz="0 -1 0" />
-      <limit
+        xyz="0 0 1" />
+     <limit
         lower="${joint1_lower_limit}"
         upper="${joint1_upper_limit}"
@@ -157,5 +157,5 @@
       <origin
         xyz="0 0 0"
-        rpy="0 0 0" />
+        rpy="-1.5708 0 0" />
       <parent
         link="${prefix}link1" />

Commit message: update DH and report length

File: xarm_description/urdf/xarm5.urdf.xacro (robot description, xacro)
@@ -213,5 +213,5 @@
       type="revolute">
       <origin
-        xyz="0.053316 -0.28467 0"
+        xyz="0.0535 -0.2845 0"
         rpy="0 0 0" />
       <parent
@@ -270,6 +270,6 @@
       type="revolute">
       <origin
-        xyz="0.077752 0.34198 0"
-        rpy="2.6191E-47 0 7.5847E-47" />
+        xyz="0.0775 0.3425 0"
+        rpy="0 0 0" />
       <parent
         link="${prefix}link3" />
@@ -327,6 +327,6 @@
       type="revolute">
       <origin
-        xyz="0.076 0.09702 0"
-        rpy="-1.5708 0 7.5847E-47" />
+        xyz="0.076 0.097 0"
+        rpy="-1.5708 0 0" />
       <parent
         link="${prefix}link4" />

File: xarm_description/urdf/xarm6.urdf.xacro (robot description, xacro)
@@ -161,5 +161,5 @@
       <parent link="${prefix}link2"/>
       <child link="${prefix}link3"/>
-      <origin xyz="0.053 -0.2845 0" rpy="0 0 0"/>
+      <origin xyz="0.0535 -0.2845 0" rpy="0 0 0"/>
       <axis xyz="0 0 1"/>
       <limit
@@ -199,5 +199,5 @@
       <parent link="${prefix}link3"/>
       <child link="${prefix}link4"/>
-      <origin xyz="0.07775 0.342 0" rpy="-1.5708 0 0"/>
+      <origin xyz="0.0775 0.3425 0" rpy="-1.5708 0 0"/>
       <axis xyz="0 0 1"/>
       <limit

File: xarm_description/urdf/xarm7.urdf.xacro (robot description, xacro)
@@ -272,5 +272,5 @@
     type="revolute">
     <origin
-      xyz="0.052423 0 0"
+      xyz="0.0525 0 0"
       rpy="1.5708 0 0" />
     <parent
@@ -329,5 +329,5 @@
     type="revolute">
     <origin
-      xyz="0.077751 -0.34248 0"
+      xyz="0.0775 -0.3425 0"
       rpy="1.5708 0 0" />
     <parent
@@ -443,5 +443,5 @@
     type="revolute">
     <origin
-      xyz="0.076 0.09702 0"
+      xyz="0.076 0.097 0"
       rpy="-1.5708 0 0" />
     <parent
