Commit message: fixed the use of prefix and added prefix to world_joint

File: xarm_description/urdf/xarm7_robot_macro.xacro (robot description, xacro)
@@ -15,5 +15,5 @@
       <link name="world" />
     </xacro:if>
-    <joint name="world_joint" type="fixed">
+    <joint name="${prefix}world_joint" type="fixed">
       <parent link="${attach_to}" />
       <child link = "${prefix}link_base" />
@@ -21,5 +21,5 @@
     </joint>
     <xacro:if value="$(arg limited)">
-      <xacro:xarm7_urdf prefix="$(arg prefix)"
+      <xacro:xarm7_urdf prefix="${prefix}"
         joint1_lower_limit="${-pi*0.99}" joint1_upper_limit="${pi*0.99}"
         joint2_lower_limit="${-2.18}" joint2_upper_limit="${2.18}"
@@ -31,13 +31,13 @@
     </xacro:if>
     <xacro:unless value="$(arg limited)">
-      <xacro:xarm7_urdf prefix="$(arg prefix)"/>
+      <xacro:xarm7_urdf prefix="${prefix}"/>
     </xacro:unless>
     <xacro:if value="$(arg effort_control)">
-      <xacro:xarm7_transmission prefix="$(arg prefix)" hard_interface="EffortJointInterface" />
+      <xacro:xarm7_transmission prefix="${prefix}" hard_interface="EffortJointInterface" />
     </xacro:if>
     <xacro:unless value="$(arg effort_control)">
-      <xacro:xarm7_transmission prefix="$(arg prefix)" hard_interface="PositionJointInterface" />
+      <xacro:xarm7_transmission prefix="${prefix}" hard_interface="PositionJointInterface" />
     </xacro:unless>
-    <xacro:xarm7_gazebo prefix="$(arg prefix)" />
+    <xacro:xarm7_gazebo prefix="${prefix}" />
   </xacro:macro>
 </robot>
