Commit message: better 6dof support

File: xarm_description/urdf/xarm6.urdf.xacro (robot description, xacro)
@@ -90,5 +90,5 @@
           <mesh filename="package://xarm_description/meshes/xarm6/visual/link2.stl"/>
         </geometry>
-        <origin xyz="0 0 -0.267" rpy="0 0 0"/>
+        <origin xyz="0 0.267 0" rpy="1.5708 0 0"/>
         <material name="White" />
       </visual>
@@ -97,23 +97,26 @@
           <mesh filename="package://xarm_description/meshes/xarm6/visual/link2.stl"/>
         </geometry>
-        <origin xyz="0 0 -0.267" rpy="0 0 0"/>
-      </collision>
-      <inertial>
-        <origin xyz="0.03917 0.03011 0.22939" rpy="0 0 0"/>
-        <mass value="1.59"/>
-        <inertia
-          ixx="0.01861081"
-          ixy="-0.00054949"
-          ixz="0.00325036"
-          iyy="0.0175515"
-          iyz="-0.0036833"
-          izz="0.00437426"/>
-      </inertial>
+        <origin xyz="0 0.267 0" rpy="1.5708 0 0"/>
+      </collision>
+      <inertial>
+      <origin
+        xyz="0.03917 -0.22939 0.03011"
+        rpy="0 0 0" />
+      <mass
+        value="1.59" />
+      <inertia
+        ixx="0.0186108"
+        ixy="-0.0032504"
+        ixz="-0.00054949"
+        iyy="0.00437426"
+        iyz="0.0036833"
+        izz="0.0175515" />
+    </inertial>
     </link>
     <joint name="${prefix}joint2" type="revolute">
       <parent link="${prefix}link1"/>
       <child link="${prefix}link2"/>
-      <origin xyz="0 0 0" rpy="0 0 0"/>
-      <axis xyz="0 1 0"/>
+      <origin xyz="0 0 0" rpy="-1.5708 0 0" />
+      <axis xyz="0 0 1"/>
       <limit
         lower="${joint2_lower_limit}"
@@ -128,5 +131,5 @@
           <mesh filename="package://xarm_description/meshes/xarm6/visual/link3.stl"/>
         </geometry>
-        <origin xyz="-0.0525 0 -0.550" rpy="0 0 0"/>
+        <origin xyz="-0.0525 0.550 0" rpy="1.5708 0 0"/>
         <material name="White" />
       </visual>
@@ -135,23 +138,26 @@
           <mesh filename="package://xarm_description/meshes/xarm6/visual/link3.stl"/>
         </geometry>
-        <origin xyz="-0.0525 0 -0.550" rpy="0 0 0"/>
-      </collision>
-      <inertial>
-        <origin xyz="0.06673 0.01669 -0.1027" rpy="0 0 0"/>
-        <mass value="1.38"/>
-        <inertia
-          ixx="0.00503299"
-          ixy="-0.00090286"
-          ixz="-0.001304"
-          iyy="0.00460762"
-          iyz="0.00161202"
-          izz="0.00311993"/>
-      </inertial>
+        <origin xyz="-0.0525 0.550 0" rpy="1.5708 0 0"/>
+      </collision>
+      <inertial>
+      <origin
+        xyz="0.06673 0.1027 0.01669"
+        rpy="0 0 0" />
+      <mass
+        value="1.38" />
+      <inertia
+        ixx="0.00503299"
+        ixy="0.001304"
+        ixz="-0.00090286"
+        iyy="0.00311993"
+        iyz="-0.00161202"
+        izz="0.00460762" />
+    </inertial>
     </link>
     <joint name="${prefix}joint3" type="revolute">
       <parent link="${prefix}link2"/>
       <child link="${prefix}link3"/>
-      <origin xyz= "0.0525 0 0.2845" rpy="0 0 0"/>
-      <axis xyz="0 1 0"/>
+      <origin xyz="0.0525 -0.2845 0" rpy="0 0 0"/>
+      <axis xyz="0 0 1"/>
       <limit
         lower="${joint3_lower_limit}"
@@ -166,5 +172,5 @@
           <mesh filename="package://xarm_description/meshes/xarm6/visual/link4.stl"/>
         </geometry>
-        <origin xyz="-0.13025 0 -0.2075" rpy="0 0 0"/>
+        <origin xyz="-0.13025 0 0.2075" rpy="3.1416 0 0"/>
         <material name="White" />
       </visual>
@@ -173,8 +179,8 @@
           <mesh filename="package://xarm_description/meshes/xarm6/visual/link4.stl"/>
         </geometry>
-        <origin xyz="-0.13025 0 -0.2075" rpy="0 0 0"/>
-      </collision>
-      <inertial>
-        <origin xyz="-0.0006 -0.02398 0.02548" rpy="0 0 0"/>
+        <origin xyz="-0.13025 0 0.2075" rpy="3.1416 0 0"/>
+      </collision>
+      <inertial>
+        <origin xyz="-0.0006 0.02398 -0.02548" rpy="0 0 0"/>
         <mass value="1.11"/>
         <inertia
@@ -190,6 +196,6 @@
       <parent link="${prefix}link3"/>
       <child link="${prefix}link4"/>
-      <origin xyz="0.07775 0 -0.3425" rpy="0 0 0"/>
-      <axis xyz="0 0 -1"/>
+      <origin xyz="0.07775 0.3425 0" rpy="-1.5708 0 0"/>
+      <axis xyz="0 0 1"/>
       <limit
         lower="${joint4_lower_limit}"
@@ -204,5 +210,5 @@
           <mesh filename="package://xarm_description/meshes/xarm6/visual/link5.stl"/>
         </geometry>
-        <origin xyz="-0.13025 0 -0.2075" rpy="0 0 0"/>
+        <origin xyz="-0.13025 0.2075 0" rpy="1.5708 0 0"/>
         <material name="White" />
       </visual>
@@ -211,23 +217,26 @@
           <mesh filename="package://xarm_description/meshes/xarm6/visual/link5.stl"/>
         </geometry>
-        <origin xyz="-0.13025 0 -0.2075" rpy="0 0 0"/>
-      </collision>
-      <inertial>
-        <origin xyz="0.06506 0.00355 -0.02154" rpy="0 0 0"/>
-        <mass value="1.06"/>
-        <inertia
-          ixx="0.00095833"
-          ixy="-0.00020353"
-          ixz="-0.00024313"
-          iyy="0.00170033"
-          iyz="7.753E-05"
-          izz="0.00137284"/>
-      </inertial>
+        <origin xyz="-0.13025 0.2075 0" rpy="1.5708 0 0"/>
+      </collision>
+      <inertial>
+      <origin
+        xyz="0.06508 0.02146 0.00355"
+        rpy="0 0 0" />
+      <mass
+        value="1.06" />
+      <inertia
+        ixx="0.00095773"
+        ixy="0.00024262"
+        ixz="-0.00020362"
+        iyy="0.00137344"
+        iyz="-7.728E-05"
+        izz="0.00170033" />
+    </inertial>
     </link>
     <joint name="${prefix}joint5" type="revolute">
       <parent link="${prefix}link4"/>
       <child link="${prefix}link5"/>
-      <origin xyz="0 0 0" rpy="0 0 0"/>
-      <axis xyz="0 1 0"/>
+      <origin xyz="0 0 0" rpy="1.5708 0 0"/>
+      <axis xyz="0 0 1"/>
       <limit
         lower="${joint5_lower_limit}"
@@ -242,5 +251,5 @@
           <mesh filename="package://xarm_description/meshes/xarm6/visual/link6.stl"/>
         </geometry>
-        <origin xyz="-0.20625 0 -0.128" rpy="0 0 0"/>
+        <origin xyz="-0.20625 0 0.128" rpy="3.1416 0 0"/>
         <material name="White" />
       </visual>
@@ -249,23 +258,26 @@
           <mesh filename="package://xarm_description/meshes/xarm6/visual/link6.stl"/>
         </geometry>
-        <origin xyz="-0.20625 0 -0.128" rpy="0 0 0"/>
-      </collision>
-      <inertial>
-        <origin xyz="-0.00061 0.00056 0.00749" rpy="0 0 0"/>
-        <mass value="0.1" />
-        <inertia
-          ixx="5.139E-05"
-          ixy="-1.76E-06"
-          ixz="-0.73E-06"
-          iyy="5.279E-05"
-          iyz="0.43E-06"
-          izz="9.249E-05"/>
-      </inertial>
+        <origin xyz="-0.20625 0 0.128" rpy="3.1416 0 0"/>
+      </collision>
+      <inertial>
+      <origin
+        xyz="-0.00060579 -0.00056166 -0.0074896"
+        rpy="0 0 0" />
+      <mass
+        value="0.10" />
+      <inertia
+        ixx="5.1386E-05"
+        ixy="-1.7552E-06"
+        ixz="-7.2889E-07"
+        iyy="5.2793E-05"
+        iyz="-4.3242E-07"
+        izz="9.2486E-05" />
+    </inertial>
     </link>
     <joint name="${prefix}joint6" type="revolute">
       <parent link="${prefix}link5"/>
       <child link="${prefix}link6"/>
-      <origin xyz="0.076 0 -0.0795" rpy=" 0 0 0"/>
-      <axis xyz="0 0 -1"/>
+      <origin xyz="0.076 0.0795 0" rpy="-1.5708 0 0"/>
+      <axis xyz="0 0 1"/>
       <limit
         lower="${joint6_lower_limit}"

File: xarm_description/urdf/xarm7.urdf.xacro (robot description, xacro)
@@ -91,5 +91,5 @@
           <mesh filename="package://xarm_description/meshes/xarm7/visual/link2.stl"/>
         </geometry>
-        <origin xyz="0 0 -0.261" rpy="0 0 0"/>
+        <origin xyz="0 0.261 0" rpy="1.5708 0 0"/>
         <material name="White" />
       </visual>
@@ -98,5 +98,5 @@
           <mesh filename="package://xarm_description/meshes/xarm7/visual/link2.stl"/>
         </geometry>
-        <origin xyz="0 0 -0.261" rpy="0 0 0"/>
+        <origin xyz="0 0.261 0" rpy="1.5708 0 0"/>
       </collision>
       <inertial>
@@ -115,6 +115,6 @@
       <parent link="${prefix}link1"/>
       <child link="${prefix}link2"/>
-      <origin xyz="0 0 0" rpy="0 0 0"/>
-      <axis xyz="0 1 0"/>
+      <origin xyz="0 0 0" rpy="-1.5708 0 0" />
+      <axis xyz="0 0 1"/>
       <limit
         lower="${joint2_lower_limit}"
@@ -153,5 +153,5 @@
       <parent link="${prefix}link2"/>
       <child link="${prefix}link3"/>
-      <origin xyz= "0 0 0.285" rpy="0 0 0"/>
+      <origin xyz="0 -0.285 0" rpy="1.5708 0 0"/>
       <axis xyz="0 0 1"/>
       <limit
@@ -167,5 +167,5 @@
           <mesh filename="package://xarm_description/meshes/xarm7/visual/link4.stl"/>
         </geometry>
-        <origin xyz="-0.050 0 -0.546" rpy="0 0 0"/>
+        <origin xyz="-0.050 0.546 0" rpy="1.5708 0 0"/>
         <material name="White" />
       </visual>
@@ -174,5 +174,5 @@
           <mesh filename="package://xarm_description/meshes/xarm7/visual/link4.stl"/>
         </geometry>
-        <origin xyz="-0.050 0 -0.546" rpy="0 0 0"/>
+        <origin xyz="-0.050 0.546 0" rpy="1.5708 0 0"/>
       </collision>
       <inertial>
@@ -191,6 +191,6 @@
       <parent link="${prefix}link3"/>
       <child link="${prefix}link4"/>
-      <origin xyz="0.050 0 0" rpy="0 0 0"/>
-      <axis xyz="0 1 0"/>
+      <origin xyz="0.05 0 0" rpy="-1.5708 0 0"/>
+      <axis xyz="0 0 1"/>
       <limit
         lower="${joint4_lower_limit}"
@@ -205,15 +205,15 @@
           <mesh filename="package://xarm_description/meshes/xarm7/visual/link5.stl"/>
         </geometry>
+        <origin xyz="-0.1285 0 0.210" rpy="3.1416 0 0"/>
+        <material name="White" />
+      </visual>
+      <collision>
+        <geometry>
+          <mesh filename="package://xarm_description/meshes/xarm7/visual/link5.stl"/>
+        </geometry>
         <origin xyz="-0.1285 0 -0.210" rpy="0 0 0"/>
-        <material name="White" />
-      </visual>
-      <collision>
-        <geometry>
-          <mesh filename="package://xarm_description/meshes/xarm7/visual/link5.stl"/>
-        </geometry>
-        <origin xyz="-0.1285 0 -0.210" rpy="0 0 0"/>
-      </collision>
-      <inertial>
-        <origin xyz="-0.00014 0.0234 -0.03053" rpy="0 0 0"/>
+      </collision>
+      <inertial>
+        <origin xyz="-0.1285 0 0.210" rpy="3.1416 0 0"/>
         <mass value="0.99"/>
         <inertia
@@ -229,6 +229,6 @@
       <parent link="${prefix}link4"/>
       <child link="${prefix}link5"/>
-      <origin xyz="0.0785 0 -0.336" rpy="0 0 0"/>
-      <axis xyz="0 0 -1"/>
+      <origin xyz="0.0785 0.336 0" rpy="-1.5708 0 0"/>
+      <axis xyz="0 0 1"/>
       <limit
         lower="${joint5_lower_limit}"
@@ -243,5 +243,5 @@
           <mesh filename="package://xarm_description/meshes/xarm7/visual/link6.stl"/>
         </geometry>
-        <origin xyz="-0.1285 0 -0.210" rpy="0 0 0"/>
+        <origin xyz="-0.1285 0.210 0" rpy="1.5708 0 0"/>
         <material name="White" />
       </visual>
@@ -250,5 +250,5 @@
           <mesh filename="package://xarm_description/meshes/xarm7/visual/link6.stl"/>
         </geometry>
-        <origin xyz="-0.1285 0 -0.210" rpy="0 0 0"/>
+        <origin xyz="-0.1285 0.210 0" rpy="1.5708 0 0"/>
       </collision>
       <inertial>
@@ -267,6 +267,6 @@
       <parent link="${prefix}link5"/>
       <child link="${prefix}link6"/>
-      <origin xyz="0 0 0" rpy=" 0 0 0"/>
-      <axis xyz="0 1 0"/>
+      <origin xyz="0 0 0" rpy="1.5708 0 0"/>
+      <axis xyz="0 0 1"/>
       <limit
         lower="${joint6_lower_limit}"
@@ -281,5 +281,5 @@
           <mesh filename="package://xarm_description/meshes/xarm7/visual/link7.stl"/>
         </geometry>
-        <origin xyz="-0.2015 0 -0.1405" rpy="0 0 0"/>
+        <origin xyz="-0.2015 0 0.1405" rpy="3.1416 0 0"/>
         <material name="White" />
       </visual>
@@ -288,5 +288,5 @@
           <mesh filename="package://xarm_description/meshes/xarm7/visual/link7.stl"/>
         </geometry>
-        <origin xyz="-0.2015 0 -0.1405" rpy="0 0 0"/>
+        <origin xyz="-0.2015 0 0.1405" rpy="3.1416 0 0"/>
       </collision>
       <inertial>
@@ -305,6 +305,6 @@
       <parent link="${prefix}link6"/>
       <child link="${prefix}link7"/>
-      <origin xyz="0.073 0 -0.0695" rpy="0 0 0"/>
-      <axis xyz="0 0 -1"/>
+      <origin xyz="0.073 0.0695 0" rpy="-1.5708 0 0"/>
+      <axis xyz="0 0 1"/>
       <limit
         lower="${joint7_lower_limit}"

Commit message: update xArm6 model

File: xarm_description/urdf/xarm6.urdf.xacro (robot description, xacro)
@@ -37,5 +37,5 @@
       <inertial>
       <origin xyz="0.0 0.0 0.09103" rpy="0 0 0" />
-      <mass value="1.91" />
+      <mass value="2.7" />
       <inertia
         ixx="0.00494875"
@@ -52,5 +52,5 @@
           <mesh filename="package://xarm_description/meshes/xarm6/visual/link1.stl"/>
         </geometry>
-        <origin xyz="0 0 -0.267" rpy="0 0 0"/>
+        <origin xyz="0 0 0" rpy="0 0 0"/>
         <material name="White" />
       </visual>
@@ -59,16 +59,16 @@
           <mesh filename="package://xarm_description/meshes/xarm6/visual/link1.stl"/>
         </geometry>
-        <origin xyz="0 0 -0.267" rpy="0 0 0"/>
-      </collision>
-      <inertial>
-        <origin xyz="0.0008 0.02437 -0.00926" rpy="0 0 0"/>
-        <mass value="1.77"/>
+        <origin xyz="0 0 0" rpy="0 0 0"/>
+      </collision>
+      <inertial>
+        <origin xyz="-0.002 0.02692 -0.01332" rpy="0 0 0"/>
+        <mass value="2.16"/>
         <inertia
-          ixx="0.0038513"
-          ixy="-1.745E-05"
-          ixz="1.382E-05"
-          iyy="0.00301075"
-          iyz="0.00041214"
-          izz="0.00261883"/>
+          ixx="0.00539427"
+          ixy="1.095E-05"
+          ixz="1.635E-06"
+          iyy="0.0048979"
+          iyz="0.000793"
+          izz="0.00311573"/>
       </inertial>
     </link>
@@ -90,5 +90,5 @@
           <mesh filename="package://xarm_description/meshes/xarm6/visual/link2.stl"/>
         </geometry>
-        <origin xyz="0 0.267 0" rpy="1.5708 0 0"/>
+        <origin xyz="0 0 0" rpy="0 0 0"/>
         <material name="White" />
       </visual>
@@ -97,19 +97,19 @@
           <mesh filename="package://xarm_description/meshes/xarm6/visual/link2.stl"/>
         </geometry>
-        <origin xyz="0 0.267 0" rpy="1.5708 0 0"/>
-      </collision>
-      <inertial>
-      <origin
-        xyz="0.03917 -0.22939 0.03011"
-        rpy="0 0 0" />
-      <mass
-        value="1.59" />
-      <inertia
-        ixx="0.0186108"
-        ixy="-0.0032504"
-        ixz="-0.00054949"
-        iyy="0.00437426"
-        iyz="0.0036833"
-        izz="0.0175515" />
+        <origin xyz="0 0 0" rpy="0 0 0"/>
+      </collision>
+      <inertial>
+      <origin
+        xyz="0.03531 -0.21398 0.03386"
+        rpy="0 0 0" />
+      <mass
+        value="1.71" />
+      <inertia
+        ixx="0.0248674"
+        ixy="-0.00430651"
+        ixz="-0.00067797"
+        iyy="0.00485548"
+        iyz="0.00457245"
+        izz="0.02387827" />
     </inertial>
     </link>
@@ -131,5 +131,5 @@
           <mesh filename="package://xarm_description/meshes/xarm6/visual/link3.stl"/>
         </geometry>
-        <origin xyz="-0.0525 0.550 0" rpy="1.5708 0 0"/>
+        <origin xyz="0 0 0" rpy="0 0 0"/>
         <material name="White" />
       </visual>
@@ -138,19 +138,19 @@
           <mesh filename="package://xarm_description/meshes/xarm6/visual/link3.stl"/>
         </geometry>
-        <origin xyz="-0.0525 0.550 0" rpy="1.5708 0 0"/>
-      </collision>
-      <inertial>
-      <origin
-        xyz="0.06673 0.1027 0.01669"
-        rpy="0 0 0" />
-      <mass
-        value="1.38" />
-      <inertia
-        ixx="0.00503299"
-        ixy="0.001304"
-        ixz="-0.00090286"
-        iyy="0.00311993"
-        iyz="-0.00161202"
-        izz="0.00460762" />
+        <origin xyz="0 0 0" rpy="0 0 0"/>
+      </collision>
+      <inertial>
+      <origin
+        xyz="0.06781 0.10749 0.01457"
+        rpy="0 0 0" />
+      <mass
+        value="1.384" />
+      <inertia
+        ixx="0.0053694"
+        ixy="0.0014185"
+        ixz="-0.00092094"
+        iyy="0.0032423"
+        iyz="-0.00169178"
+        izz="0.00501731" />
     </inertial>
     </link>
@@ -158,5 +158,5 @@
       <parent link="${prefix}link2"/>
       <child link="${prefix}link3"/>
-      <origin xyz="0.0525 -0.2845 0" rpy="0 0 0"/>
+      <origin xyz="0.053 -0.2845 0" rpy="0 0 0"/>
       <axis xyz="0 0 1"/>
       <limit
@@ -172,5 +172,5 @@
           <mesh filename="package://xarm_description/meshes/xarm6/visual/link4.stl"/>
         </geometry>
-        <origin xyz="-0.13025 0 0.2075" rpy="3.1416 0 0"/>
+        <origin xyz="0 0 0" rpy="0 0 0"/>
         <material name="White" />
       </visual>
@@ -179,16 +179,16 @@
           <mesh filename="package://xarm_description/meshes/xarm6/visual/link4.stl"/>
         </geometry>
-        <origin xyz="-0.13025 0 0.2075" rpy="3.1416 0 0"/>
-      </collision>
-      <inertial>
-        <origin xyz="-0.0006 0.02398 -0.02548" rpy="0 0 0"/>
-        <mass value="1.11"/>
+        <origin xyz="0 0 0" rpy="0 0 0"/>
+      </collision>
+      <inertial>
+        <origin xyz="-0.00021 0.02578 -0.02538" rpy="0 0 0"/>
+        <mass value="1.115"/>
         <inertia
-          ixx="0.00433331"
-          ixy="1.863E-05"
-          ixz="1.0E-05"
-          iyy="0.00394289"
-          iyz="0.00044082"
-          izz="0.00111454"/>
+          ixx="0.00439263"
+          ixy="5.028E-05"
+          ixz="1.374E-05"
+          iyy="0.0040077"
+          iyz="0.00045338"
+          izz="0.00110321"/>
       </inertial>
     </link>
@@ -196,5 +196,5 @@
       <parent link="${prefix}link3"/>
       <child link="${prefix}link4"/>
-      <origin xyz="0.07775 0.3425 0" rpy="-1.5708 0 0"/>
+      <origin xyz="0.07775 0.342 0" rpy="-1.5708 0 0"/>
       <axis xyz="0 0 1"/>
       <limit
@@ -210,5 +210,5 @@
           <mesh filename="package://xarm_description/meshes/xarm6/visual/link5.stl"/>
         </geometry>
-        <origin xyz="-0.13025 0.2075 0" rpy="1.5708 0 0"/>
+        <origin xyz="0 0 0" rpy="0 0 0"/>
         <material name="White" />
       </visual>
@@ -217,19 +217,19 @@
           <mesh filename="package://xarm_description/meshes/xarm6/visual/link5.stl"/>
         </geometry>
-        <origin xyz="-0.13025 0.2075 0" rpy="1.5708 0 0"/>
-      </collision>
-      <inertial>
-      <origin
-        xyz="0.06508 0.02146 0.00355"
-        rpy="0 0 0" />
-      <mass
-        value="1.06" />
-      <inertia
-        ixx="0.00095773"
-        ixy="0.00024262"
-        ixz="-0.00020362"
-        iyy="0.00137344"
-        iyz="-7.728E-05"
-        izz="0.00170033" />
+        <origin xyz="0 0 0" rpy="0 0 0"/>
+      </collision>
+      <inertial>
+      <origin
+        xyz="0.05428 0.01781 0.00543"
+        rpy="0 0 0" />
+      <mass
+        value="1.275" />
+      <inertia
+        ixx="0.001202758"
+        ixy="0.000492428"
+        ixz="-0.00039147"
+        iyy="0.0022876"
+        iyz="-1.235E-04"
+        izz="0.0026866" />
     </inertial>
     </link>
@@ -251,5 +251,5 @@
           <mesh filename="package://xarm_description/meshes/xarm6/visual/link6.stl"/>
         </geometry>
-        <origin xyz="-0.20625 0 0.128" rpy="3.1416 0 0"/>
+        <origin xyz="0 0 0" rpy="0 0 0"/>
         <material name="White" />
       </visual>
@@ -258,19 +258,19 @@
           <mesh filename="package://xarm_description/meshes/xarm6/visual/link6.stl"/>
         </geometry>
-        <origin xyz="-0.20625 0 0.128" rpy="3.1416 0 0"/>
-      </collision>
-      <inertial>
-      <origin
-        xyz="-0.00060579 -0.00056166 -0.0074896"
-        rpy="0 0 0" />
-      <mass
-        value="0.10" />
-      <inertia
-        ixx="5.1386E-05"
-        ixy="-1.7552E-06"
-        ixz="-7.2889E-07"
-        iyy="5.2793E-05"
-        iyz="-4.3242E-07"
-        izz="9.2486E-05" />
+        <origin xyz="0 0 0" rpy="0 0 0"/>
+      </collision>
+      <inertial>
+      <origin
+        xyz="0 0.00064 -0.00952"
+        rpy="0 0 0" />
+      <mass
+        value="0.1096" />
+      <inertia
+        ixx="4.5293E-05"
+        ixy="0"
+        ixz="0"
+        iyy="4.8111E-05"
+        iyz="0"
+        izz="7.9715E-05" />
     </inertial>
     </link>
@@ -278,5 +278,5 @@
       <parent link="${prefix}link5"/>
       <child link="${prefix}link6"/>
-      <origin xyz="0.076 0.0795 0" rpy="-1.5708 0 0"/>
+      <origin xyz="0.076 0.097 0" rpy="-1.5708 0 0"/>
       <axis xyz="0 0 1"/>
       <limit

Commit message: update xarm6 visual

File: xarm_description/urdf/xarm6.urdf.xacro (robot description, xacro)
@@ -21,4 +21,7 @@
       <color rgba="1.0 1.0 1.0 1.0"/>
     </material>
+    <material name="Silver">
+      <color rgba="0.753 0.753 0.753 1.0"/>
+    </material>
     <link name="${prefix}link_base">
       <visual>
@@ -252,5 +255,5 @@
         </geometry>
         <origin xyz="0 0 0" rpy="0 0 0"/>
-        <material name="White" />
+        <material name="Silver" />
       </visual>
       <collision>
