Commit message: add support and example for dual-arm

File: xarm_description/urdf/xarm6.urdf.xacro (robot description, xacro)
@@ -12,14 +12,14 @@
     joint5_lower_limit:=${-1.69297}  joint5_upper_limit:=${pi}
     joint6_lower_limit:=${-2.0*pi}  joint6_upper_limit:=${2.0*pi}">
-    <material name="Black">
+    <material name="${prefix}Black">
       <color rgba="0.0 0.0 0.0 1.0"/>
     </material>
-    <material name="Red">
+    <material name="${prefix}Red">
       <color rgba="0.8 0.0 0.0 1.0"/>
     </material>
-    <material name="White">
+    <material name="${prefix}White">
       <color rgba="1.0 1.0 1.0 1.0"/>
     </material>
-    <material name="Silver">
+    <material name="${prefix}Silver">
       <color rgba="0.753 0.753 0.753 1.0"/>
     </material>
@@ -30,5 +30,5 @@
         </geometry>
         <origin xyz="0 0 0" rpy="0 0 0"/>
-        <material name="White" />
+        <material name="${prefix}White" />
       </visual>
       <collision>
@@ -56,5 +56,5 @@
         </geometry>
         <origin xyz="0 0 0" rpy="0 0 0"/>
-        <material name="White" />
+        <material name="${prefix}White" />
       </visual>
       <collision>
@@ -94,5 +94,5 @@
         </geometry>
         <origin xyz="0 0 0" rpy="0 0 0"/>
-        <material name="White" />
+        <material name="${prefix}White" />
       </visual>
       <collision>
@@ -135,5 +135,5 @@
         </geometry>
         <origin xyz="0 0 0" rpy="0 0 0"/>
-        <material name="White" />
+        <material name="${prefix}White" />
       </visual>
       <collision>
@@ -176,5 +176,5 @@
         </geometry>
         <origin xyz="0 0 0" rpy="0 0 0"/>
-        <material name="White" />
+        <material name="${prefix}White" />
       </visual>
       <collision>
@@ -214,5 +214,5 @@
         </geometry>
         <origin xyz="0 0 0" rpy="0 0 0"/>
-        <material name="White" />
+        <material name="${prefix}White" />
       </visual>
       <collision>
@@ -255,5 +255,5 @@
         </geometry>
         <origin xyz="0 0 0" rpy="0 0 0"/>
-        <material name="Silver" />
+        <material name="${prefix}Silver" />
       </visual>
       <collision>

File: xarm_description/urdf/xarm6_robot_macro.xacro (robot description, xacro)
@@ -15,5 +15,5 @@
       <link name="world" />
     </xacro:if>
-    <joint name="world_joint" type="fixed">
+    <joint name="${prefix}world_joint" type="fixed">
       <parent link="${attach_to}" />
       <child link = "${prefix}link_base" />
