Commit message: add xarm_camera_gazebo demo

File: xarm_description/urdf/xarm5_with_gripper.xacro (robot description, xacro)
@@ -8,4 +8,5 @@
   <!-- To add realsense d435i and gripper, set 'add_realsense_d435i' = true -->
   <xacro:arg name="add_realsense_d435i" default="false"/>
+  <xacro:arg name="use_gazebo_camera" default="false"/>
   <!-- load xarm5 robot -->
   <xacro:include filename="$(find xarm_description)/urdf/xarm5_robot_macro.xacro" />
@@ -14,8 +15,15 @@
   <xacro:xarm5_robot prefix="$(arg prefix)" namespace="$(arg ros_namespace)" limited="$(arg limited)" effort_control="$(arg effort_control)" velocity_control="$(arg velocity_control)" rs_d435i="$(arg add_realsense_d435i)"/>
   <xacro:if value="$(arg add_realsense_d435i)">
-    <xacro:load_gripper attach_to="$(arg prefix)link_eef" xyz="0 0 0.003" effort_control="$(arg effort_control)" velocity_control="$(arg velocity_control)" />
+    <xacro:load_gripper attach_to="$(arg prefix)link_eef" xyz="0 0 0.003" effort_control="$(arg effort_control)" velocity_control="$(arg velocity_control)" robot_dof="5" />
   </xacro:if>
   <xacro:unless value="$(arg add_realsense_d435i)">
-    <xacro:load_gripper attach_to="$(arg prefix)link_eef" effort_control="$(arg effort_control)" velocity_control="$(arg velocity_control)" />
+    <xacro:load_gripper attach_to="$(arg prefix)link_eef" effort_control="$(arg effort_control)" velocity_control="$(arg velocity_control)" robot_dof="5" />
   </xacro:unless>
+  <xacro:if value="$(arg use_gazebo_camera)">
+    <!-- <xacro:include filename="$(find kinect_v2)/urdf/kinect_v2.urdf.xacro" />
+    <xacro:kinect_v2  parent="link_base">
+    </xacro:kinect_v2> -->
+    <xacro:include filename="$(find xarm_description)/urdf/camera.gazebo.xacro" />
+    <xacro:camera_gazebo prefix="${prefix}" />
+  </xacro:if>
 </robot>

File: xarm_description/urdf/xarm7_with_gripper.xacro (robot description, xacro)
@@ -8,4 +8,5 @@
   <!-- To add realsense d435i and gripper, set 'add_realsense_d435i' = true -->
   <xacro:arg name="add_realsense_d435i" default="false"/>
+  <xacro:arg name="use_gazebo_camera" default="false"/>
   <!-- load xarm7 robot -->
   <xacro:include filename="$(find xarm_description)/urdf/xarm7_robot_macro.xacro" />
@@ -14,8 +15,15 @@
   <xacro:xarm7_robot prefix="$(arg prefix)" namespace="$(arg ros_namespace)" limited="$(arg limited)" effort_control="$(arg effort_control)" velocity_control="$(arg velocity_control)" rs_d435i="$(arg add_realsense_d435i)"/>
   <xacro:if value="$(arg add_realsense_d435i)">
-    <xacro:load_gripper attach_to="$(arg prefix)link_eef" xyz="0 0 0.003" effort_control="$(arg effort_control)" velocity_control="$(arg velocity_control)" />
+    <xacro:load_gripper attach_to="$(arg prefix)link_eef" xyz="0 0 0.003" effort_control="$(arg effort_control)" velocity_control="$(arg velocity_control)" robot_dof="7" />
   </xacro:if>
   <xacro:unless value="$(arg add_realsense_d435i)">
-    <xacro:load_gripper attach_to="$(arg prefix)link_eef" effort_control="$(arg effort_control)" velocity_control="$(arg velocity_control)" />
+    <xacro:load_gripper attach_to="$(arg prefix)link_eef" effort_control="$(arg effort_control)" velocity_control="$(arg velocity_control)" robot_dof="7" />
   </xacro:unless>
+  <xacro:if value="$(arg use_gazebo_camera)">
+    <!-- <xacro:include filename="$(find kinect_v2)/urdf/kinect_v2.urdf.xacro" />
+    <xacro:kinect_v2  parent="link_base">
+    </xacro:kinect_v2> -->
+    <xacro:include filename="$(find xarm_description)/urdf/camera.gazebo.xacro" />
+    <xacro:camera_gazebo prefix="${prefix}" />
+  </xacro:if>
 </robot>

File: xarm_gripper/urdf/xarm_gripper_model.xacro (robot description, xacro)
@@ -8,5 +8,5 @@
   <xacro:include filename="$(find xarm_gripper)/urdf/xarm_gripper.transmission.xacro" />
   <xacro:include filename="$(find xarm_gripper)/urdf/xarm_gripper.gazebo.xacro" />
-  <xacro:macro name="load_gripper" params="prefix:='' attach_to:='' ns:='xarm' xyz:='0 0 0' rpy:='0 0 0' effort_control:='false' velocity_control:='false' ">
+  <xacro:macro name="load_gripper" params="prefix:='' attach_to:='' ns:='xarm' xyz:='0 0 0' rpy:='0 0 0' effort_control:='false' velocity_control:='false' robot_dof:=7 ">
     <!-- gazebo plugin -->
     <!-- <xacro:gazebo_ros_control_plugin namespace="${ns}"/> -->
@@ -14,20 +14,21 @@
     <xacro:xarm_gripper_transmission prefix="${prefix}" hard_interface="$(eval 'EffortJointInterface' if ${effort_control} else 'VelocityJointInterface' if ${velocity_control} else 'PositionJointInterface')" />
     <xacro:xarm_gripper_gazebo prefix="${prefix}" />
+    <xacro:xarm_gazebo_grasp_fix prefix="${prefix}" palm_link="${prefix}link${robot_dof}" />
     <!-- mimic_joint_plugin has to be installed: -->
     <xacro:mimic_joint_plugin_gazebo name_prefix="${prefix}left_finger_joint"
-    following_joint="${prefix}drive_joint" mimic_joint="${prefix}left_finger_joint"
-    has_pid="true" multiplier="1.0" max_effort="10.0" />
+      following_joint="${prefix}drive_joint" mimic_joint="${prefix}left_finger_joint"
+      has_pid="false" multiplier="1.0" max_effort="10.0" />
     <xacro:mimic_joint_plugin_gazebo name_prefix="${prefix}left_inner_knuckle_joint"
-    following_joint="${prefix}drive_joint" mimic_joint="${prefix}left_inner_knuckle_joint"
-    has_pid="true" multiplier="1.0" max_effort="10.0" />
+      following_joint="${prefix}drive_joint" mimic_joint="${prefix}left_inner_knuckle_joint"
+      has_pid="false" multiplier="1.0" max_effort="10.0" />
     <xacro:mimic_joint_plugin_gazebo name_prefix="${prefix}right_outer_knuckle_joint"
-    following_joint="${prefix}drive_joint" mimic_joint="${prefix}right_outer_knuckle_joint"
-    has_pid="true" multiplier="1.0" max_effort="10.0" />
+      following_joint="${prefix}drive_joint" mimic_joint="${prefix}right_outer_knuckle_joint"
+      has_pid="false" multiplier="1.0" max_effort="10.0" />
     <xacro:mimic_joint_plugin_gazebo name_prefix="${prefix}right_finger_joint"
-    following_joint="${prefix}drive_joint" mimic_joint="${prefix}right_finger_joint"
-    has_pid="true" multiplier="1.0" max_effort="10.0" />
+      following_joint="${prefix}drive_joint" mimic_joint="${prefix}right_finger_joint"
+      has_pid="false" multiplier="1.0" max_effort="10.0" />
     <xacro:mimic_joint_plugin_gazebo name_prefix="${prefix}right_inner_knuckle_joint"
-    following_joint="${prefix}drive_joint" mimic_joint="${prefix}right_inner_knuckle_joint"
-    has_pid="true" multiplier="1.0" max_effort="10.0" />
+      following_joint="${prefix}drive_joint" mimic_joint="${prefix}right_inner_knuckle_joint"
+      has_pid="false" multiplier="1.0" max_effort="10.0" />
   </xacro:macro>
 </robot>
