Commit message: Modify the collision parameters of urdf Fixed a bug where objects in gazebo did not collide when they touched.

File: xarm_description/urdf/xarm7.urdf.xacro (robot description, xacro)
@@ -60,5 +60,5 @@
           <mesh filename="package://xarm_description/meshes/xarm7/visual/link1.stl"/>
         </geometry>
-        <origin xyz="0 0 0" rpy="0 0 0"/>
+        <origin xyz="0 0 -0.261" rpy="0 0 0"/>
       </collision>
       <inertial>
@@ -91,5 +91,5 @@
           <mesh filename="package://xarm_description/meshes/xarm7/visual/link2.stl"/>
         </geometry>
-        <origin xyz="0 0 -0.260" rpy="0 0 0"/>
+        <origin xyz="0 0 -0.261" rpy="0 0 0"/>
         <material name="White" />
       </visual>
@@ -98,5 +98,5 @@
           <mesh filename="package://xarm_description/meshes/xarm7/visual/link2.stl"/>
         </geometry>
-        <origin xyz="0 0 0" rpy="0 0 0"/>
+        <origin xyz="0 0 -0.261" rpy="0 0 0"/>
       </collision>
       <inertial>
@@ -136,5 +136,5 @@
           <mesh filename="package://xarm_description/meshes/xarm7/visual/link3.stl"/>
         </geometry>
-        <origin xyz="0 0 0" rpy="0 0 0"/>
+        <origin xyz="0 0 -0.546" rpy="0 0 0"/>
       </collision>
       <inertial>
@@ -174,5 +174,5 @@
           <mesh filename="package://xarm_description/meshes/xarm7/visual/link4.stl"/>
         </geometry>
-        <origin xyz="0 0 0" rpy="0 0 0"/>
+        <origin xyz="-0.050 0 -0.546" rpy="0 0 0"/>
       </collision>
       <inertial>
@@ -212,5 +212,5 @@
           <mesh filename="package://xarm_description/meshes/xarm7/visual/link5.stl"/>
         </geometry>
-        <origin xyz="0 0 0" rpy="0 0 0"/>
+        <origin xyz="-0.1285 0 -0.210" rpy="0 0 0"/>
       </collision>
       <inertial>
@@ -250,5 +250,5 @@
           <mesh filename="package://xarm_description/meshes/xarm7/visual/link6.stl"/>
         </geometry>
-        <origin xyz="0 0 0" rpy="0 0 0"/>
+        <origin xyz="-0.1285 0 -0.210" rpy="0 0 0"/>
       </collision>
       <inertial>
@@ -288,5 +288,5 @@
           <mesh filename="package://xarm_description/meshes/xarm7/visual/link7.stl"/>
         </geometry>
-        <origin xyz="0 0 0" rpy="0 0 0"/>
+        <origin xyz="-0.2015 0 -0.1405" rpy="0 0 0"/>
       </collision>
       <inertial>

Commit message: v0.1.0

File: xarm_description/urdf/xarm7.urdf.xacro (robot description, xacro)
@@ -230,5 +230,5 @@
       <child link="${prefix}link5"/>
       <origin xyz="0.0785 0 -0.336" rpy="0 0 0"/>
-      <axis xyz="0 0 1"/>
+      <axis xyz="0 0 -1"/>
       <limit
         lower="${joint5_lower_limit}"
@@ -306,5 +306,5 @@
       <child link="${prefix}link7"/>
       <origin xyz="0.073 0 -0.0695" rpy="0 0 0"/>
-      <axis xyz="0 0 1"/>
+      <axis xyz="0 0 -1"/>
       <limit
         lower="${joint7_lower_limit}"

File: xarm_description/urdf/xarm7_robot.urdf.xacro (robot description, xacro)
@@ -17,9 +17,9 @@
     <xacro:xarm7_urdf prefix="$(arg prefix)"
       joint1_lower_limit="${-pi*0.99}" joint1_upper_limit="${pi*0.99}"
-      joint2_lower_limit="${-pi*0.99}" joint2_upper_limit="${pi*0.99}"
+      joint2_lower_limit="${-2.18}" joint2_upper_limit="${2.18}"
       joint3_lower_limit="${-pi*0.99}" joint3_upper_limit="${pi*0.99}"
-      joint4_lower_limit="${-pi*0.99}" joint4_upper_limit="${pi*0.99}"
+      joint4_lower_limit="${-pi*0.99}" joint4_upper_limit="${0.11}"
       joint5_lower_limit="${-pi*0.99}" joint5_upper_limit="${pi*0.99}"
-      joint6_lower_limit="${-pi*0.99}" joint6_upper_limit="${pi*0.99}"
+      joint6_lower_limit="${-1.75}" joint6_upper_limit="${pi*0.99}"
       joint7_lower_limit="${-pi*0.99}" joint7_upper_limit="${pi*0.99}"/>
   </xacro:if>

Commit message: update ReadMe for online planning mode and urdf for xArm7

File: xarm_description/urdf/xarm7.urdf.xacro (robot description, xacro)
@@ -33,5 +33,5 @@
         rpy="0 0 0" />
       <mass
-        value="0.88556" />
+        value="2.612" />
       <inertia
         ixx="0.0030595"
@@ -66,15 +66,15 @@
     <inertial>
       <origin
-        xyz="-0.0042142 0.02821 -0.0087788"
-        rpy="0 0 0" />
-      <mass
-        value="0.42603" />
-      <inertia
-        ixx="0.0014243"
-        ixy="3.9946E-05"
-        ixz="4.7078E-06"
-        iyy="0.00123"
-        iyz="-0.00026073"
-        izz="0.00099229" />
+        xyz="0.00013 0.0301 -0.012"
+        rpy="0 0 0" />
+      <mass
+        value="2.459" />
+      <inertia
+        ixx="0.005795"
+        ixy="-1.078E-05"
+        ixz="-2.63E-05"
+        iyy="0.004969"
+        iyz="0.000911"
+        izz="0.003428" />
     </inertial>
     <visual>
@@ -123,15 +123,15 @@
     <inertial>
       <origin
-        xyz="-3.3178E-05 -0.12849 0.026337"
-        rpy="0 0 0" />
-      <mass
-        value="0.56095" />
-      <inertia
-        ixx="0.0031915"
-        ixy="3.0892E-06"
-        ixz="2.8729E-06"
-        iyy="0.0017468"
-        iyz="-0.0010241"
-        izz="0.00235" />
+        xyz="0.0002 -0.12964 0.01692"
+        rpy="0 0 0" />
+      <mass
+        value="1.916" />
+      <inertia
+        ixx="0.0097184"
+        ixy="1.0E-06"
+        ixz="-4.83E-06"
+        iyy="0.0038705"
+        iyz="0.0032"
+        izz="0.007672" />
     </inertial>
     <visual>
@@ -180,15 +180,15 @@
     <inertial>
       <origin
-        xyz="0.04223 -0.023258 -0.0096674"
-        rpy="0 0 0" />
-      <mass
-        value="0.44463" />
-      <inertia
-        ixx="0.0011454"
-        ixy="0.0001654"
-        ixz="-0.0001951"
-        iyy="0.0010503"
-        iyz="0.00012027"
-        izz="0.0011083" />
+        xyz="0.04676 -0.02526 -0.00746"
+        rpy="0 0 0" />
+      <mass
+        value="1.6854" />
+      <inertia
+        ixx="0.0031588"
+        ixy="-3.1443E-04"
+        ixz="5.8658E-04"
+        iyy="0.002682"
+        iyz="-3.469E-04"
+        izz="0.0027105" />
     </inertial>
     <visual>
@@ -237,15 +237,15 @@
     <inertial>
       <origin
-        xyz="0.067148 -0.10732 0.024479"
-        rpy="0 0 0" />
-      <mass
-        value="0.52387" />
-      <inertia
-        ixx="0.0026033"
-        ixy="0.00053379"
-        ixz="0.00036314"
-        iyy="0.0017649"
-        iyz="-0.00083253"
-        izz="0.0022431" />
+        xyz="0.07066 -0.11664 0.0117"
+        rpy="0 0 0" />
+      <mass
+        value="1.774" />
+      <inertia
+        ixx="0.005967"
+        ixy="-0.001382"
+        ixz="-0.00088544"
+        iyy="0.00363897"
+        iyz="0.0017806"
+        izz="0.005509226" />
     </inertial>
     <visual>
@@ -294,15 +294,15 @@
     <inertial>
       <origin
-        xyz="-0.00023397 0.036705 -0.080064"
-        rpy="0 0 0" />
-      <mass
-        value="0.18554" />
-      <inertia
-        ixx="0.00099549"
-        ixy="8.9957E-07"
-        ixz="8.5285E-07"
-        iyy="0.0008853"
-        iyz="-0.00025682"
-        izz="0.00035048" />
+        xyz="-0.00031 0.01558 -0.0253"
+        rpy="0 0 0" />
+      <mass
+        value="1.357" />
+      <inertia
+        ixx="0.005396"
+        ixy="-1.53E-05"
+        ixz="-6.7E-07"
+        iyy="0.005"
+        iyz="0.00020544"
+        izz="0.00138734" />
     </inertial>
     <visual>
@@ -351,15 +351,15 @@
     <inertial>
       <origin
-        xyz="0.058911 0.028469 0.0068428"
-        rpy="0 0 0" />
-      <mass
-        value="0.31344" />
-      <inertia
-        ixx="0.00052034"
-        ixy="-0.00014989"
-        ixz="0.00011658"
-        iyy="0.00067968"
-        iyz="6.116E-05"
-        izz="0.00078345" />
+        xyz="0.065 0.03336 0.02131"
+        rpy="0 0 0" />
+      <mass
+        value="1.362" />
+      <inertia
+        ixx="0.0015057"
+        ixy="0.000496735"
+        ixz="-2.9968E-04"
+        iyy="0.0019297"
+        iyz="-1.5E-04"
+        izz="0.0024" />
     </inertial>
     <visual>
@@ -408,15 +408,15 @@
     <inertial>
       <origin
-        xyz="-1.5846E-05 -0.0046377 -0.012705"
-        rpy="0 0 0" />
-      <mass
-        value="0.31468" />
-      <inertia
-        ixx="0.00016985"
-        ixy="1.1102E-07"
-        ixz="5.1075E-08"
-        iyy="0.00011924"
-        iyz="-2.1251E-06"
-        izz="0.00026032" />
+        xyz="0 -0.00677 -0.01098"
+        rpy="0 0 0" />
+      <mass
+        value="0.17" />
+      <inertia
+        ixx="9.3E-05"
+        ixy="0.0"
+        ixz="0.0"
+        iyy="5.87E-05"
+        iyz="3.6E-06"
+        izz="1.32E-04" />
     </inertial>
     <visual>
