Commit message: [feat] add launch parameter `model1300` to replace the end model
1. add launch parameter `model1300` to replace the model of the end of xarm robot arm with the 1300 series

File: xarm_description/urdf/dual_xarm6_robot.urdf.xacro (robot description, xacro)
@@ -8,4 +8,6 @@
   <xacro:arg name="velocity_control" default="false"/>
   <xacro:arg name="add_gripper" default="false"/>
+  <xacro:arg name="add_realsense_d435i" default="false"/>
+  <xacro:arg name="model1300" default="false"/>
   <xacro:include filename="$(find xarm_description)/urdf/xarm6_robot_macro.xacro" />
   <xacro:include filename="$(find xarm_gripper)/urdf/xarm_gripper_model.xacro" />
@@ -13,10 +15,10 @@
   <link name="ground" />
   <!-- launch left arm -->
-  <xacro:xarm6_robot prefix="$(arg prefix_1)" namespace="$(arg ros_namespace)" limited="$(arg limited)" attach_to="ground" xyz="0 0 0" rpy="0 0 0" effort_control="$(arg effort_control)" velocity_control="$(arg velocity_control)"/>
+  <xacro:xarm6_robot prefix="$(arg prefix_1)" namespace="$(arg ros_namespace)" limited="$(arg limited)" attach_to="ground" xyz="0 0 0" rpy="0 0 0" effort_control="$(arg effort_control)" velocity_control="$(arg velocity_control)" model1300="$(arg model1300)" />
   <xacro:if value="$(arg add_gripper)">
     <xacro:load_gripper attach_to="$(arg prefix_1)link6" effort_control="$(arg effort_control)" velocity_control="$(arg velocity_control)" />
   </xacro:if>
   <!-- launch right arm -->
-  <xacro:xarm6_robot prefix="$(arg prefix_2)" namespace="$(arg ros_namespace)" limited="$(arg limited)" attach_to="ground" xyz="0 1 0" rpy="0 0 0" effort_control="$(arg effort_control)" velocity_control="$(arg velocity_control)"/>
+  <xacro:xarm6_robot prefix="$(arg prefix_2)" namespace="$(arg ros_namespace)" limited="$(arg limited)" attach_to="ground" xyz="0 1 0" rpy="0 0 0" effort_control="$(arg effort_control)" velocity_control="$(arg velocity_control)" model1300="$(arg model1300)" />
   <xacro:if value="$(arg add_gripper)">
     <xacro:load_gripper attach_to="$(arg prefix_2)link6" effort_control="$(arg effort_control)" velocity_control="$(arg velocity_control)" />

File: xarm_description/urdf/lite6_robot.urdf.xacro (robot description, xacro)
@@ -21,4 +21,5 @@
   <xacro:arg name="geometry_mesh_tcp_rpy" default="0 0 0"/>
   <xacro:arg name="add_realsense_d435i" default="false"/>
+  <xacro:arg name="model1300" default="false"/>
   <!-- load lite6 robot -->
   <xacro:include filename="$(find xarm_description)/urdf/lite6_robot_macro.xacro" />

File: xarm_description/urdf/xarm5.urdf.xacro (robot description, xacro)
@@ -11,5 +11,5 @@
     joint4_lower_limit:=${-1.69297}  joint4_upper_limit:=${pi}
     joint5_lower_limit:=${-2.0*pi}  joint5_upper_limit:=${2.0*pi}
-    rs_d435i:=false">
+    rs_d435i:=false  model1300:=false">
     <material name="Black">
       <color rgba="0.0 0.0 0.0 1.0"/>
@@ -309,6 +309,10 @@
           rpy="0 0 0" />
         <geometry>
-          <mesh
-            filename="package://xarm_description/meshes/xarm5/visual/link5.STL" />
+          <xacro:if value="${model1300}">
+            <mesh filename="package://xarm_description/meshes/end_tool/visual/end_tool_1300.STL" />
+          </xacro:if>
+          <xacro:unless value="${model1300}">
+            <mesh filename="package://xarm_description/meshes/xarm5/visual/link5.STL" />
+          </xacro:unless>
         </geometry>
         <material name="Silver" />
@@ -319,6 +323,10 @@
           rpy="0 0 0" />
         <geometry>
-          <mesh
-            filename="package://xarm_description/meshes/collision/end_tool.STL" />
+          <xacro:if value="${model1300}">
+            <mesh filename="package://xarm_description/meshes/end_tool/collision/end_tool_1300.STL" />
+          </xacro:if>
+          <xacro:unless value="${model1300}">
+            <mesh filename="package://xarm_description/meshes/end_tool/collision/end_tool.STL" />
+          </xacro:unless>
         </geometry>
       </collision>

File: xarm_description/urdf/xarm5_robot.urdf.xacro (robot description, xacro)
@@ -19,4 +19,5 @@
   <xacro:arg name="geometry_mesh_tcp_rpy" default="0 0 0"/>
   <xacro:arg name="add_realsense_d435i" default="false"/>
+  <xacro:arg name="model1300" default="false"/>
   <!-- load xarm5 robot -->
   <xacro:include filename="$(find xarm_description)/urdf/xarm5_robot_macro.xacro" />
@@ -24,4 +25,5 @@
     effort_control="$(arg effort_control)" velocity_control="$(arg velocity_control)"
     rs_d435i="$(arg add_realsense_d435i)"
+    model1300="$(arg model1300)"
     add_other_geometry="$(arg add_other_geometry)"
     geometry_type="$(arg geometry_type)" geometry_mass="$(arg geometry_mass)"

File: xarm_description/urdf/xarm5_robot_macro.xacro (robot description, xacro)
@@ -3,4 +3,5 @@
   <xacro:macro name="xarm5_robot" params="prefix:='' namespace:='xarm' limited:='false' effort_control:='false'
     velocity_control:='false' attach_to:='world' xyz:='0 0 0' rpy:='0 0 0' load_gazebo_plugin:='true' rs_d435i:='false'
+    model1300:='false'
     add_other_geometry:='false'
     geometry_type:='box' geometry_mass:='0.1'
@@ -37,8 +38,8 @@
         joint4_lower_limit="${-1.69297}" joint4_upper_limit="${pi*0.99}"
         joint5_lower_limit="${-pi*0.99}" joint5_upper_limit="${pi*0.99}"
-        rs_d435i="${rs_d435i}"/>
+        rs_d435i="${rs_d435i}" model1300="${model1300}"/>
     </xacro:if>
     <xacro:unless value="${limited}">
-      <xacro:xarm5_urdf prefix="${prefix}" rs_d435i="${rs_d435i}"/>
+      <xacro:xarm5_urdf prefix="${prefix}" rs_d435i="${rs_d435i}" model1300="${model1300}"/>
     </xacro:unless>
     <xacro:xarm5_transmission prefix="${prefix}" hard_interface="$(eval 'EffortJointInterface' if ${effort_control} else 'VelocityJointInterface' if ${velocity_control} else 'PositionJointInterface')" />

File: xarm_description/urdf/xarm5_with_gripper.xacro (robot description, xacro)
@@ -9,9 +9,10 @@
   <xacro:arg name="add_realsense_d435i" default="false"/>
   <xacro:arg name="use_gazebo_camera" default="false"/>
+  <xacro:arg name="model1300" default="false"/>
   <!-- load xarm5 robot -->
   <xacro:include filename="$(find xarm_description)/urdf/xarm5_robot_macro.xacro" />
   <!-- Attach gripper -->
   <xacro:include filename="$(find xarm_gripper)/urdf/xarm_gripper_model.xacro" />
-  <xacro:xarm5_robot prefix="$(arg prefix)" namespace="$(arg ros_namespace)" limited="$(arg limited)" effort_control="$(arg effort_control)" velocity_control="$(arg velocity_control)" rs_d435i="$(arg add_realsense_d435i)"/>
+  <xacro:xarm5_robot prefix="$(arg prefix)" namespace="$(arg ros_namespace)" limited="$(arg limited)" effort_control="$(arg effort_control)" velocity_control="$(arg velocity_control)" rs_d435i="$(arg add_realsense_d435i)" model1300="$(arg model1300)"/>
   <xacro:if value="$(arg add_realsense_d435i)">
     <xacro:load_gripper attach_to="$(arg prefix)link_eef" xyz="0 0 0.003" effort_control="$(arg effort_control)" velocity_control="$(arg velocity_control)" robot_dof="5" />

File: xarm_description/urdf/xarm5_with_vacuum_gripper.xacro (robot description, xacro)
@@ -8,9 +8,10 @@
   <!-- To add realsense d435i and vacuum gripper, set 'add_realsense_d435i' = true -->
   <xacro:arg name="add_realsense_d435i" default="false"/>
+  <xacro:arg name="model1300" default="false"/>
   <!-- load xarm5 robot -->
   <xacro:include filename="$(find xarm_description)/urdf/xarm5_robot_macro.xacro" />
   <!-- Attach gripper -->
   <xacro:include filename="$(find xarm_description)/urdf/xarm_vacuum_gripper.urdf.xacro" />
-  <xacro:xarm5_robot prefix="$(arg prefix)" namespace="$(arg ros_namespace)" limited="$(arg limited)" effort_control="$(arg effort_control)" velocity_control="$(arg velocity_control)" rs_d435i="$(arg add_realsense_d435i)" />
+  <xacro:xarm5_robot prefix="$(arg prefix)" namespace="$(arg ros_namespace)" limited="$(arg limited)" effort_control="$(arg effort_control)" velocity_control="$(arg velocity_control)" rs_d435i="$(arg add_realsense_d435i)" model1300="$(arg model1300)" />
   <xacro:if value="$(arg add_realsense_d435i)">
     <xacro:xarm_vacuum_gripper_urdf attach_to="$(arg prefix)link_eef" xyz="0 0 0.003" effort_control="$(arg effort_control)" velocity_control="$(arg velocity_control)" />

File: xarm_description/urdf/xarm6.urdf.xacro (robot description, xacro)
@@ -12,5 +12,5 @@
     joint5_lower_limit:=${-1.69297}  joint5_upper_limit:=${pi}
     joint6_lower_limit:=${-2.0*pi}  joint6_upper_limit:=${2.0*pi}
-    rs_d435i:=false">
+    rs_d435i:=false  model1300:=false">
     <material name="${prefix}Black">
       <color rgba="0.0 0.0 0.0 1.0"/>
@@ -253,5 +253,10 @@
       <visual>
         <geometry>
-          <mesh filename="package://xarm_description/meshes/xarm6/visual/link6.stl"/>
+          <xacro:if value="${model1300}">
+            <mesh filename="package://xarm_description/meshes/end_tool/visual/end_tool_1300.STL" />
+          </xacro:if>
+          <xacro:unless value="${model1300}">
+            <mesh filename="package://xarm_description/meshes/xarm6/visual/link6.stl"/>
+          </xacro:unless>
         </geometry>
         <origin xyz="0 0 0" rpy="0 0 0"/>
@@ -260,5 +265,10 @@
       <collision>
         <geometry>
-          <mesh filename="package://xarm_description/meshes/collision/end_tool.STL"/>
+          <xacro:if value="${model1300}">
+            <mesh filename="package://xarm_description/meshes/end_tool/collision/end_tool_1300.STL" />
+          </xacro:if>
+          <xacro:unless value="${model1300}">
+            <mesh filename="package://xarm_description/meshes/end_tool/collision/end_tool.STL"/>
+          </xacro:unless>
         </geometry>
         <origin xyz="0 0 0" rpy="0 0 0"/>

File: xarm_description/urdf/xarm6_robot.urdf.xacro (robot description, xacro)
@@ -19,4 +19,5 @@
   <xacro:arg name="geometry_mesh_tcp_rpy" default="0 0 0"/>
   <xacro:arg name="add_realsense_d435i" default="false"/>
+  <xacro:arg name="model1300" default="false"/>
   <!-- load xarm6 robot -->
   <xacro:include filename="$(find xarm_description)/urdf/xarm6_robot_macro.xacro" />
@@ -24,4 +25,5 @@
     effort_control="$(arg effort_control)" velocity_control="$(arg velocity_control)"
     rs_d435i="$(arg add_realsense_d435i)"
+    model1300="$(arg model1300)"
     add_other_geometry="$(arg add_other_geometry)"
     geometry_type="$(arg geometry_type)" geometry_mass="$(arg geometry_mass)"

File: xarm_description/urdf/xarm6_robot_macro.xacro (robot description, xacro)
@@ -3,4 +3,5 @@
   <xacro:macro name="xarm6_robot" params="prefix:='' namespace:='xarm' limited:='false' effort_control:='false'
     velocity_control:='false' attach_to:='world' xyz:='0 0 0' rpy:='0 0 0' load_gazebo_plugin:='true' rs_d435i:='false'
+    model1300:='false'
     add_other_geometry:='false'
     geometry_type:='box' geometry_mass:='0.1'
@@ -38,8 +39,8 @@
         joint5_lower_limit="${-1.69297}" joint5_upper_limit="${pi*0.99}"
         joint6_lower_limit="${-pi*0.99}" joint6_upper_limit="${pi*0.99}"
-        rs_d435i="${rs_d435i}"/>
+        rs_d435i="${rs_d435i}" model1300="${model1300}"/>
     </xacro:if>
     <xacro:unless value="${limited}">
-      <xacro:xarm6_urdf prefix="${prefix}" rs_d435i="${rs_d435i}"/>
+      <xacro:xarm6_urdf prefix="${prefix}" rs_d435i="${rs_d435i}" model1300="${model1300}"/>
     </xacro:unless>
     <xacro:xarm6_transmission prefix="${prefix}" hard_interface="$(eval 'EffortJointInterface' if ${effort_control} else 'VelocityJointInterface' if ${velocity_control} else 'PositionJointInterface')" />

File: xarm_description/urdf/xarm6_with_gripper.xacro (robot description, xacro)
@@ -9,9 +9,10 @@
   <xacro:arg name="add_realsense_d435i" default="false"/>
   <xacro:arg name="use_gazebo_camera" default="false"/>
+  <xacro:arg name="model1300" default="false"/>
   <!-- load xarm6 robot -->
   <xacro:include filename="$(find xarm_description)/urdf/xarm6_robot_macro.xacro" />
   <!-- Attach gripper -->
   <xacro:include filename="$(find xarm_gripper)/urdf/xarm_gripper_model.xacro" />
-  <xacro:xarm6_robot prefix="$(arg prefix)" namespace="$(arg ros_namespace)" limited="$(arg limited)" effort_control="$(arg effort_control)" velocity_control="$(arg velocity_control)" rs_d435i="$(arg add_realsense_d435i)"/>
+  <xacro:xarm6_robot prefix="$(arg prefix)" namespace="$(arg ros_namespace)" limited="$(arg limited)" effort_control="$(arg effort_control)" velocity_control="$(arg velocity_control)" rs_d435i="$(arg add_realsense_d435i)" model1300="$(arg model1300)"/>
   <xacro:if value="$(arg add_realsense_d435i)">
     <xacro:load_gripper attach_to="$(arg prefix)link_eef" xyz="0 0 0.003" effort_control="$(arg effort_control)" velocity_control="$(arg velocity_control)" robot_dof="6" />

File: xarm_description/urdf/xarm6_with_vacuum_gripper.xacro (robot description, xacro)
@@ -8,4 +8,5 @@
   <!-- To add realsense d435i and vacuum gripper, set 'add_realsense_d435i' = true -->
   <xacro:arg name="add_realsense_d435i" default="false"/>
+  <xacro:arg name="model1300" default="false"/>
   <!-- load xarm6 robot -->
   <xacro:include filename="$(find xarm_description)/urdf/xarm6_robot_macro.xacro" />
@@ -13,5 +14,5 @@
   <xacro:include filename="$(find xarm_description)/urdf/xarm_vacuum_gripper.urdf.xacro" />
   <!-- <xacro:load_gripper attach_to="$(arg prefix)link6" /> -->
-  <xacro:xarm6_robot prefix="$(arg prefix)" namespace="$(arg ros_namespace)" limited="$(arg limited)" effort_control="$(arg effort_control)" velocity_control="$(arg velocity_control)" rs_d435i="$(arg add_realsense_d435i)" />
+  <xacro:xarm6_robot prefix="$(arg prefix)" namespace="$(arg ros_namespace)" limited="$(arg limited)" effort_control="$(arg effort_control)" velocity_control="$(arg velocity_control)" rs_d435i="$(arg add_realsense_d435i)" model1300="$(arg model1300)" />
   <xacro:if value="$(arg add_realsense_d435i)">
     <xacro:xarm_vacuum_gripper_urdf attach_to="$(arg prefix)link_eef" xyz="0 0 0.003" effort_control="$(arg effort_control)" velocity_control="$(arg velocity_control)" />

File: xarm_description/urdf/xarm7.urdf.xacro (robot description, xacro)
@@ -13,5 +13,5 @@
     joint6_lower_limit:=${-1.69297}  joint6_upper_limit:=${pi}
     joint7_lower_limit:=${-2.0*pi}  joint7_upper_limit:=${2.0*pi}
-    rs_d435i:=false">
+    rs_d435i:=false  model1300:=false">
     <material name="Black">
       <color rgba="0.0 0.0 0.0 1.0"/>
@@ -425,6 +425,10 @@
         rpy="0 0 0" />
       <geometry>
-        <mesh
-          filename="package://xarm_description/meshes/xarm7/visual/link7.STL" />
+        <xacro:if value="${model1300}">
+          <mesh filename="package://xarm_description/meshes/end_tool/visual/end_tool_1300.STL" />
+        </xacro:if>
+        <xacro:unless value="${model1300}">
+          <mesh filename="package://xarm_description/meshes/xarm7/visual/link7.STL" />
+        </xacro:unless>
       </geometry>
       <material name="Silver" />
@@ -435,6 +439,10 @@
         rpy="0 0 0" />
       <geometry>
-        <mesh
-          filename="package://xarm_description/meshes/collision/end_tool.STL" />
+        <xacro:if value="${model1300}">
+          <mesh filename="package://xarm_description/meshes/end_tool/collision/end_tool_1300.STL" />
+        </xacro:if>
+        <xacro:unless value="${model1300}">
+          <mesh filename="package://xarm_description/meshes/end_tool/collision/end_tool.STL" />
+        </xacro:unless>
       </geometry>
     </collision>

File: xarm_description/urdf/xarm7_robot.urdf.xacro (robot description, xacro)
@@ -19,4 +19,5 @@
   <xacro:arg name="geometry_mesh_tcp_rpy" default="0 0 0"/>
   <xacro:arg name="add_realsense_d435i" default="false"/>
+  <xacro:arg name="model1300" default="false"/>
   <!-- load xarm7 robot -->
   <xacro:include filename="$(find xarm_description)/urdf/xarm7_robot_macro.xacro" />
@@ -24,4 +25,5 @@
     effort_control="$(arg effort_control)" velocity_control="$(arg velocity_control)"
     rs_d435i="$(arg add_realsense_d435i)"
+    model1300="$(arg model1300)"
     add_other_geometry="$(arg add_other_geometry)"
     geometry_type="$(arg geometry_type)" geometry_mass="$(arg geometry_mass)"

File: xarm_description/urdf/xarm7_robot_macro.xacro (robot description, xacro)
@@ -3,4 +3,5 @@
   <xacro:macro name="xarm7_robot" params="prefix:='' namespace:='xarm' limited:='false' effort_control:='false'
     velocity_control:='false' attach_to:='world' xyz:='0 0 0' rpy:='0 0 0' load_gazebo_plugin:='true' rs_d435i:='false'
+    model1300:='false'
     add_other_geometry:='false'
     geometry_type:='box' geometry_mass:='0.1'
@@ -39,8 +40,8 @@
         joint6_lower_limit="${-1.75}" joint6_upper_limit="${pi*0.99}"
         joint7_lower_limit="${-pi*0.99}" joint7_upper_limit="${pi*0.99}"
-        rs_d435i="${rs_d435i}"/>
+        rs_d435i="${rs_d435i}" model1300="${model1300}"/>
     </xacro:if>
     <xacro:unless value="${limited}">
-      <xacro:xarm7_urdf prefix="${prefix}" rs_d435i="${rs_d435i}"/>
+      <xacro:xarm7_urdf prefix="${prefix}" rs_d435i="${rs_d435i}" model1300="${model1300}"/>
     </xacro:unless>
     <xacro:xarm7_transmission prefix="${prefix}" hard_interface="$(eval 'EffortJointInterface' if ${effort_control} else 'VelocityJointInterface' if ${velocity_control} else 'PositionJointInterface')" />

File: xarm_description/urdf/xarm7_with_gripper.xacro (robot description, xacro)
@@ -9,9 +9,10 @@
   <xacro:arg name="add_realsense_d435i" default="false"/>
   <xacro:arg name="use_gazebo_camera" default="false"/>
+  <xacro:arg name="model1300" default="false"/>
   <!-- load xarm7 robot -->
   <xacro:include filename="$(find xarm_description)/urdf/xarm7_robot_macro.xacro" />
   <!-- Attach gripper -->
   <xacro:include filename="$(find xarm_gripper)/urdf/xarm_gripper_model.xacro" />
-  <xacro:xarm7_robot prefix="$(arg prefix)" namespace="$(arg ros_namespace)" limited="$(arg limited)" effort_control="$(arg effort_control)" velocity_control="$(arg velocity_control)" rs_d435i="$(arg add_realsense_d435i)"/>
+  <xacro:xarm7_robot prefix="$(arg prefix)" namespace="$(arg ros_namespace)" limited="$(arg limited)" effort_control="$(arg effort_control)" velocity_control="$(arg velocity_control)" rs_d435i="$(arg add_realsense_d435i)" model1300="$(arg model1300)"/>
   <xacro:if value="$(arg add_realsense_d435i)">
     <xacro:load_gripper attach_to="$(arg prefix)link_eef" xyz="0 0 0.003" effort_control="$(arg effort_control)" velocity_control="$(arg velocity_control)" robot_dof="7" />

File: xarm_description/urdf/xarm7_with_vacuum_gripper.xacro (robot description, xacro)
@@ -8,9 +8,10 @@
   <!-- To add realsense d435i and vacuum gripper, set 'add_realsense_d435i' = true -->
   <xacro:arg name="add_realsense_d435i" default="false"/>
+  <xacro:arg name="model1300" default="false"/>
   <!-- load xarm7 robot -->
   <xacro:include filename="$(find xarm_description)/urdf/xarm7_robot_macro.xacro" />
   <!-- Attach gripper -->
   <xacro:include filename="$(find xarm_description)/urdf/xarm_vacuum_gripper.urdf.xacro" />
-  <xacro:xarm7_robot prefix="$(arg prefix)" namespace="$(arg ros_namespace)" limited="$(arg limited)" effort_control="$(arg effort_control)" velocity_control="$(arg velocity_control)" rs_d435i="$(arg add_realsense_d435i)"/>
+  <xacro:xarm7_robot prefix="$(arg prefix)" namespace="$(arg ros_namespace)" limited="$(arg limited)" effort_control="$(arg effort_control)" velocity_control="$(arg velocity_control)" rs_d435i="$(arg add_realsense_d435i)" rs_d435i="$(arg model1300)"/>
   <xacro:if value="$(arg add_realsense_d435i)">
     <xacro:xarm_vacuum_gripper_urdf attach_to="$(arg prefix)link_eef" xyz="0 0 0.003" effort_control="$(arg effort_control)" velocity_control="$(arg velocity_control)" />
