Commit message: [fix] fix _private_macro.xacro

File: xarm_description/urdf/_private_macro.xacro (robot description, xacro)
@@ -2,6 +2,6 @@
 <robot xmlns:xacro="http://ros.org/wiki/xacro" name="private_macro">
   <xacro:property name="is_ros2" value="false" scope="parent"/>
-  <xacro:property name="use_xacro_load_yaml" value="false" scope="parent"/>
-  <xacro:property name="use_len" value="false" scope="parent"/>
+  <xacro:property name="use_xacro_load_yaml" value="true" scope="parent"/>
+  <xacro:property name="use_len" value="true" scope="parent"/>
   <xacro:macro name="device_macro_begin" params="">
     <!-- Insert at the beginning of xarm_device_macro.xacro -->

Commit message: [fix] (kinetic) fix _private_macro.xacro

File: xarm_description/urdf/_private_macro.xacro (robot description, xacro)
@@ -2,6 +2,6 @@
 <robot xmlns:xacro="http://ros.org/wiki/xacro" name="private_macro">
   <xacro:property name="is_ros2" value="false" scope="parent"/>
-  <xacro:property name="use_xacro_load_yaml" value="true" scope="parent"/>
-  <xacro:property name="use_len" value="true" scope="parent"/>
+  <xacro:property name="use_xacro_load_yaml" value="false" scope="parent"/>
+  <xacro:property name="use_len" value="false" scope="parent"/>
   <xacro:macro name="device_macro_begin" params="">
     <!-- Insert at the beginning of xarm_device_macro.xacro -->

Commit message: [fix] (urdf) default use `load_yaml()`, not `xacro.load_yaml()`
1. use `load_yaml`, `noetic` logger warnning
2. use `xacro.load_yaml`, `melodic` raise exception

File: xarm_description/urdf/_private_macro.xacro (robot description, xacro)
@@ -2,5 +2,5 @@
 <robot xmlns:xacro="http://ros.org/wiki/xacro" name="private_macro">
   <xacro:property name="is_ros2" value="false" scope="parent"/>
-  <xacro:property name="use_xacro_load_yaml" value="true" scope="parent"/>
+  <xacro:property name="use_xacro_load_yaml" value="false" scope="parent"/>
   <xacro:property name="use_len" value="true" scope="parent"/>
   <xacro:macro name="device_macro_begin" params="">
