Commit message: [fix] fix xarm_description
1. fix xarm5_1305 link5 model
2. fix urdf for gripper g2

File: xarm_description/urdf/dual_xarm_device.urdf.xacro (robot description, xacro)
@@ -25,4 +25,8 @@
   <xacro:arg name="report_type_1" default="normal"/>
   <xacro:arg name="report_type_2" default="normal"/>
+  <xacro:arg name="attach_xyz_1" default="0 0 0"/>
+  <xacro:arg name="attach_rpy_1" default="0 0 0"/>
+  <xacro:arg name="attach_xyz_2" default="0 1 0"/>
+  <xacro:arg name="attach_rpy_2" default="0 0 0"/>
   <xacro:arg name="ros2_control_plugin" default="uf_robot_hardware/UFRobotSystemHardware"/>
   <xacro:arg name="ros2_control_params" default=""/>
@@ -72,5 +76,5 @@
     ros2_control_plugin="$(arg ros2_control_plugin)" robot_type="$(arg robot_type_1)"
     load_gazebo_plugin="false" ros2_control_params="$(arg ros2_control_params)"
-    attach_to="world" attach_xyz="0 0 0" attach_rpy="0 0 0"
+    attach_to="world" attach_xyz="$(arg attach_xyz_1)" attach_rpy="$(arg attach_rpy_1)"
     add_realsense_d435i="$(arg add_realsense_d435i_1)"
     add_d435i_links="$(arg add_d435i_links_1)"
@@ -91,5 +95,5 @@
     ros2_control_plugin="$(arg ros2_control_plugin)" robot_type="$(arg robot_type_2)"
     load_gazebo_plugin="true" ros2_control_params="$(arg ros2_control_params)"
-    attach_to="world" attach_xyz="0 1 0" attach_rpy="0 0 0" create_attach_link="false"
+    attach_to="world" attach_xyz="$(arg attach_xyz_2)" attach_rpy="$(arg attach_rpy_2)" create_attach_link="false"
     add_realsense_d435i="$(arg add_realsense_d435i_2)"
     add_d435i_links="$(arg add_d435i_links_2)"

File: xarm_description/urdf/gripper/bio_gripper.urdf.xacro (robot description, xacro)
@@ -2,9 +2,11 @@
 <robot xmlns:xacro="http://ros.org/wiki/xacro" name="uf_bio_gripper">
   <xacro:macro name="bio_gripper_urdf" params="prefix:='' attach_to:='' attach_xyz:='0 0 0' attach_rpy:='0 0 0' gripper_version:='G1' ">
+    <xacro:property name="add_mesh_suffix" value="true"/>
+    <xacro:property name="other_mesh_suffix" value=""/>
     <xacro:property name="name_suffix" value=""/>
-    <xacro:if value="${mesh_suffix == 'dae'}">
-      <xacro:if value="${gripper_version == 'G2' or gripper_version == 'g2'}">
-        <xacro:property name="name_suffix" value="_g2"/>
-      </xacro:if>
+    <xacro:if value="${gripper_version == 'G2' or gripper_version == 'g2'}">
+      <xacro:property name="name_suffix" value="_g2"/>
+      <xacro:property name="other_mesh_suffix" value="dae"/>
+      <xacro:property name="add_mesh_suffix" value="false"/>
     </xacro:if>
     <xacro:unless value="${attach_to == ''}">
@@ -25,4 +27,6 @@
       <xacro:common_link_visual
         mesh_filename="gripper/bio/link_base${name_suffix}"
+        add_mesh_suffix="${add_mesh_suffix}"
+        other_mesh_suffix="${other_mesh_suffix}"
         origin_xyz="0 0 0"
         origin_rpy="0 0 0"
@@ -30,4 +34,6 @@
       <xacro:common_link_collision
         mesh_filename="gripper/bio/link_base${name_suffix}"
+        add_mesh_suffix="${add_mesh_suffix}"
+        other_mesh_suffix="${other_mesh_suffix}"
         origin_xyz="0 0 0"
         origin_rpy="0 0 0" />
@@ -43,4 +49,6 @@
       <xacro:common_link_visual
         mesh_filename="gripper/bio/left_finger${name_suffix}"
+        add_mesh_suffix="${add_mesh_suffix}"
+        other_mesh_suffix="${other_mesh_suffix}"
         origin_xyz="0 0 0"
         origin_rpy="0 0 0"
@@ -48,4 +56,6 @@
       <xacro:common_link_collision
         mesh_filename="gripper/bio/left_finger${name_suffix}"
+        add_mesh_suffix="${add_mesh_suffix}"
+        other_mesh_suffix="${other_mesh_suffix}"
         origin_xyz="0 0 0"
         origin_rpy="0 0 0" />
@@ -69,4 +79,6 @@
       <xacro:common_link_visual
         mesh_filename="gripper/bio/right_finger${name_suffix}"
+        add_mesh_suffix="${add_mesh_suffix}"
+        other_mesh_suffix="${other_mesh_suffix}"
         origin_xyz="0 0 0"
         origin_rpy="0 0 0"
@@ -74,4 +86,6 @@
       <xacro:common_link_collision
         mesh_filename="gripper/bio/right_finger${name_suffix}"
+        add_mesh_suffix="${add_mesh_suffix}"
+        other_mesh_suffix="${other_mesh_suffix}"
         origin_xyz="0 0 0"
         origin_rpy="0 0 0" />

File: xarm_description/urdf/gripper/xarm_gripper.urdf.xacro (robot description, xacro)
@@ -2,9 +2,11 @@
 <robot xmlns:xacro="http://ros.org/wiki/xacro" name="xarm_gripper">
   <xacro:macro name="xarm_gripper_urdf" params="prefix:='' attach_to:='' attach_xyz:='0 0 0' attach_rpy:='0 0 0' gripper_version:='G1' ">
+    <xacro:property name="add_mesh_suffix" value="true"/>
+    <xacro:property name="other_mesh_suffix" value=""/>
     <xacro:property name="name_suffix" value=""/>
-    <xacro:if value="${mesh_suffix == 'dae'}">
-      <xacro:if value="${gripper_version == 'G2' or gripper_version == 'g2'}">
-        <xacro:property name="name_suffix" value="_g2"/>
-      </xacro:if>
+    <xacro:if value="${gripper_version == 'G2' or gripper_version == 'g2'}">
+      <xacro:property name="name_suffix" value="_g2"/>
+      <xacro:property name="other_mesh_suffix" value="dae"/>
+      <xacro:property name="add_mesh_suffix" value="false"/>
     </xacro:if>
     <xacro:unless value="${attach_to == ''}">
@@ -25,4 +27,6 @@
       <xacro:common_link_visual
         mesh_filename="gripper/xarm/base_link${name_suffix}"
+        add_mesh_suffix="${add_mesh_suffix}"
+        other_mesh_suffix="${other_mesh_suffix}"
         origin_xyz="0 0 0"
         origin_rpy="0 0 0"
@@ -30,4 +34,6 @@
       <xacro:common_link_collision
         mesh_filename="gripper/xarm/base_link${name_suffix}"
+        add_mesh_suffix="${add_mesh_suffix}"
+        other_mesh_suffix="${other_mesh_suffix}"
         origin_xyz="0 0 0"
         origin_rpy="0 0 0" />
@@ -43,4 +49,6 @@
       <xacro:common_link_visual
         mesh_filename="gripper/xarm/left_outer_knuckle${name_suffix}"
+        add_mesh_suffix="${add_mesh_suffix}"
+        other_mesh_suffix="${other_mesh_suffix}"
         origin_xyz="0 0 0"
         origin_rpy="0 0 0"
@@ -48,4 +56,6 @@
       <xacro:common_link_collision
         mesh_filename="gripper/xarm/left_outer_knuckle${name_suffix}"
+        add_mesh_suffix="${add_mesh_suffix}"
+        other_mesh_suffix="${other_mesh_suffix}"
         origin_xyz="0 0 0"
         origin_rpy="0 0 0" />
@@ -68,4 +78,6 @@
       <xacro:common_link_visual
         mesh_filename="gripper/xarm/left_finger${name_suffix}"
+        add_mesh_suffix="${add_mesh_suffix}"
+        other_mesh_suffix="${other_mesh_suffix}"
         origin_xyz="0 0 0"
         origin_rpy="0 0 0"
@@ -73,4 +85,6 @@
       <xacro:common_link_collision
         mesh_filename="gripper/xarm/left_finger${name_suffix}"
+        add_mesh_suffix="${add_mesh_suffix}"
+        other_mesh_suffix="${other_mesh_suffix}"
         origin_xyz="0 0 0"
         origin_rpy="0 0 0" />
@@ -94,4 +108,6 @@
       <xacro:common_link_visual
         mesh_filename="gripper/xarm/left_inner_knuckle${name_suffix}"
+        add_mesh_suffix="${add_mesh_suffix}"
+        other_mesh_suffix="${other_mesh_suffix}"
         origin_xyz="0 0 0"
         origin_rpy="0 0 0"
@@ -99,4 +115,6 @@
       <xacro:common_link_collision
         mesh_filename="gripper/xarm/left_inner_knuckle${name_suffix}"
+        add_mesh_suffix="${add_mesh_suffix}"
+        other_mesh_suffix="${other_mesh_suffix}"
         origin_xyz="0 0 0"
         origin_rpy="0 0 0" />
@@ -120,4 +138,6 @@
       <xacro:common_link_visual
         mesh_filename="gripper/xarm/right_outer_knuckle${name_suffix}"
+        add_mesh_suffix="${add_mesh_suffix}"
+        other_mesh_suffix="${other_mesh_suffix}"
         origin_xyz="0 0 0"
         origin_rpy="0 0 0"
@@ -125,4 +145,6 @@
       <xacro:common_link_collision
         mesh_filename="gripper/xarm/right_outer_knuckle${name_suffix}"
+        add_mesh_suffix="${add_mesh_suffix}"
+        other_mesh_suffix="${other_mesh_suffix}"
         origin_xyz="0 0 0"
         origin_rpy="0 0 0" />
@@ -146,4 +168,6 @@
       <xacro:common_link_visual
         mesh_filename="gripper/xarm/right_finger${name_suffix}"
+        add_mesh_suffix="${add_mesh_suffix}"
+        other_mesh_suffix="${other_mesh_suffix}"
         origin_xyz="0 0 0"
         origin_rpy="0 0 0"
@@ -151,4 +175,6 @@
       <xacro:common_link_collision
         mesh_filename="gripper/xarm/right_finger${name_suffix}"
+        add_mesh_suffix="${add_mesh_suffix}"
+        other_mesh_suffix="${other_mesh_suffix}"
         origin_xyz="0 0 0"
         origin_rpy="0 0 0" />
@@ -172,4 +198,6 @@
       <xacro:common_link_visual
         mesh_filename="gripper/xarm/right_inner_knuckle${name_suffix}"
+        add_mesh_suffix="${add_mesh_suffix}"
+        other_mesh_suffix="${other_mesh_suffix}"
         origin_xyz="0 0 0"
         origin_rpy="0 0 0"
@@ -177,4 +205,6 @@
       <xacro:common_link_collision
         mesh_filename="gripper/xarm/right_inner_knuckle${name_suffix}"
+        add_mesh_suffix="${add_mesh_suffix}"
+        other_mesh_suffix="${other_mesh_suffix}"
         origin_xyz="0 0 0"
         origin_rpy="0 0 0" />
