Commit message: add modbus support and mimic joint plugin

File: xarm_gripper/urdf/xarm_gripper.gazebo.xacro (robot description, xacro)
@@ -1,25 +1,44 @@
 <?xml version="1.0"?>
 <robot xmlns:xacro="http://ros.org/wiki/xacro">
+  <!-- from mimic_joint_gazebo_tutorial by @mintar, refer: https://github.com/mintar/mimic_joint_gazebo_tutorial -->
+  <xacro:macro name="mimic_joint_plugin_gazebo" params="name_prefix following_joint mimic_joint has_pid:=false multiplier:=1.0 offset:=0 sensitiveness:=0.0 max_effort:=1.0 robot_namespace:=''">
+    <gazebo>
+      <plugin name="${name_prefix}mimic_joint_plugin" filename="libroboticsgroup_gazebo_mimic_joint_plugin.so">
+        <joint>${following_joint}</joint>
+        <mimicJoint>${mimic_joint}</mimicJoint>
+        <xacro:if value="${has_pid}">                     <!-- if set to true, PID parameters from "/gazebo_ros_control/pid_gains/${mimic_joint}" are loaded -->
+          <hasPID />
+        </xacro:if>
+        <multiplier>${multiplier}</multiplier>
+        <offset>${offset}</offset>
+        <sensitiveness>${sensitiveness}</sensitiveness>   <!-- if absolute difference between setpoint and process value is below this threshold, do nothing; 0.0 = disable [rad] -->
+        <maxEffort>${max_effort}</maxEffort>              <!-- only taken into account if has_pid:=true [Nm] -->
+        <xacro:unless value="${robot_namespace == ''}">
+          <robotNamespace>($robot_namespace)</robotNamespace>
+        </xacro:unless>
+      </plugin>
+    </gazebo>
+  </xacro:macro>
   <xacro:macro name="xarm_gripper_gazebo" params="prefix">
     <gazebo reference="${prefix}xarm_gripper_base_link">
-      <selfCollide>true</selfCollide>
+      <selfCollide>false</selfCollide>
     </gazebo>
     <gazebo reference="${prefix}left_outer_knuckle">
-      <selfCollide>true</selfCollide>
+      <selfCollide>false</selfCollide>
     </gazebo>
     <gazebo reference="${prefix}left_finger">
-      <selfCollide>true</selfCollide>
+      <selfCollide>false</selfCollide>
     </gazebo>
     <gazebo reference="${prefix}left_inner_knuckle">
-      <selfCollide>true</selfCollide>
+      <selfCollide>false</selfCollide>
     </gazebo>
     <gazebo reference="${prefix}right_outer_knuckle">
-      <selfCollide>true</selfCollide>
+      <selfCollide>false</selfCollide>
     </gazebo>
     <gazebo reference="${prefix}right_finger">
-      <selfCollide>true</selfCollide>
+      <selfCollide>false</selfCollide>
     </gazebo>
     <gazebo reference="${prefix}right_inner_knuckle">
-      <selfCollide>true</selfCollide>
+      <selfCollide>false</selfCollide>
     </gazebo>
   </xacro:macro>

File: xarm_gripper/urdf/xarm_gripper_model.xacro (robot description, xacro)
@@ -8,5 +8,5 @@
   <xacro:include filename="$(find xarm_gripper)/urdf/xarm_gripper.transmission.xacro" />
   <xacro:include filename="$(find xarm_gripper)/urdf/xarm_gripper.gazebo.xacro" />
-  <xacro:macro name="load_gripper" params="prefix:='' attach_to:='' ns:='xarm_gripper' xyz:='0 0 0' rpy:='0 0 0' effort_control:='false' ">
+  <xacro:macro name="load_gripper" params="prefix:='' attach_to:='' ns:='xarm' xyz:='0 0 0' rpy:='0 0 0' effort_control:='false' ">
     <!-- gazebo plugin -->
     <!-- <xacro:gazebo_ros_control_plugin namespace="${ns}"/> -->
@@ -19,4 +19,20 @@
     </xacro:unless>
     <xacro:xarm_gripper_gazebo prefix="${prefix}" />
+    <!-- mimic_joint_plugin has to be installed: -->
+    <xacro:mimic_joint_plugin_gazebo name_prefix="left_finger_joint"
+    following_joint="drive_joint" mimic_joint="left_finger_joint"
+    has_pid="true" multiplier="1.0" max_effort="10.0" />
+    <xacro:mimic_joint_plugin_gazebo name_prefix="left_inner_knuckle_joint"
+    following_joint="drive_joint" mimic_joint="left_inner_knuckle_joint"
+    has_pid="true" multiplier="1.0" max_effort="10.0" />
+    <xacro:mimic_joint_plugin_gazebo name_prefix="right_outer_knuckle_joint"
+    following_joint="drive_joint" mimic_joint="right_outer_knuckle_joint"
+    has_pid="true" multiplier="1.0" max_effort="10.0" />
+    <xacro:mimic_joint_plugin_gazebo name_prefix="right_finger_joint"
+    following_joint="drive_joint" mimic_joint="right_finger_joint"
+    has_pid="true" multiplier="1.0" max_effort="10.0" />
+    <xacro:mimic_joint_plugin_gazebo name_prefix="right_inner_knuckle_joint"
+    following_joint="drive_joint" mimic_joint="right_inner_knuckle_joint"
+    has_pid="true" multiplier="1.0" max_effort="10.0" />
   </xacro:macro>
 </robot>
