Commit message: add load_gazebo_plugin argument in robot_macro.xacro, to help prevent repetitive loading of gazebo_ros_control plugin for multi-robot gazebo simulations

File: xarm_gripper/urdf/xarm_gripper.urdf.xacro (robot description, xacro)
@@ -280,5 +280,5 @@
       effort="50"
       velocity="2" />
-    <mimic joint="drive_joint" multiplier="1" offset="0" />
+    <mimic joint="${prefix}drive_joint" multiplier="1" offset="0" />
   </joint>
   <link

Commit message: enable gripper/vacuum_gripper TCP offset in Moveit

File: xarm_gripper/urdf/xarm_gripper.urdf.xacro (robot description, xacro)
@@ -396,4 +396,16 @@
     <mimic joint="${prefix}drive_joint" multiplier="1" offset="0" />
   </joint>
+  <link name="${prefix}link_tcp" />
+  <joint
+    name="${prefix}joint_tcp"
+    type="fixed">
+    <origin
+      xyz="0 0 0.172"
+      rpy="0 0 0" />
+    <parent
+      link="${prefix}xarm_gripper_base_link" />
+    <child
+      link="${prefix}link_tcp" />
+  </joint>
   </xacro:macro>
 </robot>
