Commit message: optimize for ROS Kinetic

File: xarm_description/srdf/_xarm5_macro.srdf.xacro (robot description, xacro)
@@ -18,5 +18,4 @@
       <joint name="${prefix}joint4" />
       <joint name="${prefix}joint5" />
-      <joint name="${prefix}joint_eef" />
       <!-- To count in gripper TCP offset, if no need, please uncomment following 2 lines -->
       <xacro:if value="${add_gripper}">
@@ -24,13 +23,21 @@
         <joint name="${prefix}joint_tcp" />
       </xacro:if>
-      <xacro:if value="${not add_gripper and add_vacuum_gripper}">
+      <!-- 'not' seems not working in Kinetic evaluation  -->
+      <xacro:if value="${add_gripper=='false' and add_vacuum_gripper=='true'}">
         <joint name="${prefix}vacuum_gripper_fix" />
         <joint name="${prefix}joint_tcp" />
       </xacro:if>
-      <xacro:if value="${not add_gripper and not add_vacuum_gripper and add_other_geometry}">
+      <xacro:if value="${add_gripper=='false' and add_vacuum_gripper=='false' and add_other_geometry=='true'}">
         <joint name="${prefix}other_geometry_fix" />
         <joint name="${prefix}joint_tcp" />
       </xacro:if>
     </group>
+    <!-- end_effector must be defined to display planned path in xarm_planner -->
+    <xacro:if value="${add_gripper=='false' and add_vacuum_gripper=='false' and add_other_geometry=='false'}">
+      <group name="tool_end">
+        <joint name="${prefix}joint_eef" />
+      </group>
+      <end_effector name="end_effector" parent_link="link5" group="tool_end" />\
+    </xacro:if>
     <!-- GROUP STATES, Purpose, Define a named state for a particular group, in terms of joint values. This is useful to define states like 'folded arms' -->
     <group_state name="home" group="${prefix}xarm5">
@@ -113,9 +120,9 @@
     </xacro:if>
     <!-- vacuum gripper -->
-    <xacro:if value="${not add_gripper and add_vacuum_gripper}">
-      <!-- <group name="${prefix}vacuum_gripper">
+    <xacro:if value="${add_gripper=='false' and add_vacuum_gripper=='true'}">
+      <group name="${prefix}vacuum_gripper">
         <joint name="${prefix}vacuum_gripper_fix" />
-      </group> -->
-      <!-- <end_effector name="${prefix}vacuum_gripper" parent_link="${prefix}link_tcp" group="${prefix}vacuum_gripper" /> -->
+      </group>
+      <end_effector name="${prefix}vacuum_gripper" parent_link="${prefix}link_tcp" group="${prefix}vacuum_gripper" />
       <passive_joint name="${prefix}vacuum_gripper_fix" />
       <disable_collisions link1="${prefix}link4" link2="${prefix}xarm_vacuum_gripper_link" reason="Never" />
@@ -123,9 +130,9 @@
     </xacro:if>
     <!-- other box -->
-    <xacro:if value="${not add_gripper and not add_vacuum_gripper and add_other_geometry}">
-      <!-- <group name="${prefix}other_geometry">
+    <xacro:if value="${add_gripper=='false' and add_vacuum_gripper=='false' and add_other_geometry=='true'}">
+      <group name="${prefix}other_geometry">
         <joint name="${prefix}other_geometry_fix" />
-      </group> -->
-      <!-- <end_effector name="${prefix}other_geometry" parent_link="${prefix}link_tcp" group="${prefix}other_geometry" /> -->
+      </group>
+      <end_effector name="${prefix}other_geometry" parent_link="${prefix}link_tcp" group="${prefix}other_geometry" />
       <passive_joint name="${prefix}other_geometry_fix" />
       <disable_collisions link1="${prefix}link4" link2="${prefix}other_geometry_link" reason="Never" />
@@ -136,5 +143,4 @@
     <disable_collisions link1="${prefix}link2" link2="${prefix}link3" reason="Adjacent" />
     <disable_collisions link1="${prefix}link2" link2="${prefix}link4" reason="Never" />
-    <disable_collisions link1="${prefix}link2" link2="${prefix}link5" reason="Never" />
     <disable_collisions link1="${prefix}link2" link2="${prefix}link_base" reason="Never" />
     <disable_collisions link1="${prefix}link3" link2="${prefix}link4" reason="Adjacent" />

File: xarm_description/srdf/_xarm6_macro.srdf.xacro (robot description, xacro)
@@ -19,5 +19,4 @@
       <joint name="${prefix}joint5" />
       <joint name="${prefix}joint6" />
-      <joint name="${prefix}joint_eef" />
       <!-- To count in gripper TCP offset, if no need, please uncomment following 2 lines -->
       <xacro:if value="${add_gripper}">
@@ -25,13 +24,21 @@
         <joint name="${prefix}joint_tcp" />
       </xacro:if>
-      <xacro:if value="${not add_gripper and add_vacuum_gripper}">
+      <!-- 'not' seems not working in Kinetic evaluation  -->
+      <xacro:if value="${add_gripper=='false' and add_vacuum_gripper=='true'}">
         <joint name="${prefix}vacuum_gripper_fix" />
         <joint name="${prefix}joint_tcp" />
       </xacro:if>
-      <xacro:if value="${not add_gripper and not add_vacuum_gripper and add_other_geometry}">
+      <xacro:if value="${add_gripper=='false' and add_vacuum_gripper=='false' and add_other_geometry=='true'}">
         <joint name="${prefix}other_geometry_fix" />
         <joint name="${prefix}joint_tcp" />
       </xacro:if>
     </group>
+    <!-- end_effector must be defined to display planned path in xarm_planner -->
+    <xacro:if value="${add_gripper=='false' and add_vacuum_gripper=='false' and add_other_geometry=='false'}">
+      <group name="tool_end">
+        <joint name="${prefix}joint_eef" />
+      </group>
+      <end_effector name="end_effector" parent_link="link6" group="tool_end" />\
+    </xacro:if>
     <!-- GROUP STATES, Purpose, Define a named state for a particular group, in terms of joint values. This is useful to define states like 'folded arms' -->
     <group_state name="home" group="${prefix}xarm6">
@@ -121,9 +128,9 @@
     </xacro:if>
     <!-- vacuum gripper -->
-    <xacro:if value="${not add_gripper and add_vacuum_gripper}">
-      <!-- <group name="${prefix}vacuum_gripper">
+    <xacro:if value="${add_gripper=='false' and add_vacuum_gripper=='true'}">
+      <group name="${prefix}vacuum_gripper">
         <joint name="${prefix}vacuum_gripper_fix" />
-      </group> -->
-      <!-- <end_effector name="${prefix}vacuum_gripper" parent_link="${prefix}link_tcp" group="${prefix}vacuum_gripper" /> -->
+      </group>
+      <end_effector name="${prefix}vacuum_gripper" parent_link="${prefix}link_tcp" group="${prefix}vacuum_gripper" />
       <passive_joint name="${prefix}vacuum_gripper_fix" />
       <disable_collisions link1="${prefix}link5" link2="${prefix}xarm_vacuum_gripper_link" reason="Never" />
@@ -131,9 +138,9 @@
     </xacro:if>
     <!-- other box -->
-    <xacro:if value="${not add_gripper and not add_vacuum_gripper and add_other_geometry}">
-      <!-- <group name="${prefix}other_geometry">
+    <xacro:if value="${add_gripper=='false' and add_vacuum_gripper=='false' and add_other_geometry=='true'}">
+      <group name="${prefix}other_geometry">
         <joint name="${prefix}other_geometry_fix" />
-      </group> -->
-      <!-- <end_effector name="${prefix}other_geometry" parent_link="${prefix}link_tcp" group="${prefix}other_geometry" /> -->
+      </group>
+      <end_effector name="${prefix}other_geometry" parent_link="${prefix}link_tcp" group="${prefix}other_geometry" />
       <passive_joint name="${prefix}other_geometry_fix" />
       <disable_collisions link1="${prefix}link5" link2="${prefix}other_geometry_link" reason="Never" />

File: xarm_description/srdf/_xarm7_macro.srdf.xacro (robot description, xacro)
@@ -20,5 +20,4 @@
       <joint name="${prefix}joint6" />
       <joint name="${prefix}joint7" />
-      <joint name="${prefix}joint_eef" />
       <!-- To count in gripper TCP offset, if no need, please uncomment following 2 lines -->
       <xacro:if value="${add_gripper}">
@@ -26,13 +25,21 @@
         <joint name="${prefix}joint_tcp" />
       </xacro:if>
-      <xacro:if value="${not add_gripper and add_vacuum_gripper}">
+      <!-- 'not' seems not working in Kinetic evaluation  -->
+      <xacro:if value="${add_gripper=='false' and add_vacuum_gripper=='true'}">
         <joint name="${prefix}vacuum_gripper_fix" />
         <joint name="${prefix}joint_tcp" />
       </xacro:if>
-      <xacro:if value="${not add_gripper and not add_vacuum_gripper and add_other_geometry}">
+      <xacro:if value="${add_gripper=='false' and add_vacuum_gripper=='false' and add_other_geometry=='true'}">
         <joint name="${prefix}other_geometry_fix" />
         <joint name="${prefix}joint_tcp" />
       </xacro:if>
     </group>
+    <!-- end_effector must be defined to display planned path in xarm_planner -->
+    <xacro:if value="${add_gripper=='false' and add_vacuum_gripper=='false' and add_other_geometry=='false'}">
+      <group name="tool_end">
+        <joint name="${prefix}joint_eef" />
+      </group>
+      <end_effector name="end_effector" parent_link="link7" group="tool_end" />\
+    </xacro:if>
       <!-- GROUP STATES, Purpose, Define a named state for a particular group, in terms of joint values. This is useful to define states like 'folded arms' -->
     <group_state name="home" group="${prefix}xarm7">
@@ -129,9 +136,9 @@
     </xacro:if>
     <!-- vacuum gripper -->
-    <xacro:if value="${not add_gripper and add_vacuum_gripper}">
-      <!-- <group name="${prefix}vacuum_gripper">
+    <xacro:if value="${add_gripper=='false' and add_vacuum_gripper=='true'}">
+      <group name="${prefix}vacuum_gripper">
         <joint name="${prefix}vacuum_gripper_fix" />
-      </group> -->
-      <!-- <end_effector name="${prefix}vacuum_gripper" parent_link="${prefix}link_tcp" group="${prefix}vacuum_gripper" /> -->
+      </group>
+      <end_effector name="${prefix}vacuum_gripper" parent_link="${prefix}link_tcp" group="${prefix}vacuum_gripper" />
       <passive_joint name="${prefix}vacuum_gripper_fix" />
       <disable_collisions link1="${prefix}link3" link2="${prefix}xarm_vacuum_gripper_link" reason="Never" />
@@ -140,9 +147,9 @@
     </xacro:if>
     <!-- other box -->
-    <xacro:if value="${not add_gripper and not add_vacuum_gripper and add_other_geometry}">
-      <!-- <group name="${prefix}other_geometry">
+    <xacro:if value="${add_gripper=='false' and add_vacuum_gripper=='false' and add_other_geometry=='true'}">
+      <group name="${prefix}other_geometry">
         <joint name="${prefix}other_geometry_fix" />
-      </group> -->
-      <!-- <end_effector name="${prefix}other_geometry" parent_link="${prefix}link_tcp" group="${prefix}other_geometry" /> -->
+      </group>
+      <end_effector name="${prefix}other_geometry" parent_link="${prefix}link_tcp" group="${prefix}other_geometry" />
       <passive_joint name="${prefix}other_geometry_fix" />
       <disable_collisions link1="${prefix}link3" link2="${prefix}other_geometry_link" reason="Never" />
