Commit message: fix load other geometry

File: xarm_description/srdf/_xarm5_macro.srdf.xacro (robot description, xacro)
@@ -1,3 +1,3 @@
-<?xml version="1.0" ?>
+<?xml version="1.0" encoding="utf-8"?>
 <!-- This does not replace URDF, and is not an extension of URDF.
   This is a format for representing semantic information about the robot structure.
@@ -11,4 +11,28 @@
   <xacro:macro name="xarm5_macro_srdf" params="prefix=''
     add_gripper='false' add_vacuum_gripper='false' add_other_geometry='false' ">
+    <xacro:if value="${add_gripper}">
+      <xacro:property name="_use_gripper" value="true"/>
+      <xacro:property name="_use_vacuum_gripper" value="false"/>
+      <xacro:property name="_use_other_geometry" value="false"/>
+    </xacro:if>
+    <xacro:unless value="${add_gripper}">
+      <xacro:if value="${add_vacuum_gripper}">
+        <xacro:property name="_use_gripper" value="false"/>
+        <xacro:property name="_use_vacuum_gripper" value="true"/>
+        <xacro:property name="_use_other_geometry" value="false"/>
+      </xacro:if>
+      <xacro:unless value="${add_vacuum_gripper}">
+        <xacro:if value="${add_other_geometry}">
+          <xacro:property name="_use_gripper" value="false"/>
+          <xacro:property name="_use_vacuum_gripper" value="false"/>
+          <xacro:property name="_use_other_geometry" value="true"/>
+        </xacro:if>
+        <xacro:unless value="${add_other_geometry}">
+          <xacro:property name="_use_gripper" value="false"/>
+          <xacro:property name="_use_vacuum_gripper" value="false"/>
+          <xacro:property name="_use_other_geometry" value="false"/>
+        </xacro:unless>
+      </xacro:unless>
+    </xacro:unless>
     <group name="${prefix}xarm5">
       <joint name="${prefix}world_joint" />
@@ -19,14 +43,14 @@
       <joint name="${prefix}joint5" />
       <!-- To count in gripper TCP offset, if no need, please uncomment following 2 lines -->
-      <xacro:if value="${add_gripper}">
+      <xacro:if value="${_use_gripper}">
         <joint name="${prefix}gripper_fix" />
         <joint name="${prefix}joint_tcp" />
       </xacro:if>
       <!-- 'not' seems not working in Kinetic evaluation  -->
-      <xacro:if value="${add_gripper=='false' and add_vacuum_gripper=='true'}">
+      <xacro:if value="${_use_vacuum_gripper}">
         <joint name="${prefix}vacuum_gripper_fix" />
         <joint name="${prefix}joint_tcp" />
       </xacro:if>
-      <xacro:if value="${add_gripper=='false' and add_vacuum_gripper=='false' and add_other_geometry=='true'}">
+      <xacro:if value="${_use_other_geometry}">
         <joint name="${prefix}other_geometry_fix" />
         <joint name="${prefix}joint_tcp" />
@@ -34,10 +58,10 @@
     </group>
     <!-- end_effector must be defined to display planned path in xarm_planner -->
-    <xacro:if value="${add_gripper=='false' and add_vacuum_gripper=='false' and add_other_geometry=='false'}">
+    <xacro:unless value="${_use_gripper or _use_vacuum_gripper or _use_other_geometry}">
       <group name="tool_end">
         <joint name="${prefix}joint_eef" />
       </group>
-      <end_effector name="end_effector" parent_link="link5" group="tool_end" />\
-    </xacro:if>
+      <end_effector name="end_effector" parent_link="link5" group="tool_end" />
+    </xacro:unless>
     <!-- GROUP STATES, Purpose, Define a named state for a particular group, in terms of joint values. This is useful to define states like 'folded arms' -->
     <group_state name="home" group="${prefix}xarm5">
@@ -56,5 +80,5 @@
     </group_state>
     <!-- gripper -->
-    <xacro:if value="${add_gripper}">
+    <xacro:if value="${_use_gripper}">
       <group name="${prefix}xarm_gripper">
         <link name="${prefix}xarm_gripper_base_link" />
@@ -120,5 +144,5 @@
     </xacro:if>
     <!-- vacuum gripper -->
-    <xacro:if value="${add_gripper=='false' and add_vacuum_gripper=='true'}">
+    <xacro:if value="${_use_vacuum_gripper}">
       <group name="${prefix}vacuum_gripper">
         <joint name="${prefix}vacuum_gripper_fix" />
@@ -130,5 +154,5 @@
     </xacro:if>
     <!-- other box -->
-    <xacro:if value="${add_gripper=='false' and add_vacuum_gripper=='false' and add_other_geometry=='true'}">
+    <xacro:if value="${_use_other_geometry}">
       <group name="${prefix}other_geometry">
         <joint name="${prefix}other_geometry_fix" />

File: xarm_description/srdf/_xarm6_macro.srdf.xacro (robot description, xacro)
@@ -11,4 +11,28 @@
   <xacro:macro name="xarm6_macro_srdf" params="prefix=''
     add_gripper='false' add_vacuum_gripper='false' add_other_geometry='false' ">
+    <xacro:if value="${add_gripper}">
+      <xacro:property name="_use_gripper" value="true"/>
+      <xacro:property name="_use_vacuum_gripper" value="false"/>
+      <xacro:property name="_use_other_geometry" value="false"/>
+    </xacro:if>
+    <xacro:unless value="${add_gripper}">
+      <xacro:if value="${add_vacuum_gripper}">
+        <xacro:property name="_use_gripper" value="false"/>
+        <xacro:property name="_use_vacuum_gripper" value="true"/>
+        <xacro:property name="_use_other_geometry" value="false"/>
+      </xacro:if>
+      <xacro:unless value="${add_vacuum_gripper}">
+        <xacro:if value="${add_other_geometry}">
+          <xacro:property name="_use_gripper" value="false"/>
+          <xacro:property name="_use_vacuum_gripper" value="false"/>
+          <xacro:property name="_use_other_geometry" value="true"/>
+        </xacro:if>
+        <xacro:unless value="${add_other_geometry}">
+          <xacro:property name="_use_gripper" value="false"/>
+          <xacro:property name="_use_vacuum_gripper" value="false"/>
+          <xacro:property name="_use_other_geometry" value="false"/>
+        </xacro:unless>
+      </xacro:unless>
+    </xacro:unless>
     <group name="${prefix}xarm6">
       <joint name="${prefix}world_joint" />
@@ -20,14 +44,13 @@
       <joint name="${prefix}joint6" />
       <!-- To count in gripper TCP offset, if no need, please uncomment following 2 lines -->
-      <xacro:if value="${add_gripper}">
+      <xacro:if value="${_use_gripper}">
         <joint name="${prefix}gripper_fix" />
         <joint name="${prefix}joint_tcp" />
       </xacro:if>
-      <!-- 'not' seems not working in Kinetic evaluation  -->
-      <xacro:if value="${add_gripper=='false' and add_vacuum_gripper=='true'}">
+      <xacro:if value="${_use_vacuum_gripper}">
         <joint name="${prefix}vacuum_gripper_fix" />
         <joint name="${prefix}joint_tcp" />
       </xacro:if>
-      <xacro:if value="${add_gripper=='false' and add_vacuum_gripper=='false' and add_other_geometry=='true'}">
+      <xacro:if value="${_use_other_geometry}">
         <joint name="${prefix}other_geometry_fix" />
         <joint name="${prefix}joint_tcp" />
@@ -35,10 +58,10 @@
     </group>
     <!-- end_effector must be defined to display planned path in xarm_planner -->
-    <xacro:if value="${add_gripper=='false' and add_vacuum_gripper=='false' and add_other_geometry=='false'}">
+    <xacro:unless value="${_use_gripper or _use_vacuum_gripper or _use_other_geometry}">
       <group name="tool_end">
         <joint name="${prefix}joint_eef" />
       </group>
-      <end_effector name="end_effector" parent_link="link6" group="tool_end" />\
-    </xacro:if>
+      <end_effector name="end_effector" parent_link="link6" group="tool_end" />
+    </xacro:unless>
     <!-- GROUP STATES, Purpose, Define a named state for a particular group, in terms of joint values. This is useful to define states like 'folded arms' -->
     <group_state name="home" group="${prefix}xarm6">
@@ -59,5 +82,5 @@
     </group_state>
     <!-- gripper -->
-    <xacro:if value="${add_gripper}">
+    <xacro:if value="${_use_gripper}">
       <group name="${prefix}xarm_gripper">
         <link name="${prefix}xarm_gripper_base_link" />
@@ -128,5 +151,5 @@
     </xacro:if>
     <!-- vacuum gripper -->
-    <xacro:if value="${add_gripper=='false' and add_vacuum_gripper=='true'}">
+    <xacro:if value="${_use_vacuum_gripper}">
       <group name="${prefix}vacuum_gripper">
         <joint name="${prefix}vacuum_gripper_fix" />
@@ -138,5 +161,5 @@
     </xacro:if>
     <!-- other box -->
-    <xacro:if value="${add_gripper=='false' and add_vacuum_gripper=='false' and add_other_geometry=='true'}">
+    <xacro:if value="${_use_other_geometry}">
       <group name="${prefix}other_geometry">
         <joint name="${prefix}other_geometry_fix" />

File: xarm_description/srdf/_xarm7_macro.srdf.xacro (robot description, xacro)
@@ -1,3 +1,3 @@
-<?xml version="1.0" ?>
+<?xml version="1.0" encoding="utf-8"?>
 <!-- This does not replace URDF, and is not an extension of URDF.
   This is a format for representing semantic information about the robot structure.
@@ -11,4 +11,28 @@
   <xacro:macro name="xarm7_macro_srdf" params="prefix=''
     add_gripper='false' add_vacuum_gripper='false' add_other_geometry='false' ">
+    <xacro:if value="${add_gripper}">
+      <xacro:property name="_use_gripper" value="true"/>
+      <xacro:property name="_use_vacuum_gripper" value="false"/>
+      <xacro:property name="_use_other_geometry" value="false"/>
+    </xacro:if>
+    <xacro:unless value="${add_gripper}">
+      <xacro:if value="${add_vacuum_gripper}">
+        <xacro:property name="_use_gripper" value="false"/>
+        <xacro:property name="_use_vacuum_gripper" value="true"/>
+        <xacro:property name="_use_other_geometry" value="false"/>
+      </xacro:if>
+      <xacro:unless value="${add_vacuum_gripper}">
+        <xacro:if value="${add_other_geometry}">
+          <xacro:property name="_use_gripper" value="false"/>
+          <xacro:property name="_use_vacuum_gripper" value="false"/>
+          <xacro:property name="_use_other_geometry" value="true"/>
+        </xacro:if>
+        <xacro:unless value="${add_other_geometry}">
+          <xacro:property name="_use_gripper" value="false"/>
+          <xacro:property name="_use_vacuum_gripper" value="false"/>
+          <xacro:property name="_use_other_geometry" value="false"/>
+        </xacro:unless>
+      </xacro:unless>
+    </xacro:unless>
     <group name="${prefix}xarm7">
       <joint name="${prefix}world_joint" />
@@ -21,14 +45,14 @@
       <joint name="${prefix}joint7" />
       <!-- To count in gripper TCP offset, if no need, please uncomment following 2 lines -->
-      <xacro:if value="${add_gripper}">
+      <xacro:if value="${_use_gripper}">
         <joint name="${prefix}gripper_fix" />
         <joint name="${prefix}joint_tcp" />
       </xacro:if>
       <!-- 'not' seems not working in Kinetic evaluation  -->
-      <xacro:if value="${add_gripper=='false' and add_vacuum_gripper=='true'}">
+      <xacro:if value="${_use_vacuum_gripper}">
         <joint name="${prefix}vacuum_gripper_fix" />
         <joint name="${prefix}joint_tcp" />
       </xacro:if>
-      <xacro:if value="${add_gripper=='false' and add_vacuum_gripper=='false' and add_other_geometry=='true'}">
+      <xacro:if value="${_use_other_geometry}">
         <joint name="${prefix}other_geometry_fix" />
         <joint name="${prefix}joint_tcp" />
@@ -36,10 +60,10 @@
     </group>
     <!-- end_effector must be defined to display planned path in xarm_planner -->
-    <xacro:if value="${add_gripper=='false' and add_vacuum_gripper=='false' and add_other_geometry=='false'}">
+    <xacro:unless value="${_use_gripper or _use_vacuum_gripper or _use_other_geometry}">
       <group name="tool_end">
         <joint name="${prefix}joint_eef" />
       </group>
-      <end_effector name="end_effector" parent_link="link7" group="tool_end" />\
-    </xacro:if>
+      <end_effector name="end_effector" parent_link="link7" group="tool_end" />
+    </xacro:unless>
       <!-- GROUP STATES, Purpose, Define a named state for a particular group, in terms of joint values. This is useful to define states like 'folded arms' -->
     <group_state name="home" group="${prefix}xarm7">
@@ -62,5 +86,5 @@
     </group_state>
     <!-- gripper -->
-    <xacro:if value="${add_gripper}">
+    <xacro:if value="${_use_gripper}">
       <group name="${prefix}xarm_gripper">
         <link name="${prefix}xarm_gripper_base_link" />
@@ -136,5 +160,5 @@
     </xacro:if>
     <!-- vacuum gripper -->
-    <xacro:if value="${add_gripper=='false' and add_vacuum_gripper=='true'}">
+    <xacro:if value="${_use_vacuum_gripper}">
       <group name="${prefix}vacuum_gripper">
         <joint name="${prefix}vacuum_gripper_fix" />
@@ -147,5 +171,5 @@
     </xacro:if>
     <!-- other box -->
-    <xacro:if value="${add_gripper=='false' and add_vacuum_gripper=='false' and add_other_geometry=='true'}">
+    <xacro:if value="${_use_other_geometry}">
       <group name="${prefix}other_geometry">
         <joint name="${prefix}other_geometry_fix" />

Commit message: remove condition(or) in srdf

File: xarm_description/srdf/_xarm5_macro.srdf.xacro (robot description, xacro)
@@ -15,4 +15,5 @@
       <xacro:property name="_use_vacuum_gripper" value="false"/>
       <xacro:property name="_use_other_geometry" value="false"/>
+      <xacro:property name="_use_no_end_effector" value="false"/>
     </xacro:if>
     <xacro:unless value="${add_gripper}">
@@ -21,4 +22,5 @@
         <xacro:property name="_use_vacuum_gripper" value="true"/>
         <xacro:property name="_use_other_geometry" value="false"/>
+        <xacro:property name="_use_no_end_effector" value="false"/>
       </xacro:if>
       <xacro:unless value="${add_vacuum_gripper}">
@@ -27,4 +29,5 @@
           <xacro:property name="_use_vacuum_gripper" value="false"/>
           <xacro:property name="_use_other_geometry" value="true"/>
+          <xacro:property name="_use_no_end_effector" value="false"/>
         </xacro:if>
         <xacro:unless value="${add_other_geometry}">
@@ -32,4 +35,5 @@
           <xacro:property name="_use_vacuum_gripper" value="false"/>
           <xacro:property name="_use_other_geometry" value="false"/>
+          <xacro:property name="_use_no_end_effector" value="true"/>
         </xacro:unless>
       </xacro:unless>
@@ -58,10 +62,10 @@
     </group>
     <!-- end_effector must be defined to display planned path in xarm_planner -->
-    <xacro:unless value="${_use_gripper or _use_vacuum_gripper or _use_other_geometry}">
+    <xacro:if value="${_use_no_end_effector}">
       <group name="tool_end">
         <joint name="${prefix}joint_eef" />
       </group>
       <end_effector name="end_effector" parent_link="link5" group="tool_end" />
-    </xacro:unless>
+    </xacro:if>
     <!-- GROUP STATES, Purpose, Define a named state for a particular group, in terms of joint values. This is useful to define states like 'folded arms' -->
     <group_state name="home" group="${prefix}xarm5">

File: xarm_description/srdf/_xarm6_macro.srdf.xacro (robot description, xacro)
@@ -15,4 +15,5 @@
       <xacro:property name="_use_vacuum_gripper" value="false"/>
       <xacro:property name="_use_other_geometry" value="false"/>
+      <xacro:property name="_use_no_end_effector" value="false"/>
     </xacro:if>
     <xacro:unless value="${add_gripper}">
@@ -21,4 +22,5 @@
         <xacro:property name="_use_vacuum_gripper" value="true"/>
         <xacro:property name="_use_other_geometry" value="false"/>
+        <xacro:property name="_use_no_end_effector" value="false"/>
       </xacro:if>
       <xacro:unless value="${add_vacuum_gripper}">
@@ -27,4 +29,5 @@
           <xacro:property name="_use_vacuum_gripper" value="false"/>
           <xacro:property name="_use_other_geometry" value="true"/>
+          <xacro:property name="_use_no_end_effector" value="false"/>
         </xacro:if>
         <xacro:unless value="${add_other_geometry}">
@@ -32,4 +35,5 @@
           <xacro:property name="_use_vacuum_gripper" value="false"/>
           <xacro:property name="_use_other_geometry" value="false"/>
+          <xacro:property name="_use_no_end_effector" value="true"/>
         </xacro:unless>
       </xacro:unless>
@@ -58,10 +62,10 @@
     </group>
     <!-- end_effector must be defined to display planned path in xarm_planner -->
-    <xacro:unless value="${_use_gripper or _use_vacuum_gripper or _use_other_geometry}">
+    <xacro:if value="${_use_no_end_effector}">
       <group name="tool_end">
         <joint name="${prefix}joint_eef" />
       </group>
       <end_effector name="end_effector" parent_link="link6" group="tool_end" />
-    </xacro:unless>
+    </xacro:if>
     <!-- GROUP STATES, Purpose, Define a named state for a particular group, in terms of joint values. This is useful to define states like 'folded arms' -->
     <group_state name="home" group="${prefix}xarm6">

File: xarm_description/srdf/_xarm7_macro.srdf.xacro (robot description, xacro)
@@ -15,4 +15,5 @@
       <xacro:property name="_use_vacuum_gripper" value="false"/>
       <xacro:property name="_use_other_geometry" value="false"/>
+      <xacro:property name="_use_no_end_effector" value="false"/>
     </xacro:if>
     <xacro:unless value="${add_gripper}">
@@ -21,4 +22,5 @@
         <xacro:property name="_use_vacuum_gripper" value="true"/>
         <xacro:property name="_use_other_geometry" value="false"/>
+        <xacro:property name="_use_no_end_effector" value="false"/>
       </xacro:if>
       <xacro:unless value="${add_vacuum_gripper}">
@@ -27,4 +29,5 @@
           <xacro:property name="_use_vacuum_gripper" value="false"/>
           <xacro:property name="_use_other_geometry" value="true"/>
+          <xacro:property name="_use_no_end_effector" value="false"/>
         </xacro:if>
         <xacro:unless value="${add_other_geometry}">
@@ -32,4 +35,5 @@
           <xacro:property name="_use_vacuum_gripper" value="false"/>
           <xacro:property name="_use_other_geometry" value="false"/>
+          <xacro:property name="_use_no_end_effector" value="true"/>
         </xacro:unless>
       </xacro:unless>
@@ -60,10 +64,10 @@
     </group>
     <!-- end_effector must be defined to display planned path in xarm_planner -->
-    <xacro:unless value="${_use_gripper or _use_vacuum_gripper or _use_other_geometry}">
+    <xacro:if value="${_use_no_end_effector}">
       <group name="tool_end">
         <joint name="${prefix}joint_eef" />
       </group>
       <end_effector name="end_effector" parent_link="link7" group="tool_end" />
-    </xacro:unless>
+    </xacro:if>
       <!-- GROUP STATES, Purpose, Define a named state for a particular group, in terms of joint values. This is useful to define states like 'folded arms' -->
     <group_state name="home" group="${prefix}xarm7">
