Commit message: test for realsense, add some collision stl

File: xarm_description/srdf/_xarm7_macro.srdf.xacro (robot description, xacro)
@@ -142,4 +142,7 @@
       <disable_collisions link1="${prefix}left_outer_knuckle" link2="${prefix}right_outer_knuckle" reason="Never" />
       <disable_collisions link1="${prefix}left_outer_knuckle" link2="${prefix}xarm_gripper_base_link" reason="Adjacent" />
+      <disable_collisions link1="${prefix}link_eef" link2="${prefix}left_finger" reason="Never" />
+      <disable_collisions link1="${prefix}link_eef" link2="${prefix}left_inner_knuckle" reason="Never" />
+      <disable_collisions link1="${prefix}link_eef" link2="${prefix}left_outer_knuckle" reason="Never" />
       <disable_collisions link1="${prefix}link3" link2="${prefix}right_inner_knuckle" reason="Never" />
       <disable_collisions link1="${prefix}link3" link2="${prefix}right_outer_knuckle" reason="Never" />
@@ -155,5 +158,9 @@
       <disable_collisions link1="${prefix}link7" link2="${prefix}right_inner_knuckle" reason="Never" />
       <disable_collisions link1="${prefix}link7" link2="${prefix}right_outer_knuckle" reason="Never" />
-      <disable_collisions link1="${prefix}link7" link2="${prefix}xarm_gripper_base_link" reason="Adjacent" />
+      <disable_collisions link1="${prefix}link7" link2="${prefix}xarm_gripper_base_link" reason="Never" />
+      <disable_collisions link1="${prefix}link_eef" link2="${prefix}xarm_gripper_base_link" reason="Adjacent" />
+      <disable_collisions link1="${prefix}link_eef" link2="${prefix}right_finger" reason="Never" />
+      <disable_collisions link1="${prefix}link_eef" link2="${prefix}right_inner_knuckle" reason="Never" />
+      <disable_collisions link1="${prefix}link_eef" link2="${prefix}right_outer_knuckle" reason="Never" />
       <disable_collisions link1="${prefix}right_finger" link2="${prefix}right_inner_knuckle" reason="Default" />
       <disable_collisions link1="${prefix}right_finger" link2="${prefix}right_outer_knuckle" reason="Adjacent" />
@@ -202,4 +209,8 @@
     <disable_collisions link1="${prefix}link5" link2="${prefix}link7" reason="Never" />
     <disable_collisions link1="${prefix}link6" link2="${prefix}link7" reason="Adjacent" />
+    <disable_collisions link1="${prefix}link3" link2="${prefix}link_eef" reason="Never" />
+    <disable_collisions link1="${prefix}link4" link2="${prefix}link_eef" reason="Never" />
+    <disable_collisions link1="${prefix}link6" link2="${prefix}link_eef" reason="Never" />
+    <disable_collisions link1="${prefix}link7" link2="${prefix}link_eef" reason="Adjacent" />
   </xacro:macro>
 </robot>

File: xarm_description/urdf/xarm7.urdf.xacro (robot description, xacro)
@@ -435,5 +435,5 @@
       <geometry>
         <mesh
-          filename="package://xarm_description/meshes/xarm7/visual/link7.STL" />
+          filename="package://xarm_description/meshes/collision/end_tool.STL" />
       </geometry>
     </collision>
@@ -460,5 +460,25 @@
       friction="1" />
   </joint>
-  <link name="${prefix}link_eef" />
+  <link name="${prefix}link_eef">
+    <visual>
+      <origin
+        xyz="0 0 0"
+        rpy="0 0 0" />
+      <geometry>
+        <mesh
+          filename="package://d435i_xarm_setup/mesh/d435_with_cam_stand.STL" />
+      </geometry>
+      <material name="Silver" />
+    </visual>
+    <collision>
+      <origin
+        xyz="0 0 0"
+        rpy="0 0 0" />
+      <geometry>
+        <mesh
+          filename="package://d435i_xarm_setup/mesh/d435_with_cam_stand_collision.STL" />
+      </geometry>
+    </collision>
+  </link>
   <joint
     name="${prefix}joint_eef"

File: xarm_description/urdf/xarm7_with_gripper.xacro (robot description, xacro)
@@ -11,4 +11,4 @@
   <xacro:include filename="$(find xarm_gripper)/urdf/xarm_gripper_model.xacro" />
   <xacro:xarm7_robot prefix="$(arg prefix)" namespace="$(arg ros_namespace)" limited="$(arg limited)" effort_control="$(arg effort_control)" velocity_control="$(arg velocity_control)" />
-  <xacro:load_gripper attach_to="$(arg prefix)link_eef" effort_control="$(arg effort_control)" velocity_control="$(arg velocity_control)" />
+  <xacro:load_gripper attach_to="$(arg prefix)link_eef" xyz='0 0 0.003' effort_control="$(arg effort_control)" velocity_control="$(arg velocity_control)" />
 </robot>

Commit message: add xarm_vision and remove xarm_device

File: xarm_description/srdf/_xarm7_macro.srdf.xacro (robot description, xacro)
@@ -68,5 +68,5 @@
         <joint name="${prefix}joint_eef" />
       </group>
-      <end_effector name="end_effector" parent_link="link7" group="tool_end" />
+      <end_effector name="end_effector" parent_link="${prefix}link7" group="tool_end" />
     </xacro:if>
       <!-- GROUP STATES, Purpose, Define a named state for a particular group, in terms of joint values. This is useful to define states like 'folded arms' -->
@@ -179,5 +179,6 @@
       <disable_collisions link1="${prefix}link3" link2="${prefix}xarm_vacuum_gripper_link" reason="Never" />
       <disable_collisions link1="${prefix}link6" link2="${prefix}xarm_vacuum_gripper_link" reason="Never" />
-      <disable_collisions link1="${prefix}link7" link2="${prefix}xarm_vacuum_gripper_link" reason="Adjacent" />
+      <disable_collisions link1="${prefix}link7" link2="${prefix}xarm_vacuum_gripper_link" reason="Never" />
+      <disable_collisions link1="${prefix}link_eef" link2="${prefix}xarm_vacuum_gripper_link" reason="Adjacent" />
     </xacro:if>
     <!-- other box -->
@@ -190,5 +191,6 @@
       <disable_collisions link1="${prefix}link3" link2="${prefix}other_geometry_link" reason="Never" />
       <disable_collisions link1="${prefix}link6" link2="${prefix}other_geometry_link" reason="Never" />
-      <disable_collisions link1="${prefix}link7" link2="${prefix}other_geometry_link" reason="Adjacent" />
+      <disable_collisions link1="${prefix}link7" link2="${prefix}other_geometry_link" reason="Never" />
+      <disable_collisions link1="${prefix}link_eef" link2="${prefix}other_geometry_link" reason="Adjacent" />
     </xacro:if>
     <disable_collisions link1="${prefix}link1" link2="${prefix}link2" reason="Adjacent" />
@@ -209,5 +211,4 @@
     <disable_collisions link1="${prefix}link5" link2="${prefix}link7" reason="Never" />
     <disable_collisions link1="${prefix}link6" link2="${prefix}link7" reason="Adjacent" />
-    <disable_collisions link1="${prefix}link3" link2="${prefix}link_eef" reason="Never" />
     <disable_collisions link1="${prefix}link4" link2="${prefix}link_eef" reason="Never" />
     <disable_collisions link1="${prefix}link6" link2="${prefix}link_eef" reason="Never" />

File: xarm_description/urdf/xarm5_robot_macro.xacro (robot description, xacro)
@@ -2,5 +2,5 @@
 <robot xmlns:xacro="http://ros.org/wiki/xacro" name="xarm5" >
   <xacro:macro name="xarm5_robot" params="prefix:='' namespace:='xarm' limited:='false' effort_control:='false'
-    velocity_control:='false' attach_to:='world' xyz:='0 0 0' rpy:='0 0 0' load_gazebo_plugin:='true'
+    velocity_control:='false' attach_to:='world' xyz:='0 0 0' rpy:='0 0 0' load_gazebo_plugin:='true' rs_d435i:='false'
     add_other_geometry:='false'
     geometry_type:='box' geometry_mass:='0.1'
@@ -36,8 +36,9 @@
         joint3_lower_limit="${-pi*0.99}" joint3_upper_limit="${0.19198}"
         joint4_lower_limit="${-1.69297}" joint4_upper_limit="${pi*0.99}"
-        joint5_lower_limit="${-pi*0.99}" joint5_upper_limit="${pi*0.99}"/>
+        joint5_lower_limit="${-pi*0.99}" joint5_upper_limit="${pi*0.99}"
+        rs_d435i="${rs_d435i}"/>
     </xacro:if>
     <xacro:unless value="${limited}">
-      <xacro:xarm5_urdf prefix="${prefix}"/>
+      <xacro:xarm5_urdf prefix="${prefix}" rs_d435i="${rs_d435i}"/>
     </xacro:unless>
     <xacro:xarm5_transmission prefix="${prefix}" hard_interface="$(eval 'EffortJointInterface' if ${effort_control} else 'VelocityJointInterface' if ${velocity_control} else 'PositionJointInterface')" />

File: xarm_description/urdf/xarm6_robot_macro.xacro (robot description, xacro)
@@ -2,5 +2,5 @@
 <robot xmlns:xacro="http://ros.org/wiki/xacro" name="xarm6" >
   <xacro:macro name="xarm6_robot" params="prefix:='' namespace:='xarm' limited:='false' effort_control:='false'
-    velocity_control:='false' attach_to:='world' xyz:='0 0 0' rpy:='0 0 0' load_gazebo_plugin:='true'
+    velocity_control:='false' attach_to:='world' xyz:='0 0 0' rpy:='0 0 0' load_gazebo_plugin:='true' rs_d435i:='false'
     add_other_geometry:='false'
     geometry_type:='box' geometry_mass:='0.1'
@@ -37,8 +37,9 @@
         joint4_lower_limit="${-pi*0.99}" joint4_upper_limit="${pi*0.99}"
         joint5_lower_limit="${-1.69297}" joint5_upper_limit="${pi*0.99}"
-        joint6_lower_limit="${-pi*0.99}" joint6_upper_limit="${pi*0.99}"/>
+        joint6_lower_limit="${-pi*0.99}" joint6_upper_limit="${pi*0.99}"
+        rs_d435i="${rs_d435i}"/>
     </xacro:if>
     <xacro:unless value="${limited}">
-      <xacro:xarm6_urdf prefix="${prefix}"/>
+      <xacro:xarm6_urdf prefix="${prefix}" rs_d435i="${rs_d435i}"/>
     </xacro:unless>
     <xacro:xarm6_transmission prefix="${prefix}" hard_interface="$(eval 'EffortJointInterface' if ${effort_control} else 'VelocityJointInterface' if ${velocity_control} else 'PositionJointInterface')" />

File: xarm_description/urdf/xarm7.urdf.xacro (robot description, xacro)
@@ -12,5 +12,6 @@
     joint5_lower_limit:=${-2.0*pi}  joint5_upper_limit:=${2.0*pi}
     joint6_lower_limit:=${-1.69297}  joint6_upper_limit:=${pi}
-    joint7_lower_limit:=${-2.0*pi}  joint7_upper_limit:=${2.0*pi}">
+    joint7_lower_limit:=${-2.0*pi}  joint7_upper_limit:=${2.0*pi}
+    rs_d435i:=false">
     <material name="Black">
       <color rgba="0.0 0.0 0.0 1.0"/>
@@ -460,25 +461,30 @@
       friction="1" />
   </joint>
-  <link name="${prefix}link_eef">
-    <visual>
-      <origin
-        xyz="0 0 0"
-        rpy="0 0 0" />
-      <geometry>
-        <mesh
-          filename="package://d435i_xarm_setup/mesh/d435_with_cam_stand.STL" />
-      </geometry>
-      <material name="Silver" />
-    </visual>
-    <collision>
-      <origin
-        xyz="0 0 0"
-        rpy="0 0 0" />
-      <geometry>
-        <mesh
-          filename="package://d435i_xarm_setup/mesh/d435_with_cam_stand_collision.STL" />
-      </geometry>
-    </collision>
-  </link>
+  <xacro:if value="${rs_d435i}">
+    <link name="${prefix}link_eef">
+      <visual>
+        <origin
+          xyz="0 0 0"
+          rpy="0 0 0" />
+        <geometry>
+          <mesh
+            filename="package://d435i_xarm_setup/mesh/d435_with_cam_stand.STL" />
+        </geometry>
+        <material name="Silver" />
+      </visual>
+      <collision>
+        <origin
+          xyz="0 0 0"
+          rpy="0 0 0" />
+        <geometry>
+          <mesh
+            filename="package://d435i_xarm_setup/mesh/d435_with_cam_stand_collision.STL" />
+        </geometry>
+      </collision>
+    </link>
+  </xacro:if>
+  <xacro:unless value="${rs_d435i}">
+    <link name="${prefix}link_eef"/>
+  </xacro:unless>
   <joint
     name="${prefix}joint_eef"

File: xarm_description/urdf/xarm7_robot_macro.xacro (robot description, xacro)
@@ -2,5 +2,5 @@
 <robot xmlns:xacro="http://ros.org/wiki/xacro" name="xarm7" >
   <xacro:macro name="xarm7_robot" params="prefix:='' namespace:='xarm' limited:='false' effort_control:='false'
-    velocity_control:='false' attach_to:='world' xyz:='0 0 0' rpy:='0 0 0' load_gazebo_plugin:='true'
+    velocity_control:='false' attach_to:='world' xyz:='0 0 0' rpy:='0 0 0' load_gazebo_plugin:='true' rs_d435i:='false'
     add_other_geometry:='false'
     geometry_type:='box' geometry_mass:='0.1'
@@ -38,8 +38,9 @@
         joint5_lower_limit="${-pi*0.99}" joint5_upper_limit="${pi*0.99}"
         joint6_lower_limit="${-1.75}" joint6_upper_limit="${pi*0.99}"
-        joint7_lower_limit="${-pi*0.99}" joint7_upper_limit="${pi*0.99}"/>
+        joint7_lower_limit="${-pi*0.99}" joint7_upper_limit="${pi*0.99}"
+        rs_d435i="${rs_d435i}"/>
     </xacro:if>
     <xacro:unless value="${limited}">
-      <xacro:xarm7_urdf prefix="${prefix}"/>
+      <xacro:xarm7_urdf prefix="${prefix}" rs_d435i="${rs_d435i}"/>
     </xacro:unless>
     <xacro:xarm7_transmission prefix="${prefix}" hard_interface="$(eval 'EffortJointInterface' if ${effort_control} else 'VelocityJointInterface' if ${velocity_control} else 'PositionJointInterface')" />

File: xarm_description/urdf/xarm7_with_gripper.xacro (robot description, xacro)
@@ -1,4 +1,4 @@
 <?xml version='1.0' encoding='utf-8'?>
-<robot xmlns:xacro="http://ros.org/wiki/xacro" name="xarm7_with_gripper">
+<robot xmlns:xacro="http://ros.org/wiki/xacro" name="xarm7">
   <xacro:arg name="prefix" default=""/>
   <xacro:arg name="ros_namespace" default="xarm"/>
@@ -6,9 +6,16 @@
   <xacro:arg name="effort_control" default="false"/>
   <xacro:arg name="velocity_control" default="false"/>
+  <!-- To add realsense d435i and gripper, set 'add_realsense_d435i' = true -->
+  <xacro:arg name="add_realsense_d435i" default="false"/>
   <!-- load xarm7 robot -->
   <xacro:include filename="$(find xarm_description)/urdf/xarm7_robot_macro.xacro" />
   <!-- Attach gripper -->
   <xacro:include filename="$(find xarm_gripper)/urdf/xarm_gripper_model.xacro" />
-  <xacro:xarm7_robot prefix="$(arg prefix)" namespace="$(arg ros_namespace)" limited="$(arg limited)" effort_control="$(arg effort_control)" velocity_control="$(arg velocity_control)" />
-  <xacro:load_gripper attach_to="$(arg prefix)link_eef" xyz='0 0 0.003' effort_control="$(arg effort_control)" velocity_control="$(arg velocity_control)" />
+  <xacro:xarm7_robot prefix="$(arg prefix)" namespace="$(arg ros_namespace)" limited="$(arg limited)" effort_control="$(arg effort_control)" velocity_control="$(arg velocity_control)" rs_d435i="$(arg add_realsense_d435i)"/>
+  <xacro:if value="$(arg add_realsense_d435i)">
+    <xacro:load_gripper attach_to="$(arg prefix)link_eef" xyz="0 0 0.003" effort_control="$(arg effort_control)" velocity_control="$(arg velocity_control)" />
+  </xacro:if>
+  <xacro:unless value="$(arg add_realsense_d435i)">
+    <xacro:load_gripper attach_to="$(arg prefix)link_eef" effort_control="$(arg effort_control)" velocity_control="$(arg velocity_control)" />
+  </xacro:unless>
 </robot>
