Commit message: optimize support for lite6, add specific ReadMe

File: xarm_description/srdf/_lite6_macro.srdf.xacro (robot description, xacro)
@@ -77,87 +77,24 @@
       <joint name="${prefix}joint6" value="0" />
     </group_state>
-    <group_state name="hold-up" group="${prefix}lite6">
-      <joint name="${prefix}joint1" value="0" />
-      <joint name="${prefix}joint2" value="0" />
-      <joint name="${prefix}joint3" value="0" />
-      <joint name="${prefix}joint4" value="0" />
-      <joint name="${prefix}joint5" value="-1.5708" />
-      <joint name="${prefix}joint6" value="0" />
-    </group_state>
     <!-- gripper -->
     <xacro:if value="${_use_gripper}">
-      <group name="${prefix}xarm_gripper">
-        <link name="${prefix}xarm_gripper_base_link" />
-        <link name="${prefix}left_outer_knuckle" />
-        <link name="${prefix}left_finger" />
-        <link name="${prefix}left_inner_knuckle" />
-        <link name="${prefix}right_inner_knuckle" />
-        <link name="${prefix}right_outer_knuckle" />
-        <link name="${prefix}right_finger" />
+      <group name="${prefix}lite_gripper">
+        <link name="${prefix}uflite_gripper_link" />
         <link name="${prefix}link_tcp" />
-        <joint name="${prefix}drive_joint" />
+        <joint name="${prefix}gripper_fix" />
       </group>
-      <group_state name="open" group="${prefix}xarm_gripper">
+     <!--  <group_state name="open" group="${prefix}xarm_gripper">
         <joint name="${prefix}drive_joint" value="0" />
       </group_state>
       <group_state name="close" group="${prefix}xarm_gripper">
         <joint name="${prefix}drive_joint" value="0.85" />
-      </group_state>
+      </group_state> -->
       <!-- END EFFECTOR, Purpose, Represent information about an end effector. -->
-      <end_effector name="${prefix}xarm_gripper" parent_link="${prefix}link_tcp" group="${prefix}xarm_gripper" />
-      <!--PASSIVE JOINT, Purpose, this element is used to mark joints that are not actuated-->
-      <passive_joint name="${prefix}left_finger_joint" />
-      <passive_joint name="${prefix}left_inner_knuckle_joint" />
-      <passive_joint name="${prefix}right_inner_knuckle_joint" />
-      <passive_joint name="${prefix}right_outer_knuckle_joint" />
-      <passive_joint name="${prefix}right_finger_joint" />
+      <end_effector name="${prefix}lite_gripper" parent_link="${prefix}link_tcp" group="${prefix}lite_gripper" />
+      <passive_joint name="${prefix}gripper_fix" />
       <!-- DISABLE COLLISIONS, By default it is assumed that any link of the robot could potentially come into collision with any other link in the robot. This tag disables collision checking between a specified pair of links. -->
-      <disable_collisions link1="${prefix}left_finger" link2="${prefix}left_inner_knuckle" reason="Default" />
-      <disable_collisions link1="${prefix}left_finger" link2="${prefix}left_outer_knuckle" reason="Adjacent" />
-      <disable_collisions link1="${prefix}left_finger" link2="${prefix}link4" reason="Never" />
-      <disable_collisions link1="${prefix}left_finger" link2="${prefix}link5" reason="Never" />
-      <disable_collisions link1="${prefix}left_finger" link2="${prefix}link6" reason="Never" />
-      <disable_collisions link1="${prefix}left_finger" link2="${prefix}right_finger" reason="Never" />
-      <disable_collisions link1="${prefix}left_finger" link2="${prefix}right_inner_knuckle" reason="Never" />
-      <disable_collisions link1="${prefix}left_finger" link2="${prefix}right_outer_knuckle" reason="Never" />
-      <disable_collisions link1="${prefix}left_finger" link2="${prefix}xarm_gripper_base_link" reason="Never" />
-      <disable_collisions link1="${prefix}left_inner_knuckle" link2="${prefix}left_outer_knuckle" reason="Never" />
-      <disable_collisions link1="${prefix}left_inner_knuckle" link2="${prefix}link4" reason="Never" />
-      <disable_collisions link1="${prefix}left_inner_knuckle" link2="${prefix}link5" reason="Never" />
-      <disable_collisions link1="${prefix}left_inner_knuckle" link2="${prefix}link6" reason="Never" />
-      <disable_collisions link1="${prefix}left_inner_knuckle" link2="${prefix}right_finger" reason="Never" />
-      <disable_collisions link1="${prefix}left_inner_knuckle" link2="${prefix}right_inner_knuckle" reason="Never" />
-      <disable_collisions link1="${prefix}left_inner_knuckle" link2="${prefix}right_outer_knuckle" reason="Never" />
-      <disable_collisions link1="${prefix}left_inner_knuckle" link2="${prefix}xarm_gripper_base_link" reason="Adjacent" />
-      <disable_collisions link1="${prefix}left_outer_knuckle" link2="${prefix}link5" reason="Never" />
-      <disable_collisions link1="${prefix}left_outer_knuckle" link2="${prefix}link6" reason="Never" />
-      <disable_collisions link1="${prefix}left_outer_knuckle" link2="${prefix}right_finger" reason="Never" />
-      <disable_collisions link1="${prefix}left_outer_knuckle" link2="${prefix}right_inner_knuckle" reason="Never" />
-      <disable_collisions link1="${prefix}left_outer_knuckle" link2="${prefix}right_outer_knuckle" reason="Never" />
-      <disable_collisions link1="${prefix}left_outer_knuckle" link2="${prefix}xarm_gripper_base_link" reason="Adjacent" />
-      <disable_collisions link1="${prefix}link_eef" link2="${prefix}left_finger" reason="Never" />
-      <disable_collisions link1="${prefix}link_eef" link2="${prefix}left_inner_knuckle" reason="Never" />
-      <disable_collisions link1="${prefix}link_eef" link2="${prefix}left_outer_knuckle" reason="Never" />
-      <disable_collisions link1="${prefix}link4" link2="${prefix}right_finger" reason="Never" />
-      <disable_collisions link1="${prefix}link4" link2="${prefix}right_inner_knuckle" reason="Never" />
-      <disable_collisions link1="${prefix}link5" link2="${prefix}link6" reason="Adjacent" />
-      <disable_collisions link1="${prefix}link5" link2="${prefix}right_finger" reason="Never" />
-      <disable_collisions link1="${prefix}link5" link2="${prefix}right_inner_knuckle" reason="Never" />
-      <disable_collisions link1="${prefix}link5" link2="${prefix}right_outer_knuckle" reason="Never" />
-      <disable_collisions link1="${prefix}link5" link2="${prefix}xarm_gripper_base_link" reason="Never" />
-      <disable_collisions link1="${prefix}link6" link2="${prefix}right_finger" reason="Never" />
-      <disable_collisions link1="${prefix}link6" link2="${prefix}right_inner_knuckle" reason="Never" />
-      <disable_collisions link1="${prefix}link6" link2="${prefix}right_outer_knuckle" reason="Never" />
-      <disable_collisions link1="${prefix}link6" link2="${prefix}xarm_gripper_base_link" reason="Never" />
-      <disable_collisions link1="${prefix}right_finger" link2="${prefix}right_inner_knuckle" reason="Default" />
-      <disable_collisions link1="${prefix}right_finger" link2="${prefix}right_outer_knuckle" reason="Adjacent" />
-      <disable_collisions link1="${prefix}right_finger" link2="${prefix}xarm_gripper_base_link" reason="Never" />
-      <disable_collisions link1="${prefix}right_inner_knuckle" link2="${prefix}right_outer_knuckle" reason="Never" />
-      <disable_collisions link1="${prefix}right_inner_knuckle" link2="${prefix}xarm_gripper_base_link" reason="Adjacent" />
-      <disable_collisions link1="${prefix}right_outer_knuckle" link2="${prefix}xarm_gripper_base_link" reason="Adjacent" />
-      <disable_collisions link1="${prefix}link_eef" link2="${prefix}xarm_gripper_base_link" reason="Adjacent" />
-      <disable_collisions link1="${prefix}link_eef" link2="${prefix}right_finger" reason="Never" />
-      <disable_collisions link1="${prefix}link_eef" link2="${prefix}right_inner_knuckle" reason="Never" />
-      <disable_collisions link1="${prefix}link_eef" link2="${prefix}right_outer_knuckle" reason="Never" />
+      <disable_collisions link1="${prefix}link5" link2="${prefix}uflite_gripper_link" reason="Never" />
+      <disable_collisions link1="${prefix}link6" link2="${prefix}uflite_gripper_link" reason="Never" />
+      <disable_collisions link1="${prefix}link_eef" link2="${prefix}uflite_gripper_link" reason="Adjacent" />
     </xacro:if>
     <!-- vacuum gripper -->
@@ -168,7 +105,7 @@
       <end_effector name="${prefix}vacuum_gripper" parent_link="${prefix}link_tcp" group="${prefix}vacuum_gripper" />
       <passive_joint name="${prefix}vacuum_gripper_fix" />
-      <disable_collisions link1="${prefix}link5" link2="${prefix}xarm_vacuum_gripper_link" reason="Never" />
-      <disable_collisions link1="${prefix}link6" link2="${prefix}xarm_vacuum_gripper_link" reason="Never" />
-      <disable_collisions link1="${prefix}link_eef" link2="${prefix}xarm_vacuum_gripper_link" reason="Adjacent" />
+      <disable_collisions link1="${prefix}link5" link2="${prefix}uflite_vacuum_gripper_link" reason="Never" />
+      <disable_collisions link1="${prefix}link6" link2="${prefix}uflite_vacuum_gripper_link" reason="Never" />
+      <disable_collisions link1="${prefix}link_eef" link2="${prefix}uflite_vacuum_gripper_link" reason="Adjacent" />
     </xacro:if>
     <!-- other box -->

File: xarm_description/urdf/lite6.urdf.xacro (robot description, xacro)
@@ -21,5 +21,5 @@
           rpy="0 0 0" />
         <mass
-          value="1.65393501783165" />
+          value="2.11" />
         <inertia
           ixx="0"
@@ -44,5 +44,5 @@
           rpy="0 0 0" />
         <geometry>
-          <mesh filename="package://xarm_description/meshes/lite6/visual/base.stl"/>
+          <mesh filename="package://xarm_description/meshes/lite6/collision/base.stl"/>
         </geometry>
       </collision>
@@ -51,8 +51,8 @@
       <inertial>
         <origin
-          xyz="-0.00036 0.03788 -0.0027"
-          rpy="0 0 0" />
-        <mass
-          value="1.169" />
+          xyz="-0.00036 0.042 -0.0025"
+          rpy="0 0 0" />
+        <mass
+          value="1.411" />
         <inertia
           ixx="1.45164E-03"
@@ -77,5 +77,5 @@
           rpy="0 0 0" />
         <geometry>
-          <mesh filename="package://xarm_description/meshes/lite6/visual/link1.stl"/>
+          <mesh filename="package://xarm_description/meshes/lite6/collision/link1.stl"/>
         </geometry>
       </collision>
@@ -83,5 +83,5 @@
     <joint name="${prefix}joint1" type="revolute">
       <origin
-        xyz="0 0 0.2435"
+        xyz="0 0 0.2433"
         rpy="0 0 0" />
       <parent
@@ -94,5 +94,5 @@
         lower="${joint1_lower_limit}"
         upper="${joint1_upper_limit}"
-        effort="50.0"
+        effort="32.0"
         velocity="3.14"/>
       <dynamics damping="1.0" friction="1.0"/>
@@ -101,8 +101,8 @@
       <inertial>
         <origin
-          xyz="0.178 0.0 0.0576"
-          rpy="0 0 0" />
-        <mass
-          value="1.192" />
+          xyz="0.179 0.0 0.0584"
+          rpy="0 0 0" />
+        <mass
+          value="1.34" />
         <inertia
           ixx="1.5854E-03"
@@ -127,5 +127,5 @@
           rpy="0 0 0" />
         <geometry>
-          <mesh filename="package://xarm_description/meshes/lite6/visual/link2.stl"/>
+          <mesh filename="package://xarm_description/meshes/lite6/collision/link2.stl"/>
         </geometry>
       </collision>
@@ -144,5 +144,5 @@
         lower="${joint2_lower_limit}"
         upper="${joint2_upper_limit}"
-        effort="50.0"
+        effort="32.0"
         velocity="3.14"/>
       <dynamics damping="1.0" friction="1.0"/>
@@ -151,8 +151,8 @@
       <inertial>
         <origin
-          xyz="0.07285 -0.030 -0.0009"
-          rpy="0 0 0" />
-        <mass
-          value="0.930" />
+          xyz="0.072 -0.036 -0.001"
+          rpy="0 0 0" />
+        <mass
+          value="0.953" />
         <inertia
           ixx="8.861E-04"
@@ -177,5 +177,5 @@
           rpy="0 0 0" />
         <geometry>
-          <mesh filename="package://xarm_description/meshes/lite6/visual/link3.stl"/>
+          <mesh filename="package://xarm_description/meshes/lite6/collision/link3.stl"/>
         </geometry>
       </collision>
@@ -183,5 +183,5 @@
     <joint name="${prefix}joint3" type="revolute">
       <origin
-        xyz="0.2002 0 0"
+        xyz="0.2 0 0"
         rpy="-3.1416 0 1.5708" />
       <parent
@@ -194,5 +194,5 @@
         lower="${joint3_lower_limit}"
         upper="${joint3_upper_limit}"
-        effort="32.0"
+        effort="18.0"
         velocity="3.14"/>
       <dynamics damping="1.0" friction="1.0"/>
@@ -201,8 +201,8 @@
       <inertial>
         <origin
-          xyz="-0.0004 -0.0275 -0.0817"
-          rpy="0 0 0" />
-        <mass
-          value="1.31" />
+          xyz="-0.002 -0.0285 -0.0813"
+          rpy="0 0 0" />
+        <mass
+          value="1.284" />
         <inertia
           ixx="3.705E-03"
@@ -227,5 +227,5 @@
           rpy="0 0 0" />
         <geometry>
-          <mesh filename="package://xarm_description/meshes/lite6/visual/link4.stl"/>
+          <mesh filename="package://xarm_description/meshes/lite6/collision/link4.stl"/>
         </geometry>
       </collision>
@@ -233,5 +233,5 @@
     <joint name="${prefix}joint4" type="revolute">
       <origin
-        xyz="0.087 -0.22761 0"
+        xyz="0.087 -0.2276 0"
         rpy="1.5708 0 0" />
       <parent
@@ -244,7 +244,7 @@
         lower="${joint4_lower_limit}"
         upper="${joint4_upper_limit}"
-        effort="32.0"
-        velocity="3.14"/>
-      <dynamics damping="1.0" friction="1.0"/>
+        effort="2.5"
+        velocity="3.14"/>
+      <dynamics damping="0.1" friction="0.1"/>
     </joint>
     <link name="${prefix}link5">
@@ -254,5 +254,5 @@
           rpy="0 0 0" />
         <mass
-          value="0.784" />
+          value="0.804" />
         <inertia
           ixx="5.668E-04"
@@ -270,12 +270,12 @@
           <mesh filename="package://xarm_description/meshes/lite6/visual/link5.stl"/>
         </geometry>
-        <material name="${prefix}White" />
-      </visual>
-      <collision>
-        <origin
-          xyz="0 0 0"
-          rpy="0 0 0" />
-        <geometry>
-          <mesh filename="package://xarm_description/meshes/lite6/visual/link5.stl"/>
+        <material name="${prefix}Silver" />
+      </visual>
+      <collision>
+        <origin
+          xyz="0 0 0"
+          rpy="0 0 0" />
+        <geometry>
+          <mesh filename="package://xarm_description/meshes/lite6/collision/link5.stl"/>
         </geometry>
       </collision>
@@ -294,7 +294,7 @@
         lower="${joint5_lower_limit}"
         upper="${joint5_upper_limit}"
-        effort="32.0"
-        velocity="3.14"/>
-      <dynamics damping="1.0" friction="1.0"/>
+        effort="2.5"
+        velocity="3.14"/>
+      <dynamics damping="0.1" friction="0.1"/>
     </joint>
     <link name="${prefix}link6">
@@ -327,5 +327,5 @@
           rpy="0 0 0" />
         <geometry>
-          <mesh filename="package://xarm_description/meshes/lite6/visual/link6.stl"/>
+          <mesh filename="package://xarm_description/meshes/lite6/collision/link6.stl"/>
         </geometry>
       </collision>
@@ -333,5 +333,5 @@
     <joint name="${prefix}joint6" type="revolute">
       <origin
-        xyz="0 0.0625 0"
+        xyz="0 0.0615 0"
         rpy="-1.5708 0 0" />
       <parent
@@ -344,7 +344,7 @@
         lower="${joint6_lower_limit}"
         upper="${joint6_upper_limit}"
-        effort="20.0"
-        velocity="3.14"/>
-      <dynamics damping="1.0" friction="1.0"/>
+        effort="2.5"
+        velocity="3.14"/>
+      <dynamics damping="0.1" friction="0.1"/>
     </joint>
     <xacro:if value="${rs_d435i}">

File: xarm_description/urdf/lite6_robot.urdf.xacro (robot description, xacro)
@@ -6,4 +6,6 @@
   <xacro:arg name="effort_control" default="false"/>
   <xacro:arg name="velocity_control" default="false"/>
+  <xacro:arg name="add_gripper" default="false"/>
+  <xacro:arg name="add_vacuum_gripper" default="false"/>
   <xacro:arg name="add_other_geometry" default="false"/>
   <xacro:arg name="geometry_type" default="box"/>
@@ -31,3 +33,13 @@
     geometry_mesh_origin_xyz="$(arg geometry_mesh_origin_xyz)" geometry_mesh_origin_rpy="$(arg geometry_mesh_origin_rpy)"
     geometry_mesh_tcp_xyz="$(arg geometry_mesh_tcp_xyz)" geometry_mesh_tcp_rpy="$(arg geometry_mesh_tcp_rpy)" />
+  <xacro:if value="$(arg add_gripper)">
+    <xacro:include filename="$(find xarm_description)/urdf/lite_gripper.urdf.xacro" />
+    <xacro:uflite_gripper_urdf attach_to="$(arg prefix)link_eef" />
+  </xacro:if>
+  <xacro:unless value="$(arg add_gripper)">
+    <xacro:if value="$(arg add_vacuum_gripper)" >
+      <xacro:include filename="$(find xarm_description)/urdf/lite_vacuum_gripper.urdf.xacro" />
+      <xacro:uflite_vacuum_gripper_urdf attach_to="$(arg prefix)link_eef" />
+    </xacro:if>
+  </xacro:unless>
 </robot>

File: xarm_description/urdf/lite6_robot_macro.xacro (robot description, xacro)
@@ -32,10 +32,10 @@
     <xacro:if value="${limited}">
       <xacro:lite6_urdf prefix="${prefix}"
-        joint1_lower_limit="${-2.0*pi}"   joint1_upper_limit="${2.0*pi}"
+        joint1_lower_limit="${-pi}"   joint1_upper_limit="${pi}"
         joint2_lower_limit="${-2.61799}"  joint2_upper_limit="${2.61799}"
         joint3_lower_limit="${-0.061087}" joint3_upper_limit="${5.235988}"
-        joint4_lower_limit="${-2.0*pi}"   joint4_upper_limit="${2.0*pi}"
+        joint4_lower_limit="${-pi}"   joint4_upper_limit="${pi}"
         joint5_lower_limit="${-2.1642}"   joint5_upper_limit="${2.1642}"
-        joint6_lower_limit="${-2.0*pi}"   joint6_upper_limit="${2.0*pi}"
+        joint6_lower_limit="${-pi}"   joint6_upper_limit="${pi}"
         rs_d435i="${rs_d435i}"/>
     </xacro:if>
