Commit message: [feat] add uf850 models

File: xarm_description/srdf/_uf850_macro.srdf.xacro (robot description, xacro)
@@ -3,5 +3,5 @@
   This is a format for representing semantic information about the robot structure.
   A URDF file must exist for this robot as well, where the joints and the links that are referenced are defined -->
-<robot xmlns:xacro="http://ros.org/wiki/xacro" name="lite6_srdf">
+<robot xmlns:xacro="http://ros.org/wiki/xacro" name="uf850_srdf">
   <!-- GROUPS: Representation of a set of joints and links. This can be useful for specifying DOF to plan for, defining arms, end effectors, etc -->
   <!-- LINKS: When a link is specified, the parent joint of that link (if it exists) is automatically included -->
@@ -9,5 +9,5 @@
   <!-- CHAINS: When a chain is specified, all the links along the chain (including endpoints) are included in the group. Additionally, all the joints that are parents to included links are also included. This means that joints along the chain and the parent joint of the base link are included in the group -->
   <!-- SUBGROUPS: Groups can also be formed by referencing to already defined group names -->
-  <xacro:macro name="lite6_macro_srdf" params="prefix=''
+  <xacro:macro name="uf850_macro_srdf" params="prefix=''
     add_gripper='false' add_vacuum_gripper='false' add_other_geometry='false' ">
     <xacro:if value="${add_gripper}">
@@ -39,5 +39,5 @@
       </xacro:unless>
     </xacro:unless>
-    <group name="${prefix}lite6">
+    <group name="${prefix}uf850">
       <joint name="${prefix}world_joint" />
       <joint name="${prefix}joint1" />
@@ -69,5 +69,5 @@
     </xacro:if>
     <!-- GROUP STATES, Purpose, Define a named state for a particular group, in terms of joint values. This is useful to define states like 'folded arms' -->
-    <group_state name="home" group="${prefix}lite6">
+    <group_state name="home" group="${prefix}uf850">
       <joint name="${prefix}joint1" value="0" />
       <joint name="${prefix}joint2" value="0" />
@@ -77,24 +77,87 @@
       <joint name="${prefix}joint6" value="0" />
     </group_state>
+    <group_state name="hold-up" group="${prefix}uf850">
+      <joint name="${prefix}joint1" value="0" />
+      <joint name="${prefix}joint2" value="0" />
+      <joint name="${prefix}joint3" value="0" />
+      <joint name="${prefix}joint4" value="0" />
+      <joint name="${prefix}joint5" value="-1.5708" />
+      <joint name="${prefix}joint6" value="0" />
+    </group_state>
     <!-- gripper -->
     <xacro:if value="${_use_gripper}">
-      <!-- <group name="${prefix}lite_gripper">
-        <link name="${prefix}uflite_gripper_link" />
+      <group name="${prefix}uf850_gripper">
+        <link name="${prefix}xarm_gripper_base_link" />
+        <link name="${prefix}left_outer_knuckle" />
+        <link name="${prefix}left_finger" />
+        <link name="${prefix}left_inner_knuckle" />
+        <link name="${prefix}right_inner_knuckle" />
+        <link name="${prefix}right_outer_knuckle" />
+        <link name="${prefix}right_finger" />
         <link name="${prefix}link_tcp" />
-        <joint name="${prefix}gripper_fix" />
-      </group> -->
-     <!--  <group_state name="open" group="${prefix}xarm_gripper">
+        <joint name="${prefix}drive_joint" />
+      </group>
+      <group_state name="open" group="${prefix}uf850_gripper">
         <joint name="${prefix}drive_joint" value="0" />
       </group_state>
-      <group_state name="close" group="${prefix}xarm_gripper">
+      <group_state name="close" group="${prefix}uf850_gripper">
         <joint name="${prefix}drive_joint" value="0.85" />
-      </group_state> -->
+      </group_state>
       <!-- END EFFECTOR, Purpose, Represent information about an end effector. -->
-      <!-- <end_effector name="${prefix}lite_gripper" parent_link="${prefix}link_tcp" group="${prefix}lite_gripper" /> -->
-      <passive_joint name="${prefix}gripper_fix" />
+      <end_effector name="${prefix}uf850_gripper" parent_link="${prefix}link_tcp" group="${prefix}uf850_gripper" />
+      <!--PASSIVE JOINT, Purpose, this element is used to mark joints that are not actuated-->
+      <passive_joint name="${prefix}left_finger_joint" />
+      <passive_joint name="${prefix}left_inner_knuckle_joint" />
+      <passive_joint name="${prefix}right_inner_knuckle_joint" />
+      <passive_joint name="${prefix}right_outer_knuckle_joint" />
+      <passive_joint name="${prefix}right_finger_joint" />
       <!-- DISABLE COLLISIONS, By default it is assumed that any link of the robot could potentially come into collision with any other link in the robot. This tag disables collision checking between a specified pair of links. -->
-      <disable_collisions link1="${prefix}link5" link2="${prefix}uflite_gripper_link" reason="Never" />
-      <disable_collisions link1="${prefix}link6" link2="${prefix}uflite_gripper_link" reason="Never" />
-      <disable_collisions link1="${prefix}link_eef" link2="${prefix}uflite_gripper_link" reason="Adjacent" />
+      <disable_collisions link1="${prefix}left_finger" link2="${prefix}left_inner_knuckle" reason="Default" />
+      <disable_collisions link1="${prefix}left_finger" link2="${prefix}left_outer_knuckle" reason="Adjacent" />
+      <disable_collisions link1="${prefix}left_finger" link2="${prefix}link4" reason="Never" />
+      <disable_collisions link1="${prefix}left_finger" link2="${prefix}link5" reason="Never" />
+      <disable_collisions link1="${prefix}left_finger" link2="${prefix}link6" reason="Never" />
+      <disable_collisions link1="${prefix}left_finger" link2="${prefix}right_finger" reason="Never" />
+      <disable_collisions link1="${prefix}left_finger" link2="${prefix}right_inner_knuckle" reason="Never" />
+      <disable_collisions link1="${prefix}left_finger" link2="${prefix}right_outer_knuckle" reason="Never" />
+      <disable_collisions link1="${prefix}left_finger" link2="${prefix}xarm_gripper_base_link" reason="Never" />
+      <disable_collisions link1="${prefix}left_inner_knuckle" link2="${prefix}left_outer_knuckle" reason="Never" />
+      <disable_collisions link1="${prefix}left_inner_knuckle" link2="${prefix}link4" reason="Never" />
+      <disable_collisions link1="${prefix}left_inner_knuckle" link2="${prefix}link5" reason="Never" />
+      <disable_collisions link1="${prefix}left_inner_knuckle" link2="${prefix}link6" reason="Never" />
+      <disable_collisions link1="${prefix}left_inner_knuckle" link2="${prefix}right_finger" reason="Never" />
+      <disable_collisions link1="${prefix}left_inner_knuckle" link2="${prefix}right_inner_knuckle" reason="Never" />
+      <disable_collisions link1="${prefix}left_inner_knuckle" link2="${prefix}right_outer_knuckle" reason="Never" />
+      <disable_collisions link1="${prefix}left_inner_knuckle" link2="${prefix}xarm_gripper_base_link" reason="Adjacent" />
+      <disable_collisions link1="${prefix}left_outer_knuckle" link2="${prefix}link5" reason="Never" />
+      <disable_collisions link1="${prefix}left_outer_knuckle" link2="${prefix}link6" reason="Never" />
+      <disable_collisions link1="${prefix}left_outer_knuckle" link2="${prefix}right_finger" reason="Never" />
+      <disable_collisions link1="${prefix}left_outer_knuckle" link2="${prefix}right_inner_knuckle" reason="Never" />
+      <disable_collisions link1="${prefix}left_outer_knuckle" link2="${prefix}right_outer_knuckle" reason="Never" />
+      <disable_collisions link1="${prefix}left_outer_knuckle" link2="${prefix}xarm_gripper_base_link" reason="Adjacent" />
+      <disable_collisions link1="${prefix}link_eef" link2="${prefix}left_finger" reason="Never" />
+      <disable_collisions link1="${prefix}link_eef" link2="${prefix}left_inner_knuckle" reason="Never" />
+      <disable_collisions link1="${prefix}link_eef" link2="${prefix}left_outer_knuckle" reason="Never" />
+      <disable_collisions link1="${prefix}link4" link2="${prefix}right_finger" reason="Never" />
+      <disable_collisions link1="${prefix}link4" link2="${prefix}right_inner_knuckle" reason="Never" />
+      <disable_collisions link1="${prefix}link5" link2="${prefix}link6" reason="Adjacent" />
+      <disable_collisions link1="${prefix}link5" link2="${prefix}right_finger" reason="Never" />
+      <disable_collisions link1="${prefix}link5" link2="${prefix}right_inner_knuckle" reason="Never" />
+      <disable_collisions link1="${prefix}link5" link2="${prefix}right_outer_knuckle" reason="Never" />
+      <disable_collisions link1="${prefix}link5" link2="${prefix}xarm_gripper_base_link" reason="Never" />
+      <disable_collisions link1="${prefix}link6" link2="${prefix}right_finger" reason="Never" />
+      <disable_collisions link1="${prefix}link6" link2="${prefix}right_inner_knuckle" reason="Never" />
+      <disable_collisions link1="${prefix}link6" link2="${prefix}right_outer_knuckle" reason="Never" />
+      <disable_collisions link1="${prefix}link6" link2="${prefix}xarm_gripper_base_link" reason="Never" />
+      <disable_collisions link1="${prefix}right_finger" link2="${prefix}right_inner_knuckle" reason="Default" />
+      <disable_collisions link1="${prefix}right_finger" link2="${prefix}right_outer_knuckle" reason="Adjacent" />
+      <disable_collisions link1="${prefix}right_finger" link2="${prefix}xarm_gripper_base_link" reason="Never" />
+      <disable_collisions link1="${prefix}right_inner_knuckle" link2="${prefix}right_outer_knuckle" reason="Never" />
+      <disable_collisions link1="${prefix}right_inner_knuckle" link2="${prefix}xarm_gripper_base_link" reason="Adjacent" />
+      <disable_collisions link1="${prefix}right_outer_knuckle" link2="${prefix}xarm_gripper_base_link" reason="Adjacent" />
+      <disable_collisions link1="${prefix}link_eef" link2="${prefix}xarm_gripper_base_link" reason="Adjacent" />
+      <disable_collisions link1="${prefix}link_eef" link2="${prefix}right_finger" reason="Never" />
+      <disable_collisions link1="${prefix}link_eef" link2="${prefix}right_inner_knuckle" reason="Never" />
+      <disable_collisions link1="${prefix}link_eef" link2="${prefix}right_outer_knuckle" reason="Never" />
     </xacro:if>
     <!-- vacuum gripper -->
@@ -105,7 +168,7 @@
       <end_effector name="${prefix}vacuum_gripper" parent_link="${prefix}link_tcp" group="${prefix}vacuum_gripper" />
       <passive_joint name="${prefix}vacuum_gripper_fix" />
-      <disable_collisions link1="${prefix}link5" link2="${prefix}uflite_vacuum_gripper_link" reason="Never" />
-      <disable_collisions link1="${prefix}link6" link2="${prefix}uflite_vacuum_gripper_link" reason="Never" />
-      <disable_collisions link1="${prefix}link_eef" link2="${prefix}uflite_vacuum_gripper_link" reason="Adjacent" />
+      <disable_collisions link1="${prefix}link5" link2="${prefix}xarm_vacuum_gripper_link" reason="Never" />
+      <disable_collisions link1="${prefix}link6" link2="${prefix}xarm_vacuum_gripper_link" reason="Never" />
+      <disable_collisions link1="${prefix}link_eef" link2="${prefix}xarm_vacuum_gripper_link" reason="Adjacent" />
     </xacro:if>
     <!-- other box -->

File: xarm_description/srdf/xarm.srdf.xacro (robot description, xacro)
@@ -1,4 +1,4 @@
 <?xml version="1.0" encoding="UTF-8"?>
-<robot xmlns:xacro="http://wiki.ros.org/xacro" name="$(arg robot_type)$(arg dof)">
+<robot xmlns:xacro="http://wiki.ros.org/xacro" name="UF_ROBOT">
   <!-- parameters -->
   <xacro:arg name="prefix" default="" />

File: xarm_description/srdf/xarm_macro.srdf.xacro (robot description, xacro)
@@ -9,4 +9,9 @@
     </xacro:if>
     <xacro:if value="${dof == 6}">
+      <xacro:if value="${robot_type == 'uf850'}">
+        <xacro:include filename="$(find xarm_description)/srdf/_uf850_macro.srdf.xacro" />
+        <xacro:uf850_macro_srdf prefix="${prefix}"
+          add_gripper="${add_gripper}" add_vacuum_gripper="${add_vacuum_gripper}" add_other_geometry="${add_other_geometry}"  />
+      </xacro:if>
       <xacro:if value="${robot_type == 'lite'}">
         <xacro:include filename="$(find xarm_description)/srdf/_lite6_macro.srdf.xacro" />
@@ -14,5 +19,5 @@
           add_gripper="${add_gripper}" add_vacuum_gripper="${add_vacuum_gripper}" add_other_geometry="${add_other_geometry}"  />
       </xacro:if>
-      <xacro:unless value="${robot_type == 'lite'}">
+      <xacro:unless value="${robot_type == 'lite' or robot_type == 'uf850'}">
         <xacro:include filename="$(find xarm_description)/srdf/_xarm6_macro.srdf.xacro" />
         <xacro:xarm6_macro_srdf prefix="${prefix}"

File: xarm_description/urdf/uf850/uf850_robot_macro.xacro (robot description, xacro)
@@ -1,5 +1,5 @@
 <?xml version="1.0"?>
-<robot xmlns:xacro="http://ros.org/wiki/xacro" name="lite6" >
-  <xacro:macro name="lite6_robot" params="
+<robot xmlns:xacro="http://ros.org/wiki/xacro" name="uf850" >
+  <xacro:macro name="uf850_robot" params="
     prefix:=''
     hw_ns:='xarm'
@@ -11,18 +11,19 @@
     robot_ip:=''
     report_type:='normal'
-    baud_checkset:=true
+    baud_checkset:='true'
     default_gripper_baud:=2000000
+    model1300:=false
     inertial_params_filename:='' "
     >
-    <!-- include lite6 relative macros: -->
+    <!-- include uf850 relative macros: -->
     <xacro:if value="${is_ros2}">
-      <xacro:include filename="$(find xarm_description)/urdf/lite6/lite6.ros2_control.xacro" />
+      <xacro:include filename="$(find xarm_description)/urdf/uf850/uf850.ros2_control.xacro" />
     </xacro:if>
-    <xacro:include filename="$(find xarm_description)/urdf/lite6/lite6.urdf.xacro" />
-    <xacro:include filename="$(find xarm_description)/urdf/lite6/lite6.transmission.xacro" />
-    <xacro:include filename="$(find xarm_description)/urdf/lite6/lite6.gazebo.xacro" />
+    <xacro:include filename="$(find xarm_description)/urdf/uf850/uf850.urdf.xacro" />
+    <xacro:include filename="$(find xarm_description)/urdf/uf850/uf850.transmission.xacro" />
+    <xacro:include filename="$(find xarm_description)/urdf/uf850/uf850.gazebo.xacro" />
     <xacro:if value="${limited}">
       <xacro:if value="${is_ros2}">
-        <xacro:lite6_ros2_control prefix="${prefix}"
+        <xacro:uf850_ros2_control prefix="${prefix}"
           velocity_control="${velocity_control}"
           ros2_control_plugin="${ros2_control_plugin}"
@@ -31,22 +32,23 @@
           baud_checkset="${baud_checkset}" default_gripper_baud="${default_gripper_baud}"
           joint1_lower_limit="${-pi*0.99}" joint1_upper_limit="${pi*0.99}"
-          joint2_lower_limit="${-2.61799}" joint2_upper_limit="${2.61799}"
-          joint3_lower_limit="${-0.061087}" joint3_upper_limit="${pi*0.99}"
+          joint2_lower_limit="${-2.3038346}" joint2_upper_limit="${2.3038346}"
+          joint3_lower_limit="${-pi*0.99}" joint3_upper_limit="${0.061087}"
           joint4_lower_limit="${-pi*0.99}" joint4_upper_limit="${pi*0.99}"
           joint5_lower_limit="${-2.1642}" joint5_upper_limit="${2.1642}"
           joint6_lower_limit="${-pi*0.99}" joint6_upper_limit="${pi*0.99}"/>
       </xacro:if>
-      <xacro:lite6_urdf prefix="${prefix}"
+      <xacro:uf850_urdf prefix="${prefix}"
         joint1_lower_limit="${-pi*0.99}" joint1_upper_limit="${pi*0.99}"
-        joint2_lower_limit="${-2.61799}" joint2_upper_limit="${2.61799}"
-        joint3_lower_limit="${-0.061087}" joint3_upper_limit="${pi*0.99}"
+        joint2_lower_limit="${-2.3038346}" joint2_upper_limit="${2.3038346}"
+        joint3_lower_limit="${-pi*0.99}" joint3_upper_limit="${0.061087}"
         joint4_lower_limit="${-pi*0.99}" joint4_upper_limit="${pi*0.99}"
         joint5_lower_limit="${-2.1642}" joint5_upper_limit="${2.1642}"
         joint6_lower_limit="${-pi*0.99}" joint6_upper_limit="${pi*0.99}"
-        inertial_params_filename="${inertial_params_filename}" />
+        model1300="${model1300}"
+        inertial_params_filename="${inertial_params_filename}"/>
     </xacro:if>
     <xacro:unless value="${limited}">
       <xacro:if value="${is_ros2}">
-        <xacro:lite6_ros2_control prefix="${prefix}" velocity_control="${velocity_control}"
+        <xacro:uf850_ros2_control prefix="${prefix}" velocity_control="${velocity_control}"
           ros2_control_plugin="${ros2_control_plugin}"
           hw_ns="${hw_ns}" add_gripper="${add_gripper}"
@@ -54,8 +56,9 @@
           baud_checkset="${baud_checkset}" default_gripper_baud="${default_gripper_baud}" />
       </xacro:if>
-      <xacro:lite6_urdf prefix="${prefix}" inertial_params_filename="${inertial_params_filename}"/>
+      <xacro:uf850_urdf prefix="${prefix}" model1300="${model1300}"
+        inertial_params_filename="${inertial_params_filename}"/>
     </xacro:unless>
-    <xacro:lite6_transmission prefix="${prefix}" hard_interface="${'EffortJointInterface' if effort_control else 'VelocityJointInterface' if velocity_control else 'PositionJointInterface'}" />
-    <xacro:lite6_gazebo prefix="${prefix}" />
+    <xacro:uf850_transmission prefix="${prefix}" hard_interface="${'EffortJointInterface' if effort_control else 'VelocityJointInterface' if velocity_control else 'PositionJointInterface'}" />
+    <xacro:uf850_gazebo prefix="${prefix}" />
   </xacro:macro>
 </robot>

File: xarm_description/urdf/xarm_device.urdf.xacro (robot description, xacro)
@@ -1,4 +1,4 @@
 <?xml version='1.0' encoding='utf-8'?>
-<robot xmlns:xacro="http://ros.org/wiki/xacro" name="$(arg robot_type)$(arg dof)">
+<robot xmlns:xacro="http://ros.org/wiki/xacro" name="UF_ROBOT">
   <xacro:arg name="prefix" default=""/>
   <xacro:arg name="hw_ns" default="xarm"/>
@@ -15,5 +15,5 @@
   <xacro:arg name="report_type" default="normal"/>
   <xacro:arg name="ros2_control_plugin" default="uf_robot_hardware/UFRobotSystemHardware"/>
-  <xacro:arg name="ros2_control_params" default="$(find xarm_controller)/config/xarm$(arg dof)_controllers.yaml"/>
+  <xacro:arg name="ros2_control_params" default=""/>
   <xacro:arg name="add_realsense_d435i" default="false"/>
   <xacro:arg name="add_d435i_links" default="true"/>

File: xarm_description/urdf/xarm_device_macro.xacro (robot description, xacro)
@@ -15,4 +15,5 @@
     attach_xyz:='0 0 0'
     attach_rpy:='0 0 0'
+    create_attach_link:=true
     ros2_control_params:=''
     load_gazebo_plugin:=false
@@ -46,9 +47,9 @@
     <xacro:common_material prefix="${prefix}"/>
     <!-- Specify Mesh file path -->
-    <xacro:if value="${ros2_control_plugin == 'gazebo_ros2_control/GazeboSystem'}">
+    <xacro:if value="${ros2_control_plugin == 'gazebo_ros2_control/GazeboSystem' or ros2_control_plugin == 'ign_ros2_control/IgnitionSystem'}">
       <!-- gazebo use -->
       <xacro:property name="mesh_path" value="file://$(find xarm_description)/meshes" scope="parent"/>
     </xacro:if>
-    <xacro:unless value="${ros2_control_plugin == 'gazebo_ros2_control/GazeboSystem'}">
+    <xacro:unless value="${ros2_control_plugin == 'gazebo_ros2_control/GazeboSystem' or ros2_control_plugin == 'ign_ros2_control/IgnitionSystem'}">
       <xacro:property name="mesh_path" value="package://xarm_description/meshes" scope="parent"/>
     </xacro:unless>
@@ -59,5 +60,5 @@
     <xacro:property name="new_model1300" value="${scope_parent_model1300}"/>
     <!-- add one world link if no 'attach_to' specified  -->
-    <xacro:if value="${attach_to == 'world'}">
+    <xacro:if value="${attach_to == 'world' and create_attach_link}">
       <link name="world" />
     </xacro:if>
@@ -82,4 +83,18 @@
     </xacro:if>
     <xacro:if value="${dof == 6}">
+      <xacro:if value="${robot_type == 'uf850'}">
+        <!-- Load UFACTORY 850 Robot Model URDF -->
+        <xacro:include filename="$(find xarm_description)/urdf/uf850/uf850_robot_macro.xacro" />
+        <xacro:uf850_robot prefix="${prefix}" hw_ns="${hw_ns}" limited="${limited}"
+          effort_control="${effort_control}" velocity_control="${velocity_control}"
+          ros2_control_plugin="${ros2_control_plugin}"
+          add_gripper="${add_gripper}"
+          robot_ip="${robot_ip}"
+          report_type="${report_type}"
+          baud_checkset="${baud_checkset}"
+          default_gripper_baud="${default_gripper_baud}"
+          model1300="${new_model1300}"
+          inertial_params_filename="${inertial_params_filename}" />
+      </xacro:if>
       <xacro:if value="${robot_type == 'lite'}">
         <!-- Load Lite6 Robot Model URDF -->
@@ -95,5 +110,5 @@
           inertial_params_filename="${inertial_params_filename}" />
       </xacro:if>
-      <xacro:unless value="${robot_type == 'lite'}">
+      <xacro:unless value="${robot_type == 'lite' or robot_type == 'uf850'}">
         <!-- Load XArm6 Robot Model URDF -->
         <xacro:include filename="$(find xarm_description)/urdf/xarm6/xarm6_robot_macro.xacro" />
@@ -182,5 +197,19 @@
       <xacro:include filename="$(find xarm_description)/urdf/common/common.gazebo.xacro" />
       <xacro:if value="${is_ros2}">
-        <xacro:gazebo_ros2_control_plugin ros2_control_params="${ros2_control_params}"/>
+        <xacro:if value="${robot_type == 'uf850'}">
+          <xacro:property name="new_ros2_control_params" value="$(find xarm_controller)/config/${robot_type}_controllers.yaml"/>
+        </xacro:if>
+        <xacro:unless value="${robot_type == 'uf850'}">
+          <xacro:property name="new_ros2_control_params" value="$(find xarm_controller)/config/${robot_type}${dof}_controllers.yaml"/>
+        </xacro:unless>
+        <xacro:if value="${ros2_control_params != ''}">
+          <xacro:property name="new_ros2_control_params" value="${ros2_control_params}"/>
+        </xacro:if>
+        <xacro:if value="${ros2_control_plugin == 'ign_ros2_control/IgnitionSystem'}">
+          <xacro:ignition_ros2_control_plugin prefix="${prefix}" ros2_control_params="${new_ros2_control_params}"/>
+        </xacro:if>
+        <xacro:unless value="${ros2_control_plugin == 'ign_ros2_control/IgnitionSystem'}">
+          <xacro:gazebo_ros2_control_plugin ros2_control_params="${new_ros2_control_params}"/>
+        </xacro:unless>
       </xacro:if>
       <xacro:unless value="${is_ros2}">

Commit message: [fix] fix group hold-up of uf850

File: xarm_description/srdf/_uf850_macro.srdf.xacro (robot description, xacro)
@@ -82,5 +82,5 @@
       <joint name="${prefix}joint3" value="0" />
       <joint name="${prefix}joint4" value="0" />
-      <joint name="${prefix}joint5" value="-1.5708" />
+      <joint name="${prefix}joint5" value="1.5708" />
       <joint name="${prefix}joint6" value="0" />
     </group_state>
