Commit message: [fix] URDF syntax compatible

File: xarm_description/urdf/gripper/xarm_gripper.gazebo.xacro (robot description, xacro)
@@ -3,6 +3,15 @@
   <!-- from mimic_joint_gazebo_tutorial by @mintar, refer: https://github.com/mintar/mimic_joint_gazebo_tutorial -->
   <xacro:macro name="mimic_joint_plugin_gazebo" params="name_prefix following_joint mimic_joint has_pid:=false multiplier:=1.0 offset:=0 sensitiveness:=0.0 max_effort:=1.0 robot_namespace:=''">
+    <!-- ros2 -->
+    <xacro:if value="${is_ros2}">
+      <xacro:property name="filename" value="libgazebo_mimic_joint_plugin.so" />
+    </xacro:if>
+    <!-- ros1 -->
+    <xacro:unless value="${is_ros2}">
+      <xacro:property name="filename" value="libroboticsgroup_gazebo_mimic_joint_plugin.so" />
+      <!-- <xacro:property name="filename" value="libroboticsgroup_upatras_gazebo_mimic_joint_plugin.so" /> -->
+    </xacro:unless>
     <gazebo>
-      <plugin name="${name_prefix}mimic_joint_plugin" filename="$(eval 'libgazebo_mimic_joint_plugin.so' if ${is_ros2} else 'libroboticsgroup_gazebo_mimic_joint_plugin.so')">
+      <plugin name="${name_prefix}mimic_joint_plugin" filename="${filename}">
         <joint>${following_joint}</joint>
         <mimicJoint>${mimic_joint}</mimicJoint>

File: xarm_description/urdf/gripper/xarm_gripper_macro.xacro (robot description, xacro)
@@ -6,11 +6,11 @@
   <xacro:include filename="$(find xarm_description)/urdf/gripper/xarm_gripper.transmission.xacro" />
   <xacro:include filename="$(find xarm_description)/urdf/gripper/xarm_gripper.gazebo.xacro" />
-  <xacro:macro name="xarm_gripper_macro" params="prefix:='' attach_to:='' ns:='xarm' attach_xyz:='0 0 0' attach_rpy:='0 0 0' effort_control:='false' velocity_control:='false'
-    ros2_control_plugin:='uf_robot_hardware/UFRobotFakeSystemHardware' dof:=7 ">
+  <xacro:macro name="xarm_gripper_macro" params="prefix:='' attach_to:='' ns:='xarm' attach_xyz:='0 0 0' attach_rpy:='0 0 0'
+    ros2_control_plugin:='uf_robot_hardware/UFRobotFakeSystemHardware' dof:=7 hard_interface:='PositionJointInterface' ">
     <xacro:if value="${is_ros2 and ros2_control_plugin != 'uf_robot_hardware/UFRobotSystemHardware'}">
       <xacro:xarm_gripper_ros2_control prefix="${prefix}" ros2_control_plugin="${ros2_control_plugin}" />
     </xacro:if>
     <xacro:xarm_gripper_urdf prefix="${prefix}" attach_to="${attach_to}" attach_xyz="${attach_xyz}" attach_rpy="${attach_rpy}" />
-    <xacro:xarm_gripper_transmission prefix="${prefix}" hard_interface="$(eval 'EffortJointInterface' if ${effort_control} else 'VelocityJointInterface' if ${velocity_control} else 'PositionJointInterface')" />
+    <xacro:xarm_gripper_transmission prefix="${prefix}" hard_interface="${hard_interface}" />
     <xacro:xarm_gripper_gazebo prefix="${prefix}" />
     <xacro:if value="${not is_ros2}">

File: xarm_description/urdf/lite6/lite6_robot_macro.xacro (robot description, xacro)
@@ -5,5 +5,4 @@
     hw_ns:='xarm'
     limited:=false
-    effort_control:=false
     velocity_control:=false
     add_gripper:=false
@@ -13,5 +12,6 @@
     baud_checkset:=true
     default_gripper_baud:=2000000
-    inertial_params_filename:='' "
+    inertial_params_filename:=''
+    hard_interface:='PositionJointInterface' "
     >
     <!-- include lite6 relative macros: -->
@@ -56,5 +56,5 @@
       <xacro:lite6_urdf prefix="${prefix}" inertial_params_filename="${inertial_params_filename}"/>
     </xacro:unless>
-    <xacro:lite6_transmission prefix="${prefix}" hard_interface="$(eval 'EffortJointInterface' if ${effort_control} else 'VelocityJointInterface' if ${velocity_control} else 'PositionJointInterface')" />
+    <xacro:lite6_transmission prefix="${prefix}" hard_interface="${hard_interface}" />
     <xacro:lite6_gazebo prefix="${prefix}" />
   </xacro:macro>

File: xarm_description/urdf/uf850/uf850_robot_macro.xacro (robot description, xacro)
@@ -5,5 +5,4 @@
     hw_ns:='xarm'
     limited:=false
-    effort_control:=false
     velocity_control:=false
     add_gripper:=false
@@ -14,5 +13,6 @@
     default_gripper_baud:=2000000
     model1300:=false
-    inertial_params_filename:='' "
+    inertial_params_filename:=''
+    hard_interface:='PositionJointInterface' "
     >
     <!-- include uf850 relative macros: -->
@@ -59,5 +59,5 @@
         inertial_params_filename="${inertial_params_filename}"/>
     </xacro:unless>
-    <xacro:uf850_transmission prefix="${prefix}" hard_interface="$(eval 'EffortJointInterface' if ${effort_control} else 'VelocityJointInterface' if ${velocity_control} else 'PositionJointInterface')" />
+    <xacro:uf850_transmission prefix="${prefix}" hard_interface="${hard_interface}" />
     <xacro:uf850_gazebo prefix="${prefix}" />
   </xacro:macro>

File: xarm_description/urdf/xarm5/xarm5_robot_macro.xacro (robot description, xacro)
@@ -5,5 +5,4 @@
     hw_ns:='xarm'
     limited:=false
-    effort_control:=false
     velocity_control:=false
     add_gripper:=false
@@ -14,5 +13,6 @@
     default_gripper_baud:=2000000
     model1300:=false
-    inertial_params_filename:='' "
+    inertial_params_filename:=''
+    hard_interface:='PositionJointInterface' "
     >
     <!-- include xarm5 relative macros: -->
@@ -57,5 +57,5 @@
         inertial_params_filename="${inertial_params_filename}"/>
     </xacro:unless>
-    <xacro:xarm5_transmission prefix="${prefix}" hard_interface="$(eval 'EffortJointInterface' if ${effort_control} else 'VelocityJointInterface' if ${velocity_control} else 'PositionJointInterface')" />
+    <xacro:xarm5_transmission prefix="${prefix}" hard_interface="${hard_interface}" />
     <xacro:xarm5_gazebo prefix="${prefix}" />
   </xacro:macro>

File: xarm_description/urdf/xarm6/xarm6_robot_macro.xacro (robot description, xacro)
@@ -5,5 +5,4 @@
     hw_ns:='xarm'
     limited:=false
-    effort_control:=false
     velocity_control:=false
     add_gripper:=false
@@ -14,5 +13,6 @@
     default_gripper_baud:=2000000
     model1300:=false
-    inertial_params_filename:='' "
+    inertial_params_filename:=''
+    hard_interface:='PositionJointInterface' "
     >
     <!-- include xarm6 relative macros: -->
@@ -59,5 +59,5 @@
         inertial_params_filename="${inertial_params_filename}"/>
     </xacro:unless>
-    <xacro:xarm6_transmission prefix="${prefix}" hard_interface="$(eval 'EffortJointInterface' if ${effort_control} else 'VelocityJointInterface' if ${velocity_control} else 'PositionJointInterface')" />
+    <xacro:xarm6_transmission prefix="${prefix}" hard_interface="${hard_interface}" />
     <xacro:xarm6_gazebo prefix="${prefix}" />
   </xacro:macro>

File: xarm_description/urdf/xarm7/xarm7_robot_macro.xacro (robot description, xacro)
@@ -5,5 +5,4 @@
     hw_ns:='xarm'
     limited:=false
-    effort_control:=false
     velocity_control:=false
     add_gripper:=false
@@ -14,5 +13,6 @@
     default_gripper_baud:=2000000
     model1300:=false
-    inertial_params_filename:='' "
+    inertial_params_filename:=''
+    hard_interface:='PositionJointInterface' "
     >
     <!-- xarm7 -->
@@ -61,5 +61,5 @@
         inertial_params_filename="${inertial_params_filename}"/>
     </xacro:unless>
-    <xacro:xarm7_transmission prefix="${prefix}" hard_interface="$(eval 'EffortJointInterface' if ${effort_control} else 'VelocityJointInterface' if ${velocity_control} else 'PositionJointInterface')" />
+    <xacro:xarm7_transmission prefix="${prefix}" hard_interface="${hard_interface}" />
     <xacro:xarm7_gazebo prefix="${prefix}" />
   </xacro:macro>
