Commit message: [fix] URDF syntax compatible

File: xarm_description/urdf/lite6/lite6_robot_macro.xacro (robot description, xacro)
@@ -5,5 +5,4 @@
     hw_ns:='xarm'
     limited:=false
-    effort_control:=false
     velocity_control:=false
     add_gripper:=false
@@ -13,5 +12,6 @@
     baud_checkset:=true
     default_gripper_baud:=2000000
-    inertial_params_filename:='' "
+    inertial_params_filename:=''
+    hard_interface:='PositionJointInterface' "
     >
     <!-- include lite6 relative macros: -->
@@ -56,5 +56,5 @@
       <xacro:lite6_urdf prefix="${prefix}" inertial_params_filename="${inertial_params_filename}"/>
     </xacro:unless>
-    <xacro:lite6_transmission prefix="${prefix}" hard_interface="${'EffortJointInterface' if effort_control else 'VelocityJointInterface' if velocity_control else 'PositionJointInterface'}" />
+    <xacro:lite6_transmission prefix="${prefix}" hard_interface="${hard_interface}" />
     <xacro:lite6_gazebo prefix="${prefix}" />
   </xacro:macro>

File: xarm_description/urdf/uf850/uf850_robot_macro.xacro (robot description, xacro)
@@ -5,5 +5,4 @@
     hw_ns:='xarm'
     limited:=false
-    effort_control:=false
     velocity_control:=false
     add_gripper:=false
@@ -14,5 +13,6 @@
     default_gripper_baud:=2000000
     model1300:=false
-    inertial_params_filename:='' "
+    inertial_params_filename:=''
+    hard_interface:='PositionJointInterface' "
     >
     <!-- include uf850 relative macros: -->
@@ -59,5 +59,5 @@
         inertial_params_filename="${inertial_params_filename}"/>
     </xacro:unless>
-    <xacro:uf850_transmission prefix="${prefix}" hard_interface="${'EffortJointInterface' if effort_control else 'VelocityJointInterface' if velocity_control else 'PositionJointInterface'}" />
+    <xacro:uf850_transmission prefix="${prefix}" hard_interface="${hard_interface}" />
     <xacro:uf850_gazebo prefix="${prefix}" />
   </xacro:macro>

File: xarm_description/urdf/xarm_device_macro.xacro (robot description, xacro)
@@ -68,9 +68,20 @@
       <origin xyz="${attach_xyz}" rpy="${attach_rpy}" />
     </joint>
+    <xacro:if value="${effort_control}">
+      <xacro:property name="hard_interface" value="EffortJointInterface" />
+    </xacro:if>
+    <xacro:unless value="${effort_control}">
+      <xacro:if value="${velocity_control}">
+        <xacro:property name="hard_interface" value="VelocityJointInterface" />
+      </xacro:if>
+      <xacro:unless value="${velocity_control}">
+        <xacro:property name="hard_interface" value="PositionJointInterface" />
+      </xacro:unless>
+    </xacro:unless>
     <xacro:if value="${dof == 5}">
       <!-- Load XArm5 Robot Model URDF -->
       <xacro:include filename="$(find xarm_description)/urdf/xarm5/xarm5_robot_macro.xacro" />
       <xacro:xarm5_robot prefix="${prefix}" hw_ns="${hw_ns}" limited="${limited}"
-        effort_control="${effort_control}" velocity_control="${velocity_control}"
+        velocity_control="${velocity_control}"
         ros2_control_plugin="${ros2_control_plugin}"
         add_gripper="${add_gripper}"
@@ -80,5 +91,6 @@
         default_gripper_baud="${default_gripper_baud}"
         model1300="${new_model1300}"
-        inertial_params_filename="${inertial_params_filename}" />
+        inertial_params_filename="${inertial_params_filename}"
+        hard_interface="${hard_interface}" />
     </xacro:if>
     <xacro:if value="${dof == 6}">
@@ -87,5 +99,5 @@
         <xacro:include filename="$(find xarm_description)/urdf/uf850/uf850_robot_macro.xacro" />
         <xacro:uf850_robot prefix="${prefix}" hw_ns="${hw_ns}" limited="${limited}"
-          effort_control="${effort_control}" velocity_control="${velocity_control}"
+          velocity_control="${velocity_control}"
           ros2_control_plugin="${ros2_control_plugin}"
           add_gripper="${add_gripper}"
@@ -95,5 +107,6 @@
           default_gripper_baud="${default_gripper_baud}"
           model1300="${new_model1300}"
-          inertial_params_filename="${inertial_params_filename}" />
+          inertial_params_filename="${inertial_params_filename}"
+          hard_interface="${hard_interface}" />
       </xacro:if>
       <xacro:if value="${robot_type == 'lite'}">
@@ -101,5 +114,5 @@
         <xacro:include filename="$(find xarm_description)/urdf/lite6/lite6_robot_macro.xacro" />
         <xacro:lite6_robot prefix="${prefix}" hw_ns="${hw_ns}" limited="${limited}"
-          effort_control="${effort_control}" velocity_control="${velocity_control}"
+          velocity_control="${velocity_control}"
           ros2_control_plugin="${ros2_control_plugin}"
           add_gripper="${add_gripper}"
@@ -108,5 +121,6 @@
           baud_checkset="${baud_checkset}"
           default_gripper_baud="${default_gripper_baud}"
-          inertial_params_filename="${inertial_params_filename}" />
+          inertial_params_filename="${inertial_params_filename}"
+          hard_interface="${hard_interface}" />
       </xacro:if>
       <xacro:unless value="${robot_type == 'lite' or robot_type == 'uf850'}">
@@ -114,5 +128,5 @@
         <xacro:include filename="$(find xarm_description)/urdf/xarm6/xarm6_robot_macro.xacro" />
         <xacro:xarm6_robot prefix="${prefix}" hw_ns="${hw_ns}" limited="${limited}"
-          effort_control="${effort_control}" velocity_control="${velocity_control}"
+          velocity_control="${velocity_control}"
           ros2_control_plugin="${ros2_control_plugin}"
           add_gripper="${add_gripper}"
@@ -122,5 +136,6 @@
           default_gripper_baud="${default_gripper_baud}"
           model1300="${new_model1300}"
-          inertial_params_filename="${inertial_params_filename}" />
+          inertial_params_filename="${inertial_params_filename}"
+          hard_interface="${hard_interface}" />
       </xacro:unless>
     </xacro:if>
@@ -129,5 +144,5 @@
       <xacro:include filename="$(find xarm_description)/urdf/xarm7/xarm7_robot_macro.xacro" />
       <xacro:xarm7_robot prefix="${prefix}" hw_ns="${hw_ns}" limited="${limited}"
-        effort_control="${effort_control}" velocity_control="${velocity_control}"
+        velocity_control="${velocity_control}"
         ros2_control_plugin="${ros2_control_plugin}"
         add_gripper="${add_gripper}"
@@ -137,5 +152,6 @@
         default_gripper_baud="${default_gripper_baud}"
         model1300="${new_model1300}"
-        inertial_params_filename="${inertial_params_filename}" />
+        inertial_params_filename="${inertial_params_filename}"
+        hard_interface="${hard_interface}" />
     </xacro:unless>
     <xacro:if value="${add_realsense_d435i}">
@@ -165,6 +181,6 @@
         <!-- Load XArm Gripper Model URDF -->
         <xacro:include filename="$(find xarm_description)/urdf/gripper/xarm_gripper_macro.xacro" />
-        <xacro:xarm_gripper_macro prefix="${prefix}" attach_to="${prefix}link_eef" effort_control="${effort_control}" velocity_control="${velocity_control}"
-          ros2_control_plugin="${ros2_control_plugin}" dof="${dof}" />
+        <xacro:xarm_gripper_macro prefix="${prefix}" attach_to="${prefix}link_eef"
+          ros2_control_plugin="${ros2_control_plugin}" dof="${dof}" hard_interface="${hard_interface}" />
       </xacro:unless>
     </xacro:if>
@@ -178,5 +194,5 @@
         <!-- Load XArm Vacuum Gripper Model URDF -->
         <xacro:include filename="$(find xarm_description)/urdf/vacuum_gripper/xarm_vacuum_gripper.urdf.xacro" />
-        <xacro:xarm_vacuum_gripper_urdf prefix="${prefix}" attach_to="${prefix}link_eef" effort_control="${effort_control}" velocity_control="${velocity_control}" />
+        <xacro:xarm_vacuum_gripper_urdf prefix="${prefix}" attach_to="${prefix}link_eef" />
       </xacro:unless>
     </xacro:if>
