Commit message: [fix] (urdf) update the effort limit

File: xarm_description/urdf/lite6/lite6.urdf.xacro (robot description, xacro)
@@ -15,4 +15,5 @@
     <xacro:property name="collison_mesh_suffix" value="stl"/>
     <!-- load params and define property -->
+    <xacro:property name="joint_limits_params_filename" value="$(find xarm_description)/config/lite6/joint_limits.yaml"/>
     <xacro:property name="default_inertial_params_filename" value="xarm6_type9_HT_BR2"/>
     <xacro:if value="${inertial_params_filename != ''}">
@@ -25,10 +26,13 @@
       <xacro:property name="inertial_params" value="${xacro.load_yaml(link_inertial_params_file)}"/>
       <xacro:property name="kinematics_config" value="${xacro.load_yaml(kinematics_params_filename)}"/>
+      <xacro:property name="joint_limits_config" value="${xacro.load_yaml(joint_limits_params_filename)}"/>
     </xacro:if>
     <xacro:unless value="${use_xacro_load_yaml}">
       <xacro:property name="inertial_params" value="${load_yaml(link_inertial_params_file)}"/>
       <xacro:property name="kinematics_config" value="${load_yaml(kinematics_params_filename)}"/>
+      <xacro:property name="joint_limits_config" value="${load_yaml(joint_limits_params_filename)}"/>
     </xacro:unless>
     <xacro:property name="kinematics_params" value="${kinematics_config['kinematics']}"/>
+    <xacro:property name="joint_limits" value="${joint_limits_config['joint_limits']}"/>
     <link name="${prefix}link_base">
       <inertial>
@@ -76,5 +80,5 @@
         lower="${joint1_lower_limit}"
         upper="${joint1_upper_limit}"
-        effort="50.0"
+        effort="${joint_limits['joint1']['max_effort']}"
         velocity="3.14"/>
       <dynamics damping="1.0" friction="1.0"/>
@@ -105,5 +109,5 @@
         lower="${joint2_lower_limit}"
         upper="${joint2_upper_limit}"
-        effort="50.0"
+        effort="${joint_limits['joint2']['max_effort']}"
         velocity="3.14"/>
       <dynamics damping="1.0" friction="1.0"/>
@@ -134,5 +138,5 @@
         lower="${joint3_lower_limit}"
         upper="${joint3_upper_limit}"
-        effort="32.0"
+        effort="${joint_limits['joint3']['max_effort']}"
         velocity="3.14"/>
       <dynamics damping="1.0" friction="1.0"/>
@@ -163,5 +167,5 @@
         lower="${joint4_lower_limit}"
         upper="${joint4_upper_limit}"
-        effort="32.0"
+        effort="${joint_limits['joint4']['max_effort']}"
         velocity="3.14"/>
       <dynamics damping="1.0" friction="1.0"/>
@@ -192,5 +196,5 @@
         lower="${joint5_lower_limit}"
         upper="${joint5_upper_limit}"
-        effort="32.0"
+        effort="${joint_limits['joint5']['max_effort']}"
         velocity="3.14"/>
       <dynamics damping="1.0" friction="1.0"/>
@@ -221,5 +225,5 @@
         lower="${joint6_lower_limit}"
         upper="${joint6_upper_limit}"
-        effort="20.0"
+        effort="${joint_limits['joint6']['max_effort']}"
         velocity="3.14"/>
       <dynamics damping="1.0" friction="1.0"/>

File: xarm_description/urdf/uf850/uf850.urdf.xacro (robot description, xacro)
@@ -15,4 +15,5 @@
     <xacro:property name="collison_mesh_suffix" value="stl"/>
     <!-- load params and define property -->
+    <xacro:property name="joint_limits_params_filename" value="$(find xarm_description)/config/uf850/joint_limits.yaml"/>
     <xacro:property name="default_inertial_params_filename" value="xarm6_type12_HT_LDBR2"/>
     <xacro:if value="${inertial_params_filename != ''}">
@@ -25,10 +26,13 @@
       <xacro:property name="inertial_params" value="${xacro.load_yaml(link_inertial_params_file)}"/>
       <xacro:property name="kinematics_config" value="${xacro.load_yaml(kinematics_params_filename)}"/>
+      <xacro:property name="joint_limits_config" value="${xacro.load_yaml(joint_limits_params_filename)}"/>
     </xacro:if>
     <xacro:unless value="${use_xacro_load_yaml}">
       <xacro:property name="inertial_params" value="${load_yaml(link_inertial_params_file)}"/>
       <xacro:property name="kinematics_config" value="${load_yaml(kinematics_params_filename)}"/>
+      <xacro:property name="joint_limits_config" value="${load_yaml(joint_limits_params_filename)}"/>
     </xacro:unless>
     <xacro:property name="kinematics_params" value="${kinematics_config['kinematics']}"/>
+    <xacro:property name="joint_limits" value="${joint_limits_config['joint_limits']}"/>
     <link name="${prefix}link_base">
       <inertial>
@@ -76,5 +80,5 @@
         lower="${joint1_lower_limit}"
         upper="${joint1_upper_limit}"
-        effort="200.0"
+        effort="${joint_limits['joint1']['max_effort']}"
         velocity="3.14"/>
       <dynamics damping="16.6" friction="9.6"/>
@@ -105,5 +109,5 @@
         lower="${joint2_lower_limit}"
         upper="${joint2_upper_limit}"
-        effort="200.0"
+        effort="${joint_limits['joint2']['max_effort']}"
         velocity="3.14"/>
       <dynamics damping="12.5" friction="12.1"/>
@@ -134,5 +138,5 @@
         lower="${joint3_lower_limit}"
         upper="${joint3_upper_limit}"
-        effort="90.0"
+        effort="${joint_limits['joint3']['max_effort']}"
         velocity="3.14"/>
       <dynamics damping="4.0" friction="5.5"/>
@@ -163,5 +167,5 @@
         lower="${joint4_lower_limit}"
         upper="${joint4_upper_limit}"
-        effort="68.0"
+        effort="${joint_limits['joint4']['max_effort']}"
         velocity="3.14"/>
       <dynamics damping="3.6" friction="2.2"/>
@@ -192,5 +196,5 @@
         lower="${joint5_lower_limit}"
         upper="${joint5_upper_limit}"
-        effort="19.0"
+        effort="${joint_limits['joint5']['max_effort']}"
         velocity="3.14"/>
       <dynamics damping="3.45" friction="3.2"/>
@@ -221,5 +225,5 @@
         lower="${joint6_lower_limit}"
         upper="${joint6_upper_limit}"
-        effort="19.0"
+        effort="${joint_limits['joint6']['max_effort']}"
         velocity="3.14"/>
       <dynamics damping="3.4" friction="1.1"/>

File: xarm_description/urdf/xarm5/xarm5.urdf.xacro (robot description, xacro)
@@ -33,4 +33,10 @@
       </xacro:unless>
     </xacro:unless>
+    <xacro:if value="${model_num >= 1305}">
+      <xacro:property name="joint_limits_params_filename" value="$(find xarm_description)/config/xarm5/joint_limits_1305.yaml"/>
+    </xacro:if>
+    <xacro:unless value="${model_num >= 1305}">
+      <xacro:property name="joint_limits_params_filename" value="$(find xarm_description)/config/xarm5/joint_limits.yaml"/>
+    </xacro:unless>
     <!-- load params and define property -->
     <xacro:property name="default_inertial_params_filename" value="xarm5_type5_HT_BR2"/>
@@ -44,10 +50,13 @@
       <xacro:property name="inertial_params" value="${xacro.load_yaml(link_inertial_params_file)}"/>
       <xacro:property name="kinematics_config" value="${xacro.load_yaml(kinematics_params_filename)}"/>
+      <xacro:property name="joint_limits_config" value="${xacro.load_yaml(joint_limits_params_filename)}"/>
     </xacro:if>
     <xacro:unless value="${use_xacro_load_yaml}">
       <xacro:property name="inertial_params" value="${load_yaml(link_inertial_params_file)}"/>
       <xacro:property name="kinematics_config" value="${load_yaml(kinematics_params_filename)}"/>
+      <xacro:property name="joint_limits_config" value="${load_yaml(joint_limits_params_filename)}"/>
     </xacro:unless>
     <xacro:property name="kinematics_params" value="${kinematics_config['kinematics']}"/>
+    <xacro:property name="joint_limits" value="${joint_limits_config['joint_limits']}"/>
     <link name="${prefix}link_base">
       <inertial>
@@ -95,5 +104,5 @@
         lower="${joint1_lower_limit}"
         upper="${joint1_upper_limit}"
-        effort="50"
+        effort="${joint_limits['joint1']['max_effort']}"
         velocity="3.14" />
       <dynamics damping="10" friction="1" />
@@ -124,5 +133,5 @@
         lower="${joint2_lower_limit}"
         upper="${joint2_upper_limit}"
-        effort="50"
+        effort="${joint_limits['joint2']['max_effort']}"
         velocity="3.14" />
       <dynamics damping="10" friction="1" />
@@ -153,5 +162,5 @@
         lower="${joint3_lower_limit}"
         upper="${joint3_upper_limit}"
-        effort="30"
+        effort="${joint_limits['joint3']['max_effort']}"
         velocity="3.14" />
       <dynamics damping="5" friction="1" />
@@ -182,5 +191,5 @@
         lower="${joint4_lower_limit}"
         upper="${joint4_upper_limit}"
-        effort="20"
+        effort="${joint_limits['joint4']['max_effort']}"
         velocity="3.14" />
       <dynamics damping="3" friction="1" />
@@ -211,5 +220,5 @@
         lower="${joint5_lower_limit}"
         upper="${joint5_upper_limit}"
-        effort="20"
+        effort="${joint_limits['joint5']['max_effort']}"
         velocity="3.14" />
       <dynamics damping="3" friction="1" />

File: xarm_description/urdf/xarm6/xarm6.urdf.xacro (robot description, xacro)
@@ -34,4 +34,10 @@
       </xacro:unless>
     </xacro:unless>
+    <xacro:if value="${model_num >= 1305}">
+      <xacro:property name="joint_limits_params_filename" value="$(find xarm_description)/config/xarm6/joint_limits_1305.yaml"/>
+    </xacro:if>
+    <xacro:unless value="${model_num >= 1305}">
+      <xacro:property name="joint_limits_params_filename" value="$(find xarm_description)/config/xarm6/joint_limits.yaml"/>
+    </xacro:unless>
     <!-- load params and define property -->
     <xacro:property name="default_inertial_params_filename" value="xarm6_type6_HT_BR2"/>
@@ -45,10 +51,13 @@
       <xacro:property name="inertial_params" value="${xacro.load_yaml(link_inertial_params_file)}"/>
       <xacro:property name="kinematics_config" value="${xacro.load_yaml(kinematics_params_filename)}"/>
+      <xacro:property name="joint_limits_config" value="${xacro.load_yaml(joint_limits_params_filename)}"/>
     </xacro:if>
     <xacro:unless value="${use_xacro_load_yaml}">
       <xacro:property name="inertial_params" value="${load_yaml(link_inertial_params_file)}"/>
       <xacro:property name="kinematics_config" value="${load_yaml(kinematics_params_filename)}"/>
+      <xacro:property name="joint_limits_config" value="${load_yaml(joint_limits_params_filename)}"/>
     </xacro:unless>
     <xacro:property name="kinematics_params" value="${kinematics_config['kinematics']}"/>
+    <xacro:property name="joint_limits" value="${joint_limits_config['joint_limits']}"/>
     <link name="${prefix}link_base">
       <inertial>
@@ -96,5 +105,5 @@
         lower="${joint1_lower_limit}"
         upper="${joint1_upper_limit}"
-        effort="50.0"
+        effort="${joint_limits['joint1']['max_effort']}"
         velocity="3.14"/>
       <dynamics damping="1.0" friction="1.0"/>
@@ -125,5 +134,5 @@
         lower="${joint2_lower_limit}"
         upper="${joint2_upper_limit}"
-        effort="50.0"
+        effort="${joint_limits['joint2']['max_effort']}"
         velocity="3.14"/>
       <dynamics damping="1.0" friction="1.0"/>
@@ -154,5 +163,5 @@
         lower="${joint3_lower_limit}"
         upper="${joint3_upper_limit}"
-        effort="32.0"
+        effort="${joint_limits['joint3']['max_effort']}"
         velocity="3.14"/>
       <dynamics damping="1.0" friction="1.0"/>
@@ -183,5 +192,5 @@
         lower="${joint4_lower_limit}"
         upper="${joint4_upper_limit}"
-        effort="32.0"
+        effort="${joint_limits['joint4']['max_effort']}"
         velocity="3.14"/>
       <dynamics damping="1.0" friction="1.0"/>
@@ -211,5 +220,5 @@
         lower="${joint5_lower_limit}"
         upper="${joint5_upper_limit}"
-        effort="32.0"
+        effort="${joint_limits['joint5']['max_effort']}"
         velocity="3.14"/>
       <dynamics damping="1.0" friction="1.0"/>
@@ -240,5 +249,5 @@
         lower="${joint6_lower_limit}"
         upper="${joint6_upper_limit}"
-        effort="20.0"
+        effort="${joint_limits['joint6']['max_effort']}"
         velocity="3.14"/>
       <dynamics damping="1.0" friction="1.0"/>

File: xarm_description/urdf/xarm7/xarm7.urdf.xacro (robot description, xacro)
@@ -35,4 +35,10 @@
       </xacro:unless>
     </xacro:unless>
+    <xacro:if value="${model_num >= 1305}">
+      <xacro:property name="joint_limits_params_filename" value="$(find xarm_description)/config/xarm7/joint_limits_1305.yaml"/>
+    </xacro:if>
+    <xacro:unless value="${model_num >= 1305}">
+      <xacro:property name="joint_limits_params_filename" value="$(find xarm_description)/config/xarm7/joint_limits.yaml"/>
+    </xacro:unless>
     <!-- load params and define property -->
     <xacro:property name="default_inertial_params_filename" value="xarm7_type7_HT_BR2"/>
@@ -46,10 +52,13 @@
       <xacro:property name="inertial_params" value="${xacro.load_yaml(link_inertial_params_file)}"/>
       <xacro:property name="kinematics_config" value="${xacro.load_yaml(kinematics_params_filename)}"/>
+      <xacro:property name="joint_limits_config" value="${xacro.load_yaml(joint_limits_params_filename)}"/>
     </xacro:if>
     <xacro:unless value="${use_xacro_load_yaml}">
       <xacro:property name="inertial_params" value="${load_yaml(link_inertial_params_file)}"/>
       <xacro:property name="kinematics_config" value="${load_yaml(kinematics_params_filename)}"/>
+      <xacro:property name="joint_limits_config" value="${load_yaml(joint_limits_params_filename)}"/>
     </xacro:unless>
     <xacro:property name="kinematics_params" value="${kinematics_config['kinematics']}"/>
+    <xacro:property name="joint_limits" value="${joint_limits_config['joint_limits']}"/>
     <link name="${prefix}link_base">
       <inertial>
@@ -97,5 +106,5 @@
         lower="${joint1_lower_limit}"
         upper="${joint1_upper_limit}"
-        effort="50"
+        effort="${joint_limits['joint1']['max_effort']}"
         velocity="3.14" />
       <dynamics damping="10" friction="1" />
@@ -126,5 +135,5 @@
         lower="${joint2_lower_limit}"
         upper="${joint2_upper_limit}"
-        effort="50"
+        effort="${joint_limits['joint2']['max_effort']}"
         velocity="3.14" />
       <dynamics damping="10" friction="1" />
@@ -155,5 +164,5 @@
         lower="${joint3_lower_limit}"
         upper="${joint3_upper_limit}"
-        effort="30"
+        effort="${joint_limits['joint3']['max_effort']}"
         velocity="3.14" />
       <dynamics damping="5" friction="1" />
@@ -184,5 +193,5 @@
         lower="${joint4_lower_limit}"
         upper="${joint4_upper_limit}"
-        effort="30"
+        effort="${joint_limits['joint4']['max_effort']}"
         velocity="3.14" />
       <dynamics damping="5" friction="1" />
@@ -213,5 +222,5 @@
         lower="${joint5_lower_limit}"
         upper="${joint5_upper_limit}"
-        effort="30"
+        effort="${joint_limits['joint5']['max_effort']}"
         velocity="3.14" />
       <dynamics damping="5" friction="1" />
@@ -242,5 +251,5 @@
         lower="${joint6_lower_limit}"
         upper="${joint6_upper_limit}"
-        effort="20"
+        effort="${joint_limits['joint6']['max_effort']}"
         velocity="3.14" />
       <dynamics damping="2" friction="1" />
@@ -271,5 +280,5 @@
         lower="${joint7_lower_limit}"
         upper="${joint7_upper_limit}"
-        effort="20"
+        effort="${joint_limits['joint7']['max_effort']}"
         velocity="3.14" />
       <dynamics damping="2" friction="1" />
