Commit message: [feat] Lite6 support load Realsense D435i model
1. Lite6 support load Realsense D435i model
1. raname parameter `add_d435i_camera_link` to `add_d435i_links`

File: xarm_description/urdf/camera/realsense_d435i.urdf.xacro (robot description, xacro)
@@ -1,5 +1,5 @@
 <?xml version="1.0"?>
 <robot xmlns:xacro="http://ros.org/wiki/xacro">
-  <xacro:macro name="d435i_urdf" params="prefix:='' add_d435i_camera_link:=false">
+  <xacro:macro name="d435i_urdf" params="prefix:='' add_d435i_links:=false">
     <!-- define property -->
     <xacro:property name="M_PI" value="3.1415926535897931" />
@@ -15,5 +15,5 @@
         origin_rpy="0 0 0" />
     </link>
-    <xacro:if value="${add_d435i_camera_link}">
+    <xacro:if value="${add_d435i_links}">
       <link name="${prefix}camera_link"></link>
       <link name="${prefix}camera_depth_frame"></link>

File: xarm_description/urdf/common/common.link.xacro (robot description, xacro)
@@ -41,5 +41,5 @@
     </collision>
   </xacro:macro>
-  <xacro:macro name="parse_link_inertial_filename" params="dof robot_type robot_sn">
+  <xacro:macro name="parse_link_inertial_filename" params="dof robot_type robot_sn model1300">
     <!-- default inertial params filename -->
     <xacro:property name="inertial_params_filename" value="xarm${dof}_type${dof}_HT_BR2"/>
@@ -56,4 +56,5 @@
     <xacro:property name="mass_type" value="-1" />
     <xacro:property name="model_type" value="-1" />
+    <xacro:property name="_model1300" value="${model1300}" />
     <!-- parse model_type and mass_type from robot_sn -->
     <xacro:if value="${robot_sn_len >= 14 and (robot_sn[0] == 'X' or robot_sn[0] == 'L')}">
@@ -67,4 +68,7 @@
         <xacro:property name="model_type" value="11" />
         <xacro:property name="mass_type" value="1" />
+      </xacro:if>
+      <xacro:if value="${model_num >= 1300}">
+        <xacro:property name="_model1300" value="true" />
       </xacro:if>
       <xacro:if value="${robot_sn[8] == '0'}">
@@ -143,4 +147,5 @@
     </xacro:unless>
     <xacro:property name="scope_parent_inertial_params_filename" value="${inertial_params_filename}" scope="parent"/>
+    <xacro:property name="scope_parent_model1300" value="${_model1300}" scope="parent"/>
   </xacro:macro>
 </robot>

File: xarm_description/urdf/dual_xarm_device.urdf.xacro (robot description, xacro)
@@ -27,6 +27,6 @@
   <xacro:arg name="add_realsense_d435i_1" default="false"/>
   <xacro:arg name="add_realsense_d435i_2" default="false"/>
-  <xacro:arg name="add_d435i_camera_link_1" default="true"/>
-  <xacro:arg name="add_d435i_camera_link_2" default="true"/>
+  <xacro:arg name="add_d435i_links_1" default="true"/>
+  <xacro:arg name="add_d435i_links_2" default="true"/>
   <xacro:arg name="add_other_geometry_1" default="false"/>
   <xacro:arg name="geometry_type_1" default="box"/>
@@ -71,5 +71,5 @@
     attach_to="ground" attach_xyz="0 0 0" attach_rpy="0 0 0"
     add_realsense_d435i="$(arg add_realsense_d435i_1)"
-    add_d435i_camera_link="$(arg add_d435i_camera_link_1)"
+    add_d435i_links="$(arg add_d435i_links_1)"
     add_other_geometry="$(arg add_other_geometry_1)"
     geometry_type="$(arg geometry_type_1)" geometry_mass="$(arg geometry_mass_1)"
@@ -89,5 +89,5 @@
     attach_to="ground" attach_xyz="0 1 0" attach_rpy="0 0 0"
     add_realsense_d435i="$(arg add_realsense_d435i_2)"
-    add_d435i_camera_link="$(arg add_d435i_camera_link_2)"
+    add_d435i_links="$(arg add_d435i_links_2)"
     add_other_geometry="$(arg add_other_geometry_2)"
     geometry_type="$(arg geometry_type_2)" geometry_mass="$(arg geometry_mass_2)"

File: xarm_description/urdf/other/other_geometry.urdf.xacro (robot description, xacro)
@@ -1,7 +1,4 @@
 <?xml version="1.0"?>
-<robot xmlns:xacro="http://ros.org/wiki/xacro" name="xarm_vacuum_gripper">
-<!--
-  Author: Jason Peng <jason@ufactory.cc>
--->
+<robot xmlns:xacro="http://ros.org/wiki/xacro" name="other_geometry">
   <xacro:macro name="other_geometry" params="
     prefix:=''

File: xarm_description/urdf/xarm_device.urdf.xacro (robot description, xacro)
@@ -17,5 +17,5 @@
   <xacro:arg name="ros2_control_params" default="$(find xarm_controller)/config/xarm$(arg dof)_controllers.yaml"/>
   <xacro:arg name="add_realsense_d435i" default="false"/>
-  <xacro:arg name="add_d435i_camera_link" default="true"/>
+  <xacro:arg name="add_d435i_links" default="true"/>
   <xacro:arg name="use_gazebo_camera" default="false"/>
   <xacro:arg name="add_other_geometry" default="false"/>
@@ -44,5 +44,5 @@
     load_gazebo_plugin="true" ros2_control_params="$(arg ros2_control_params)"
     add_realsense_d435i="$(arg add_realsense_d435i)"
-    add_d435i_camera_link="$(arg add_d435i_camera_link)"
+    add_d435i_links="$(arg add_d435i_links)"
     add_other_geometry="$(arg add_other_geometry)"
     geometry_type="$(arg geometry_type)" geometry_mass="$(arg geometry_mass)"

File: xarm_description/urdf/xarm_device_macro.xacro (robot description, xacro)
@@ -18,5 +18,5 @@
     load_gazebo_plugin:=false
     add_realsense_d435i:=false
-    add_d435i_camera_link:=true
+    add_d435i_links:=true
     use_gazebo_camera:=false
     add_other_geometry:=false
@@ -55,6 +55,7 @@
     <!-- include common.link.xacro -->
     <xacro:include filename="$(find xarm_description)/urdf/common/common.link.xacro" />
-    <xacro:parse_link_inertial_filename dof="${dof}" robot_type="${robot_type}" robot_sn="${robot_sn}"/>
+    <xacro:parse_link_inertial_filename dof="${dof}" robot_type="${robot_type}" robot_sn="${robot_sn}" model1300="${model1300}" />
     <xacro:property name="inertial_params_filename" value="${scope_parent_inertial_params_filename}"/>
+    <xacro:property name="new_model1300" value="${scope_parent_model1300}"/>
     <!-- add one world link if no 'attach_to' specified  -->
     <xacro:if value="${attach_to == 'world'}">
@@ -77,5 +78,5 @@
         baud_checkset="${baud_checkset}"
         default_gripper_baud="${default_gripper_baud}"
-        model1300="${model1300}"
+        model1300="${new_model1300}"
         inertial_params_filename="${inertial_params_filename}" />
     </xacro:if>
@@ -105,5 +106,5 @@
           baud_checkset="${baud_checkset}"
           default_gripper_baud="${default_gripper_baud}"
-          model1300="${model1300}"
+          model1300="${new_model1300}"
           inertial_params_filename="${inertial_params_filename}" />
       </xacro:unless>
@@ -120,17 +121,17 @@
         baud_checkset="${baud_checkset}"
         default_gripper_baud="${default_gripper_baud}"
-        model1300="${model1300}"
+        model1300="${new_model1300}"
         inertial_params_filename="${inertial_params_filename}" />
     </xacro:unless>
-    <xacro:if value="${robot_type != 'lite' and add_realsense_d435i}">
+    <xacro:if value="${add_realsense_d435i}">
       <!-- (xarm) Load RealSense D435i URDF -->
       <xacro:include filename="$(find xarm_description)/urdf/camera/realsense_d435i.urdf.xacro" />
-      <xacro:d435i_urdf prefix="${prefix}" add_d435i_camera_link="${add_d435i_camera_link}" />
-      <xacro:if value="${add_d435i_camera_link}">
+      <xacro:d435i_urdf prefix="${prefix}" add_d435i_links="${add_d435i_links}" />
+      <xacro:if value="${add_d435i_links}">
         <xacro:include filename="$(find xarm_description)/urdf/camera/realsense.gazebo.xacro" />
         <xacro:realsense_gazebo prefix="${prefix}" />
       </xacro:if>
     </xacro:if>
-    <xacro:unless value="${robot_type != 'lite' and add_realsense_d435i}">
+    <xacro:unless value="${add_realsense_d435i}">
       <link name="${prefix}link_eef"/>
     </xacro:unless>
