Commit message: [fix] fix mesh file name or suffix
1. use the same suffix uniformly (stl)
2. the suffix name is instructed by parameters, which is convenient for replacing a whole set of modeles (such as obj or dae) in some scenes.

File: xarm_description/urdf/camera/realsense_d435i.urdf.xacro (robot description, xacro)
@@ -6,10 +6,10 @@
     <link name="${prefix}link_eef">
       <xacro:common_link_visual
-        mesh_filename="camera/realsense/visual/d435_with_cam_stand.STL"
+        mesh_filename="camera/realsense/visual/d435_with_cam_stand"
         origin_xyz="0 0 0"
         origin_rpy="0 0 0"
         material_name="${prefix}Silver" />
       <xacro:common_link_collision
-        mesh_filename="camera/realsense/collision/d435_with_cam_stand.STL"
+        mesh_filename="camera/realsense/collision/d435_with_cam_stand"
         origin_xyz="0 0 0"
         origin_rpy="0 0 0" />

File: xarm_description/urdf/common/common.link.xacro (robot description, xacro)
@@ -24,8 +24,13 @@
     </xacro:unless>
   </xacro:macro>
-  <xacro:macro name="common_link_visual" params="mesh_filename material_name:='White' origin_xyz:='0 0 0' origin_rpy:='0 0 0'">
+  <xacro:macro name="common_link_visual" params="mesh_filename add_mesh_suffix:=true material_name:='White' origin_xyz:='0 0 0' origin_rpy:='0 0 0'">
     <visual>
       <geometry>
-        <mesh filename="${mesh_path}/${mesh_filename}"/>
+        <xacro:if value="${add_mesh_suffix}">
+          <mesh filename="${mesh_path}/${mesh_filename}.${mesh_suffix}"/>
+        </xacro:if>
+        <xacro:unless value="${add_mesh_suffix}">
+          <mesh filename="${mesh_path}/${mesh_filename}"/>
+        </xacro:unless>
       </geometry>
       <origin xyz="${origin_xyz}" rpy="${origin_rpy}"/>
@@ -33,8 +38,13 @@
     </visual>
   </xacro:macro>
-  <xacro:macro name="common_link_collision" params="mesh_filename origin_xyz:='0 0 0' origin_rpy:='0 0 0'">
+  <xacro:macro name="common_link_collision" params="mesh_filename add_mesh_suffix:=true origin_xyz:='0 0 0' origin_rpy:='0 0 0'">
     <collision>
       <geometry>
-        <mesh filename="${mesh_path}/${mesh_filename}"/>
+        <xacro:if value="${add_mesh_suffix}">
+          <mesh filename="${mesh_path}/${mesh_filename}.${mesh_suffix}"/>
+        </xacro:if>
+        <xacro:unless value="${add_mesh_suffix}">
+          <mesh filename="${mesh_path}/${mesh_filename}"/>
+        </xacro:unless>
       </geometry>
       <origin xyz="${origin_xyz}" rpy="${origin_rpy}"/>

File: xarm_description/urdf/dual_xarm_device.urdf.xacro (robot description, xacro)
@@ -57,4 +57,5 @@
   <xacro:arg name="default_gripper_baud_1" default="2000000"/>
   <xacro:arg name="default_gripper_baud_2" default="2000000"/>
+  <xacro:arg name="mesh_suffix" default="stl"/>
   <!-- load xarm device -->
   <xacro:include filename="$(find xarm_description)/urdf/xarm_device_macro.xacro" />
@@ -76,5 +77,5 @@
     robot_ip="$(arg robot_ip_1)" report_type="$(arg report_type_1)"
     baud_checkset="$(arg baud_checkset_1)" default_gripper_baud="$(arg default_gripper_baud_1)"
-    model1300="$(arg model1300_1)" robot_sn="$(arg robot_sn_1)"/>
+    model1300="$(arg model1300_1)" robot_sn="$(arg robot_sn_1)" mesh_suffix="$(arg mesh_suffix)" />
   <xacro:xarm_device prefix="$(arg prefix_2)" hw_ns="$(arg hw_ns)" limited="$(arg limited)"
     effort_control="$(arg effort_control)" velocity_control="$(arg velocity_control)"
@@ -94,4 +95,4 @@
     robot_ip="$(arg robot_ip_2)" report_type="$(arg report_type_2)"
     baud_checkset="$(arg baud_checkset_2)" default_gripper_baud="$(arg default_gripper_baud_2)"
-    model1300="$(arg model1300_2)" robot_sn="$(arg robot_sn_2)"/>
+    model1300="$(arg model1300_2)" robot_sn="$(arg robot_sn_2)" mesh_suffix="$(arg mesh_suffix)" />
 </robot>

File: xarm_description/urdf/gripper/lite_gripper.urdf.xacro (robot description, xacro)
@@ -18,10 +18,10 @@
       </inertial>
       <xacro:common_link_visual
-        mesh_filename="gripper/lite/visual/gripper_lite.stl"
+        mesh_filename="gripper/lite/visual/gripper_lite"
         origin_xyz="0 0 0"
         origin_rpy="0 0 0"
         material_name="${prefix}White" />
       <xacro:common_link_collision
-        mesh_filename="gripper/lite/collision/gripper_lite.stl"
+        mesh_filename="gripper/lite/collision/gripper_lite"
         origin_xyz="0 0 0"
         origin_rpy="0 0 0" />

File: xarm_description/urdf/gripper/xarm_gripper.urdf.xacro (robot description, xacro)
@@ -18,10 +18,10 @@
       </inertial>
       <xacro:common_link_visual
-        mesh_filename="gripper/xarm/base_link.STL"
+        mesh_filename="gripper/xarm/base_link"
         origin_xyz="0 0 0"
         origin_rpy="0 0 0"
         material_name="${prefix}White" />
       <xacro:common_link_collision
-        mesh_filename="gripper/xarm/base_link.STL"
+        mesh_filename="gripper/xarm/base_link"
         origin_xyz="0 0 0"
         origin_rpy="0 0 0" />
@@ -36,10 +36,10 @@
       </inertial>
       <xacro:common_link_visual
-        mesh_filename="gripper/xarm/left_outer_knuckle.STL"
+        mesh_filename="gripper/xarm/left_outer_knuckle"
         origin_xyz="0 0 0"
         origin_rpy="0 0 0"
         material_name="${prefix}Silver" />
       <xacro:common_link_collision
-        mesh_filename="gripper/xarm/left_outer_knuckle.STL"
+        mesh_filename="gripper/xarm/left_outer_knuckle"
         origin_xyz="0 0 0"
         origin_rpy="0 0 0" />
@@ -61,10 +61,10 @@
       </inertial>
       <xacro:common_link_visual
-        mesh_filename="gripper/xarm/left_finger.STL"
+        mesh_filename="gripper/xarm/left_finger"
         origin_xyz="0 0 0"
         origin_rpy="0 0 0"
         material_name="${prefix}Silver" />
       <xacro:common_link_collision
-        mesh_filename="gripper/xarm/left_finger.STL"
+        mesh_filename="gripper/xarm/left_finger"
         origin_xyz="0 0 0"
         origin_rpy="0 0 0" />
@@ -87,10 +87,10 @@
       </inertial>
       <xacro:common_link_visual
-        mesh_filename="gripper/xarm/left_inner_knuckle.STL"
+        mesh_filename="gripper/xarm/left_inner_knuckle"
         origin_xyz="0 0 0"
         origin_rpy="0 0 0"
         material_name="${prefix}Silver" />
       <xacro:common_link_collision
-        mesh_filename="gripper/xarm/left_inner_knuckle.STL"
+        mesh_filename="gripper/xarm/left_inner_knuckle"
         origin_xyz="0 0 0"
         origin_rpy="0 0 0" />
@@ -113,10 +113,10 @@
       </inertial>
       <xacro:common_link_visual
-        mesh_filename="gripper/xarm/right_outer_knuckle.STL"
+        mesh_filename="gripper/xarm/right_outer_knuckle"
         origin_xyz="0 0 0"
         origin_rpy="0 0 0"
         material_name="${prefix}Silver" />
       <xacro:common_link_collision
-        mesh_filename="gripper/xarm/right_outer_knuckle.STL"
+        mesh_filename="gripper/xarm/right_outer_knuckle"
         origin_xyz="0 0 0"
         origin_rpy="0 0 0" />
@@ -139,10 +139,10 @@
       </inertial>
       <xacro:common_link_visual
-        mesh_filename="gripper/xarm/right_finger.STL"
+        mesh_filename="gripper/xarm/right_finger"
         origin_xyz="0 0 0"
         origin_rpy="0 0 0"
         material_name="${prefix}Silver" />
       <xacro:common_link_collision
-        mesh_filename="gripper/xarm/right_finger.STL"
+        mesh_filename="gripper/xarm/right_finger"
         origin_xyz="0 0 0"
         origin_rpy="0 0 0" />
@@ -165,10 +165,10 @@
       </inertial>
       <xacro:common_link_visual
-        mesh_filename="gripper/xarm/right_inner_knuckle.STL"
+        mesh_filename="gripper/xarm/right_inner_knuckle"
         origin_xyz="0 0 0"
         origin_rpy="0 0 0"
         material_name="${prefix}Silver" />
       <xacro:common_link_collision
-        mesh_filename="gripper/xarm/right_inner_knuckle.STL"
+        mesh_filename="gripper/xarm/right_inner_knuckle"
         origin_xyz="0 0 0"
         origin_rpy="0 0 0" />

File: xarm_description/urdf/lite6/lite6.urdf.xacro (robot description, xacro)
@@ -33,10 +33,10 @@
       </inertial>
       <xacro:common_link_visual
-        mesh_filename="lite6/visual/base.stl"
-        origin_xyz="0 0 0"
-        origin_rpy="0 0 0"
-        material_name="${prefix}White" />
-      <xacro:common_link_collision
-        mesh_filename="lite6/visual/base.stl"
+        mesh_filename="lite6/visual/link_base"
+        origin_xyz="0 0 0"
+        origin_rpy="0 0 0"
+        material_name="${prefix}White" />
+      <xacro:common_link_collision
+        mesh_filename="lite6/collision/link_base"
         origin_xyz="0 0 0"
         origin_rpy="0 0 0" />
@@ -47,10 +47,10 @@
         origin_rpy="0 0 0"/>
       <xacro:common_link_visual
-        mesh_filename="lite6/visual/link1.stl"
-        origin_xyz="0 0 0"
-        origin_rpy="0 0 0"
-        material_name="${prefix}White" />
-      <xacro:common_link_collision
-        mesh_filename="lite6/visual/link1.stl"
+        mesh_filename="lite6/visual/link1"
+        origin_xyz="0 0 0"
+        origin_rpy="0 0 0"
+        material_name="${prefix}White" />
+      <xacro:common_link_collision
+        mesh_filename="lite6/collision/link1"
         origin_xyz="0 0 0"
         origin_rpy="0 0 0" />
@@ -73,10 +73,10 @@
         origin_rpy="0 0 0"/>
       <xacro:common_link_visual
-        mesh_filename="lite6/visual/link2.stl"
-        origin_xyz="0 0 0"
-        origin_rpy="0 0 0"
-        material_name="${prefix}White" />
-      <xacro:common_link_collision
-        mesh_filename="lite6/visual/link2.stl"
+        mesh_filename="lite6/visual/link2"
+        origin_xyz="0 0 0"
+        origin_rpy="0 0 0"
+        material_name="${prefix}White" />
+      <xacro:common_link_collision
+        mesh_filename="lite6/collision/link2"
         origin_xyz="0 0 0"
         origin_rpy="0 0 0" />
@@ -99,10 +99,10 @@
         origin_rpy="0 0 0"/>
       <xacro:common_link_visual
-        mesh_filename="lite6/visual/link3.stl"
-        origin_xyz="0 0 0"
-        origin_rpy="0 0 0"
-        material_name="${prefix}White" />
-      <xacro:common_link_collision
-        mesh_filename="lite6/visual/link3.stl"
+        mesh_filename="lite6/visual/link3"
+        origin_xyz="0 0 0"
+        origin_rpy="0 0 0"
+        material_name="${prefix}White" />
+      <xacro:common_link_collision
+        mesh_filename="lite6/collision/link3"
         origin_xyz="0 0 0"
         origin_rpy="0 0 0" />
@@ -125,10 +125,10 @@
         origin_rpy="0 0 0"/>
       <xacro:common_link_visual
-        mesh_filename="lite6/visual/link4.stl"
-        origin_xyz="0 0 0"
-        origin_rpy="0 0 0"
-        material_name="${prefix}White" />
-      <xacro:common_link_collision
-        mesh_filename="lite6/visual/link4.stl"
+        mesh_filename="lite6/visual/link4"
+        origin_xyz="0 0 0"
+        origin_rpy="0 0 0"
+        material_name="${prefix}White" />
+      <xacro:common_link_collision
+        mesh_filename="lite6/collision/link4"
         origin_xyz="0 0 0"
         origin_rpy="0 0 0" />
@@ -151,10 +151,10 @@
         origin_rpy="0 0 0"/>
       <xacro:common_link_visual
-        mesh_filename="lite6/visual/link5.stl"
-        origin_xyz="0 0 0"
-        origin_rpy="0 0 0"
-        material_name="${prefix}White" />
-      <xacro:common_link_collision
-        mesh_filename="lite6/visual/link5.stl"
+        mesh_filename="lite6/visual/link5"
+        origin_xyz="0 0 0"
+        origin_rpy="0 0 0"
+        material_name="${prefix}White" />
+      <xacro:common_link_collision
+        mesh_filename="lite6/collision/link5"
         origin_xyz="0 0 0"
         origin_rpy="0 0 0" />
@@ -177,10 +177,10 @@
         origin_rpy="0 0 0"/>
       <xacro:common_link_visual
-        mesh_filename="lite6/visual/link6.stl"
+        mesh_filename="lite6/visual/link6"
         origin_xyz="0 0 0"
         origin_rpy="0 0 0"
         material_name="${prefix}Silver" />
       <xacro:common_link_collision
-        mesh_filename="lite6/visual/link6.stl"
+        mesh_filename="lite6/collision/link6"
         origin_xyz="0 0 0"
         origin_rpy="0 0 0" />

File: xarm_description/urdf/uf850/uf850.urdf.xacro (robot description, xacro)
@@ -34,10 +34,10 @@
       </inertial>
       <xacro:common_link_visual
-        mesh_filename="uf850/visual/link_base.STL"
-        origin_xyz="0 0 0"
-        origin_rpy="0 0 0"
-        material_name="${prefix}White" />
-      <xacro:common_link_collision
-        mesh_filename="uf850/collision/link_base.STL"
+        mesh_filename="uf850/visual/link_base"
+        origin_xyz="0 0 0"
+        origin_rpy="0 0 0"
+        material_name="${prefix}White" />
+      <xacro:common_link_collision
+        mesh_filename="uf850/collision/link_base"
         origin_xyz="0 0 0"
         origin_rpy="0 0 0" />
@@ -48,10 +48,10 @@
         origin_rpy="0 0 0"/>
       <xacro:common_link_visual
-        mesh_filename="uf850/visual/link1.STL"
-        origin_xyz="0 0 0"
-        origin_rpy="0 0 0"
-        material_name="${prefix}White" />
-      <xacro:common_link_collision
-        mesh_filename="uf850/collision/link1.STL"
+        mesh_filename="uf850/visual/link1"
+        origin_xyz="0 0 0"
+        origin_rpy="0 0 0"
+        material_name="${prefix}White" />
+      <xacro:common_link_collision
+        mesh_filename="uf850/collision/link1"
         origin_xyz="0 0 0"
         origin_rpy="0 0 0" />
@@ -74,10 +74,10 @@
         origin_rpy="0 0 0"/>
       <xacro:common_link_visual
-        mesh_filename="uf850/visual/link2.STL"
-        origin_xyz="0 0 0"
-        origin_rpy="0 0 0"
-        material_name="${prefix}White" />
-      <xacro:common_link_collision
-        mesh_filename="uf850/collision/link2.STL"
+        mesh_filename="uf850/visual/link2"
+        origin_xyz="0 0 0"
+        origin_rpy="0 0 0"
+        material_name="${prefix}White" />
+      <xacro:common_link_collision
+        mesh_filename="uf850/collision/link2"
         origin_xyz="0 0 0"
         origin_rpy="0 0 0" />
@@ -100,10 +100,10 @@
         origin_rpy="0 0 0"/>
       <xacro:common_link_visual
-        mesh_filename="uf850/visual/link3.STL"
-        origin_xyz="0 0 0"
-        origin_rpy="0 0 0"
-        material_name="${prefix}White" />
-      <xacro:common_link_collision
-        mesh_filename="uf850/collision/link3.STL"
+        mesh_filename="uf850/visual/link3"
+        origin_xyz="0 0 0"
+        origin_rpy="0 0 0"
+        material_name="${prefix}White" />
+      <xacro:common_link_collision
+        mesh_filename="uf850/collision/link3"
         origin_xyz="0 0 0"
         origin_rpy="0 0 0" />
@@ -126,10 +126,10 @@
         origin_rpy="0 0 0"/>
       <xacro:common_link_visual
-        mesh_filename="uf850/visual/link4.STL"
-        origin_xyz="0 0 0"
-        origin_rpy="0 0 0"
-        material_name="${prefix}White" />
-      <xacro:common_link_collision
-        mesh_filename="uf850/collision/link4.STL"
+        mesh_filename="uf850/visual/link4"
+        origin_xyz="0 0 0"
+        origin_rpy="0 0 0"
+        material_name="${prefix}White" />
+      <xacro:common_link_collision
+        mesh_filename="uf850/collision/link4"
         origin_xyz="0 0 0"
         origin_rpy="0 0 0" />
@@ -152,10 +152,10 @@
         origin_rpy="0 0 0"/>
       <xacro:common_link_visual
-        mesh_filename="uf850/visual/link5.STL"
-        origin_xyz="0 0 0"
-        origin_rpy="0 0 0"
-        material_name="${prefix}White" />
-      <xacro:common_link_collision
-        mesh_filename="uf850/collision/link5.STL"
+        mesh_filename="uf850/visual/link5"
+        origin_xyz="0 0 0"
+        origin_rpy="0 0 0"
+        material_name="${prefix}White" />
+      <xacro:common_link_collision
+        mesh_filename="uf850/collision/link5"
         origin_xyz="0 0 0"
         origin_rpy="0 0 0" />
@@ -178,10 +178,10 @@
         origin_rpy="0 0 0"/>
       <xacro:common_link_visual
-        mesh_filename="uf850/visual/link6.STL"
-        origin_xyz="0 0 0"
-        origin_rpy="0 0 0"
-        material_name="${prefix}White" />
-      <xacro:common_link_collision
-        mesh_filename="uf850/collision/link6.STL"
+        mesh_filename="uf850/visual/link6"
+        origin_xyz="0 0 0"
+        origin_rpy="0 0 0"
+        material_name="${prefix}White" />
+      <xacro:common_link_collision
+        mesh_filename="uf850/collision/link6"
         origin_xyz="0 0 0"
         origin_rpy="0 0 0" />

File: xarm_description/urdf/vacuum_gripper/lite_vacuum_gripper.urdf.xacro (robot description, xacro)
@@ -18,10 +18,10 @@
       </inertial>
       <xacro:common_link_visual
-        mesh_filename="vacuum_gripper/lite/visual/vacuum_gripper_lite.stl"
+        mesh_filename="vacuum_gripper/lite/visual/vacuum_gripper_lite"
         origin_xyz="0 0 0"
         origin_rpy="0 0 0"
         material_name="${prefix}White" />
       <xacro:common_link_collision
-        mesh_filename="vacuum_gripper/lite/collision/vacuum_gripper_lite.stl"
+        mesh_filename="vacuum_gripper/lite/collision/vacuum_gripper_lite"
         origin_xyz="0 0 0"
         origin_rpy="0 0 0" />

File: xarm_description/urdf/vacuum_gripper/xarm_vacuum_gripper.urdf.xacro (robot description, xacro)
@@ -18,10 +18,10 @@
       </inertial>
       <xacro:common_link_visual
-        mesh_filename="vacuum_gripper/xarm/visual/vacuum_gripper.STL"
+        mesh_filename="vacuum_gripper/xarm/visual/vacuum_gripper"
         origin_xyz="0 0 0"
         origin_rpy="0 0 0"
         material_name="${prefix}White" />
       <xacro:common_link_collision
-        mesh_filename="vacuum_gripper/xarm/collision/vacuum_gripper.STL"
+        mesh_filename="vacuum_gripper/xarm/collision/vacuum_gripper"
         origin_xyz="0 0 0"
         origin_rpy="0 0 0" />

File: xarm_description/urdf/xarm5/xarm5.urdf.xacro (robot description, xacro)
@@ -12,10 +12,10 @@
     <!-- define property -->
     <xacro:if value="${model1300}">
-      <xacro:property name="end_tool_visual_filename" value="end_tool/visual/end_tool_1300.STL"/>
-      <xacro:property name="end_tool_collision_filename" value="end_tool/collision/end_tool_1300.STL"/>
+      <xacro:property name="end_tool_visual_filename" value="end_tool/visual/end_tool_1300"/>
+      <xacro:property name="end_tool_collision_filename" value="end_tool/collision/end_tool_1300"/>
     </xacro:if>
     <xacro:unless value="${model1300}">
-      <xacro:property name="end_tool_visual_filename" value="xarm5/visual/link5.STL"/>
-      <xacro:property name="end_tool_collision_filename" value="end_tool/collision/end_tool.STL"/>
+      <xacro:property name="end_tool_visual_filename" value="xarm5/visual/link5"/>
+      <xacro:property name="end_tool_collision_filename" value="end_tool/collision/end_tool"/>
     </xacro:unless>
     <!-- load params and define property -->
@@ -42,10 +42,10 @@
       </inertial>
       <xacro:common_link_visual
-        mesh_filename="xarm5/visual/base_link.STL"
+        mesh_filename="xarm5/visual/link_base"
         origin_xyz="0 0 0"
         origin_rpy="0 0 0"
         material_name="${prefix}White" />
       <xacro:common_link_collision
-        mesh_filename="xarm5/visual/base_link.STL"
+        mesh_filename="xarm5/visual/link_base"
         origin_xyz="0 0 0"
         origin_rpy="0 0 0" />
@@ -56,10 +56,10 @@
         origin_rpy="0 0 0"/>
       <xacro:common_link_visual
-        mesh_filename="xarm5/visual/link1.STL"
+        mesh_filename="xarm5/visual/link1"
         origin_xyz="0 0 0"
         origin_rpy="0 0 0"
         material_name="${prefix}White" />
       <xacro:common_link_collision
-        mesh_filename="xarm5/visual/link1.STL"
+        mesh_filename="xarm5/visual/link1"
         origin_xyz="0 0 0"
         origin_rpy="0 0 0" />
@@ -82,10 +82,10 @@
         origin_rpy="0 0 0"/>
       <xacro:common_link_visual
-        mesh_filename="xarm5/visual/link2.STL"
+        mesh_filename="xarm5/visual/link2"
         origin_xyz="0 0 0"
         origin_rpy="0 0 0"
         material_name="${prefix}White" />
       <xacro:common_link_collision
-        mesh_filename="xarm5/visual/link2.STL"
+        mesh_filename="xarm5/visual/link2"
         origin_xyz="0 0 0"
         origin_rpy="0 0 0" />
@@ -108,10 +108,10 @@
         origin_rpy="0 0 0"/>
       <xacro:common_link_visual
-        mesh_filename="xarm5/visual/link3.STL"
+        mesh_filename="xarm5/visual/link3"
         origin_xyz="0 0 0"
         origin_rpy="0 0 0"
         material_name="${prefix}White" />
       <xacro:common_link_collision
-        mesh_filename="xarm5/visual/link3.STL"
+        mesh_filename="xarm5/visual/link3"
         origin_xyz="0 0 0"
         origin_rpy="0 0 0" />
@@ -134,10 +134,10 @@
         origin_rpy="0 0 0"/>
       <xacro:common_link_visual
-        mesh_filename="xarm5/visual/link4.STL"
+        mesh_filename="xarm5/visual/link4"
         origin_xyz="0 0 0"
         origin_rpy="0 0 0"
         material_name="${prefix}White" />
       <xacro:common_link_collision
-        mesh_filename="xarm5/visual/link4.STL"
+        mesh_filename="xarm5/visual/link4"
         origin_xyz="0 0 0"
         origin_rpy="0 0 0" />
