Commit message: [fix] fix mesh file name or suffix
1. use the same suffix uniformly (stl)
2. the suffix name is instructed by parameters, which is convenient for replacing a whole set of modeles (such as obj or dae) in some scenes.

File: xarm_description/urdf/xarm6/xarm6.urdf.xacro (robot description, xacro)
@@ -13,10 +13,10 @@
     <!-- define property -->
     <xacro:if value="${model1300}">
-      <xacro:property name="end_tool_visual_filename" value="end_tool/visual/end_tool_1300.STL"/>
-      <xacro:property name="end_tool_collision_filename" value="end_tool/collision/end_tool_1300.STL"/>
+      <xacro:property name="end_tool_visual_filename" value="end_tool/visual/end_tool_1300"/>
+      <xacro:property name="end_tool_collision_filename" value="end_tool/collision/end_tool_1300"/>
     </xacro:if>
     <xacro:unless value="${model1300}">
-      <xacro:property name="end_tool_visual_filename" value="xarm6/visual/link6.stl"/>
-      <xacro:property name="end_tool_collision_filename" value="end_tool/collision/end_tool.STL"/>
+      <xacro:property name="end_tool_visual_filename" value="xarm6/visual/link6"/>
+      <xacro:property name="end_tool_collision_filename" value="end_tool/collision/end_tool"/>
     </xacro:unless>
     <!-- load params and define property -->
@@ -43,10 +43,10 @@
       </inertial>
       <xacro:common_link_visual
-        mesh_filename="xarm6/visual/base.stl"
-        origin_xyz="0 0 0"
-        origin_rpy="0 0 0"
-        material_name="${prefix}White" />
-      <xacro:common_link_collision
-        mesh_filename="xarm6/visual/base.stl"
+        mesh_filename="xarm6/visual/link_base"
+        origin_xyz="0 0 0"
+        origin_rpy="0 0 0"
+        material_name="${prefix}White" />
+      <xacro:common_link_collision
+        mesh_filename="xarm6/visual/link_base"
         origin_xyz="0 0 0"
         origin_rpy="0 0 0" />
@@ -57,10 +57,10 @@
         origin_rpy="0 0 0"/>
       <xacro:common_link_visual
-        mesh_filename="xarm6/visual/link1.stl"
-        origin_xyz="0 0 0"
-        origin_rpy="0 0 0"
-        material_name="${prefix}White" />
-      <xacro:common_link_collision
-        mesh_filename="xarm6/visual/link1.stl"
+        mesh_filename="xarm6/visual/link1"
+        origin_xyz="0 0 0"
+        origin_rpy="0 0 0"
+        material_name="${prefix}White" />
+      <xacro:common_link_collision
+        mesh_filename="xarm6/visual/link1"
         origin_xyz="0 0 0"
         origin_rpy="0 0 0" />
@@ -83,10 +83,10 @@
         origin_rpy="0 0 0"/>
       <xacro:common_link_visual
-        mesh_filename="xarm6/visual/link2.stl"
-        origin_xyz="0 0 0"
-        origin_rpy="0 0 0"
-        material_name="${prefix}White" />
-      <xacro:common_link_collision
-        mesh_filename="xarm6/visual/link2.stl"
+        mesh_filename="xarm6/visual/link2"
+        origin_xyz="0 0 0"
+        origin_rpy="0 0 0"
+        material_name="${prefix}White" />
+      <xacro:common_link_collision
+        mesh_filename="xarm6/visual/link2"
         origin_xyz="0 0 0"
         origin_rpy="0 0 0" />
@@ -109,10 +109,10 @@
         origin_rpy="0 0 0"/>
       <xacro:common_link_visual
-        mesh_filename="xarm6/visual/link3.stl"
-        origin_xyz="0 0 0"
-        origin_rpy="0 0 0"
-        material_name="${prefix}White" />
-      <xacro:common_link_collision
-        mesh_filename="xarm6/visual/link3.stl"
+        mesh_filename="xarm6/visual/link3"
+        origin_xyz="0 0 0"
+        origin_rpy="0 0 0"
+        material_name="${prefix}White" />
+      <xacro:common_link_collision
+        mesh_filename="xarm6/visual/link3"
         origin_xyz="0 0 0"
         origin_rpy="0 0 0" />
@@ -135,10 +135,10 @@
         origin_rpy="0 0 0"/>
       <xacro:common_link_visual
-        mesh_filename="xarm6/visual/link4.stl"
-        origin_xyz="0 0 0"
-        origin_rpy="0 0 0"
-        material_name="${prefix}White" />
-      <xacro:common_link_collision
-        mesh_filename="xarm6/visual/link4.stl"
+        mesh_filename="xarm6/visual/link4"
+        origin_xyz="0 0 0"
+        origin_rpy="0 0 0"
+        material_name="${prefix}White" />
+      <xacro:common_link_collision
+        mesh_filename="xarm6/visual/link4"
         origin_xyz="0 0 0"
         origin_rpy="0 0 0" />
@@ -161,10 +161,10 @@
         origin_rpy="0 0 0"/>
       <xacro:common_link_visual
-        mesh_filename="xarm6/visual/link5.stl"
-        origin_xyz="0 0 0"
-        origin_rpy="0 0 0"
-        material_name="${prefix}White" />
-      <xacro:common_link_collision
-        mesh_filename="xarm6/visual/link5.stl"
+        mesh_filename="xarm6/visual/link5"
+        origin_xyz="0 0 0"
+        origin_rpy="0 0 0"
+        material_name="${prefix}White" />
+      <xacro:common_link_collision
+        mesh_filename="xarm6/visual/link5"
         origin_xyz="0 0 0"
         origin_rpy="0 0 0" />

File: xarm_description/urdf/xarm7/xarm7.urdf.xacro (robot description, xacro)
@@ -14,10 +14,10 @@
     <!-- define property -->
     <xacro:if value="${model1300}">
-      <xacro:property name="end_tool_visual_filename" value="end_tool/visual/end_tool_1300.STL"/>
-      <xacro:property name="end_tool_collision_filename" value="end_tool/collision/end_tool_1300.STL"/>
+      <xacro:property name="end_tool_visual_filename" value="end_tool/visual/end_tool_1300"/>
+      <xacro:property name="end_tool_collision_filename" value="end_tool/collision/end_tool_1300"/>
     </xacro:if>
     <xacro:unless value="${model1300}">
-      <xacro:property name="end_tool_visual_filename" value="xarm7/visual/link7.STL"/>
-      <xacro:property name="end_tool_collision_filename" value="end_tool/collision/end_tool.STL"/>
+      <xacro:property name="end_tool_visual_filename" value="xarm7/visual/link7"/>
+      <xacro:property name="end_tool_collision_filename" value="end_tool/collision/end_tool"/>
     </xacro:unless>
     <!-- load params and define property -->
@@ -44,10 +44,10 @@
       </inertial>
       <xacro:common_link_visual
-        mesh_filename="xarm7/visual/link_base.STL"
-        origin_xyz="0 0 0"
-        origin_rpy="0 0 0"
-        material_name="${prefix}White" />
-      <xacro:common_link_collision
-        mesh_filename="xarm7/visual/link_base.STL"
+        mesh_filename="xarm7/visual/link_base"
+        origin_xyz="0 0 0"
+        origin_rpy="0 0 0"
+        material_name="${prefix}White" />
+      <xacro:common_link_collision
+        mesh_filename="xarm7/visual/link_base"
         origin_xyz="0 0 0"
         origin_rpy="0 0 0" />
@@ -58,10 +58,10 @@
         origin_rpy="0 0 0"/>
       <xacro:common_link_visual
-        mesh_filename="xarm7/visual/link1.STL"
-        origin_xyz="0 0 0"
-        origin_rpy="0 0 0"
-        material_name="${prefix}White" />
-      <xacro:common_link_collision
-        mesh_filename="xarm7/visual/link1.STL"
+        mesh_filename="xarm7/visual/link1"
+        origin_xyz="0 0 0"
+        origin_rpy="0 0 0"
+        material_name="${prefix}White" />
+      <xacro:common_link_collision
+        mesh_filename="xarm7/visual/link1"
         origin_xyz="0 0 0"
         origin_rpy="0 0 0" />
@@ -84,10 +84,10 @@
         origin_rpy="0 0 0"/>
       <xacro:common_link_visual
-        mesh_filename="xarm7/visual/link2.STL"
-        origin_xyz="0 0 0"
-        origin_rpy="0 0 0"
-        material_name="${prefix}White" />
-      <xacro:common_link_collision
-        mesh_filename="xarm7/visual/link2.STL"
+        mesh_filename="xarm7/visual/link2"
+        origin_xyz="0 0 0"
+        origin_rpy="0 0 0"
+        material_name="${prefix}White" />
+      <xacro:common_link_collision
+        mesh_filename="xarm7/visual/link2"
         origin_xyz="0 0 0"
         origin_rpy="0 0 0" />
@@ -110,10 +110,10 @@
         origin_rpy="0 0 0"/>
       <xacro:common_link_visual
-        mesh_filename="xarm7/visual/link3.STL"
-        origin_xyz="0 0 0"
-        origin_rpy="0 0 0"
-        material_name="${prefix}White" />
-      <xacro:common_link_collision
-        mesh_filename="xarm7/visual/link3.STL"
+        mesh_filename="xarm7/visual/link3"
+        origin_xyz="0 0 0"
+        origin_rpy="0 0 0"
+        material_name="${prefix}White" />
+      <xacro:common_link_collision
+        mesh_filename="xarm7/visual/link3"
         origin_xyz="0 0 0"
         origin_rpy="0 0 0" />
@@ -136,10 +136,10 @@
         origin_rpy="0 0 0"/>
       <xacro:common_link_visual
-        mesh_filename="xarm7/visual/link4.STL"
-        origin_xyz="0 0 0"
-        origin_rpy="0 0 0"
-        material_name="${prefix}White" />
-      <xacro:common_link_collision
-        mesh_filename="xarm7/visual/link4.STL"
+        mesh_filename="xarm7/visual/link4"
+        origin_xyz="0 0 0"
+        origin_rpy="0 0 0"
+        material_name="${prefix}White" />
+      <xacro:common_link_collision
+        mesh_filename="xarm7/visual/link4"
         origin_xyz="0 0 0"
         origin_rpy="0 0 0" />
@@ -162,10 +162,10 @@
         origin_rpy="0 0 0"/>
       <xacro:common_link_visual
-        mesh_filename="xarm7/visual/link5.STL"
-        origin_xyz="0 0 0"
-        origin_rpy="0 0 0"
-        material_name="${prefix}White" />
-      <xacro:common_link_collision
-        mesh_filename="xarm7/visual/link5.STL"
+        mesh_filename="xarm7/visual/link5"
+        origin_xyz="0 0 0"
+        origin_rpy="0 0 0"
+        material_name="${prefix}White" />
+      <xacro:common_link_collision
+        mesh_filename="xarm7/visual/link5"
         origin_xyz="0 0 0"
         origin_rpy="0 0 0" />
@@ -188,10 +188,10 @@
         origin_rpy="0 0 0"/>
       <xacro:common_link_visual
-        mesh_filename="xarm7/visual/link6.STL"
-        origin_xyz="0 0 0"
-        origin_rpy="0 0 0"
-        material_name="${prefix}White" />
-      <xacro:common_link_collision
-        mesh_filename="xarm7/visual/link6.STL"
+        mesh_filename="xarm7/visual/link6"
+        origin_xyz="0 0 0"
+        origin_rpy="0 0 0"
+        material_name="${prefix}White" />
+      <xacro:common_link_collision
+        mesh_filename="xarm7/visual/link6"
         origin_xyz="0 0 0"
         origin_rpy="0 0 0" />

File: xarm_description/urdf/xarm_device.urdf.xacro (robot description, xacro)
@@ -36,4 +36,5 @@
   <xacro:arg name="attach_xyz" default="0 0 0"/>
   <xacro:arg name="attach_rpy" default="0 0 0"/>
+  <xacro:arg name="mesh_suffix" default="stl"/>
   <!-- load xarm device -->
   <xacro:include filename="$(find xarm_description)/urdf/xarm_device_macro.xacro" />
@@ -55,4 +56,4 @@
     baud_checkset="$(arg baud_checkset)" default_gripper_baud="$(arg default_gripper_baud)"
     model1300="$(arg model1300)" attach_to="$(arg attach_to)" attach_xyz="$(arg attach_xyz)" attach_rpy="$(arg attach_rpy)"
-    robot_sn="$(arg robot_sn)" use_gazebo_camera="$(arg use_gazebo_camera)" />
+    robot_sn="$(arg robot_sn)" use_gazebo_camera="$(arg use_gazebo_camera)" mesh_suffix="$(arg mesh_suffix)" />
 </robot>

File: xarm_description/urdf/xarm_device_macro.xacro (robot description, xacro)
@@ -38,5 +38,6 @@
     default_gripper_baud:=2000000
     model1300:=false
-    robot_sn:='' "
+    robot_sn:=''
+    mesh_suffix:='stl' "
     >
     <!-- Load Common Material -->
@@ -47,4 +48,5 @@
     <xacro:common_material prefix="${prefix}"/>
     <!-- Specify Mesh file path -->
+    <xacro:property name="mesh_suffix" value="${mesh_suffix}" scope="parent"/>
     <xacro:if value="${ros2_control_plugin == 'gazebo_ros2_control/GazeboSystem' or ros2_control_plugin == 'ign_ros2_control/IgnitionSystem'}">
       <!-- gazebo use -->

File: xarm_gripper/urdf/xarm_gripper.urdf.xacro (robot description, xacro)
@@ -34,5 +34,5 @@
       <geometry>
         <mesh
-          filename="package://xarm_gripper/meshes/base_link.STL" />
+          filename="package://xarm_gripper/meshes/base_link.stl" />
       </geometry>
       <!-- <material
@@ -51,5 +51,5 @@
       <geometry>
         <mesh
-          filename="package://xarm_gripper/meshes/base_link_collision.STL" />
+          filename="package://xarm_gripper/meshes/base_link_collision.stl" />
       </geometry>
     </collision>
@@ -77,17 +77,17 @@
       <geometry>
         <mesh
-          filename="package://xarm_gripper/meshes/left_outer_knuckle.STL" />
-      </geometry>
-      <material name="Silver">
-        <color rgba="0.753 0.753 0.753 1.0"/>
-      </material>
-    </visual>
-    <collision>
-      <origin
-        xyz="0 0 0"
-        rpy="0 0 0" />
-      <geometry>
-        <mesh
-          filename="package://xarm_gripper/meshes/left_outer_knuckle.STL" />
+          filename="package://xarm_gripper/meshes/left_outer_knuckle.stl" />
+      </geometry>
+      <material name="Silver">
+        <color rgba="0.753 0.753 0.753 1.0"/>
+      </material>
+    </visual>
+    <collision>
+      <origin
+        xyz="0 0 0"
+        rpy="0 0 0" />
+      <geometry>
+        <mesh
+          filename="package://xarm_gripper/meshes/left_outer_knuckle.stl" />
       </geometry>
     </collision>
@@ -133,17 +133,17 @@
       <geometry>
         <mesh
-          filename="package://xarm_gripper/meshes/left_finger.STL" />
-      </geometry>
-      <material name="Silver">
-        <color rgba="0.753 0.753 0.753 1.0"/>
-      </material>
-    </visual>
-    <collision>
-      <origin
-        xyz="0 0 0"
-        rpy="0 0 0" />
-      <geometry>
-        <mesh
-          filename="package://xarm_gripper/meshes/left_finger.STL" />
+          filename="package://xarm_gripper/meshes/left_finger.stl" />
+      </geometry>
+      <material name="Silver">
+        <color rgba="0.753 0.753 0.753 1.0"/>
+      </material>
+    </visual>
+    <collision>
+      <origin
+        xyz="0 0 0"
+        rpy="0 0 0" />
+      <geometry>
+        <mesh
+          filename="package://xarm_gripper/meshes/left_finger.stl" />
       </geometry>
     </collision>
@@ -190,17 +190,17 @@
       <geometry>
         <mesh
-          filename="package://xarm_gripper/meshes/left_inner_knuckle.STL" />
-      </geometry>
-      <material name="Silver">
-        <color rgba="0.753 0.753 0.753 1.0"/>
-      </material>
-    </visual>
-    <collision>
-      <origin
-        xyz="0 0 0"
-        rpy="0 0 0" />
-      <geometry>
-        <mesh
-          filename="package://xarm_gripper/meshes/left_inner_knuckle.STL" />
+          filename="package://xarm_gripper/meshes/left_inner_knuckle.stl" />
+      </geometry>
+      <material name="Silver">
+        <color rgba="0.753 0.753 0.753 1.0"/>
+      </material>
+    </visual>
+    <collision>
+      <origin
+        xyz="0 0 0"
+        rpy="0 0 0" />
+      <geometry>
+        <mesh
+          filename="package://xarm_gripper/meshes/left_inner_knuckle.stl" />
       </geometry>
     </collision>
@@ -247,17 +247,17 @@
       <geometry>
         <mesh
-          filename="package://xarm_gripper/meshes/right_outer_knuckle.STL" />
-      </geometry>
-      <material name="Silver">
-        <color rgba="0.753 0.753 0.753 1.0"/>
-      </material>
-    </visual>
-    <collision>
-      <origin
-        xyz="0 0 0"
-        rpy="0 0 0" />
-      <geometry>
-        <mesh
-          filename="package://xarm_gripper/meshes/right_outer_knuckle.STL" />
+          filename="package://xarm_gripper/meshes/right_outer_knuckle.stl" />
+      </geometry>
+      <material name="Silver">
+        <color rgba="0.753 0.753 0.753 1.0"/>
+      </material>
+    </visual>
+    <collision>
+      <origin
+        xyz="0 0 0"
+        rpy="0 0 0" />
+      <geometry>
+        <mesh
+          filename="package://xarm_gripper/meshes/right_outer_knuckle.stl" />
       </geometry>
     </collision>
@@ -304,17 +304,17 @@
       <geometry>
         <mesh
-          filename="package://xarm_gripper/meshes/right_finger.STL" />
-      </geometry>
-      <material name="Silver">
-        <color rgba="0.753 0.753 0.753 1.0"/>
-      </material>
-    </visual>
-    <collision>
-      <origin
-        xyz="0 0 0"
-        rpy="0 0 0" />
-      <geometry>
-        <mesh
-          filename="package://xarm_gripper/meshes/right_finger.STL" />
+          filename="package://xarm_gripper/meshes/right_finger.stl" />
+      </geometry>
+      <material name="Silver">
+        <color rgba="0.753 0.753 0.753 1.0"/>
+      </material>
+    </visual>
+    <collision>
+      <origin
+        xyz="0 0 0"
+        rpy="0 0 0" />
+      <geometry>
+        <mesh
+          filename="package://xarm_gripper/meshes/right_finger.stl" />
       </geometry>
     </collision>
@@ -361,17 +361,17 @@
       <geometry>
         <mesh
-          filename="package://xarm_gripper/meshes/right_inner_knuckle.STL" />
-      </geometry>
-      <material name="Silver">
-        <color rgba="0.753 0.753 0.753 1.0"/>
-      </material>
-    </visual>
-    <collision>
-      <origin
-        xyz="0 0 0"
-        rpy="0 0 0" />
-      <geometry>
-        <mesh
-          filename="package://xarm_gripper/meshes/right_inner_knuckle.STL" />
+          filename="package://xarm_gripper/meshes/right_inner_knuckle.stl" />
+      </geometry>
+      <material name="Silver">
+        <color rgba="0.753 0.753 0.753 1.0"/>
+      </material>
+    </visual>
+    <collision>
+      <origin
+        xyz="0 0 0"
+        rpy="0 0 0" />
+      <geometry>
+        <mesh
+          filename="package://xarm_gripper/meshes/right_inner_knuckle.stl" />
       </geometry>
     </collision>
