Commit message: [fix] (xacro) fix str to int exception

File: xarm_description/urdf/common/common.link.xacro (robot description, xacro)
@@ -72,9 +72,10 @@
         <xacro:property name="_model1300" value="true" />
       </xacro:if>
-      <xacro:if value="${robot_sn[8] == '0'}">
+      <xacro:property name="is_num" value="${robot_sn[8] == '0' or robot_sn[8] == '1' or robot_sn[8] == '2' or robot_sn[8] == '3' or robot_sn[8] == '4' or robot_sn[8] == '5' or robot_sn[8] == '6' or robot_sn[8] == '7' or robot_sn[8] == '8' or robot_sn[8] == '9'}" />
+      <xacro:if value="${is_num}">
+        <xacro:property name="date_str" value="${robot_sn[8:10]}${robot_sn[6:8]}" />
+      </xacro:if>
+      <xacro:unless value="${is_num}">
         <xacro:property name="date_str" value="2${robot_sn[9]}${robot_sn[6:8]}" />
-      </xacro:if>
-      <xacro:unless value="${robot_sn[8] == '0'}">
-        <xacro:property name="date_str" value="${robot_sn[8:10]}${robot_sn[6:8]}" />
       </xacro:unless>
       <xacro:property name="date_int" value="${int(date_str)}" />

Commit message: [feat] add kinematics_suffix parameter

File: xarm_description/urdf/common/common.link.xacro (robot description, xacro)
@@ -51,4 +51,7 @@
     </collision>
   </xacro:macro>
+  <xacro:macro name="common_joint_origin" params="joint_kinematic_params">
+    <origin xyz="${joint_kinematic_params['x']} ${joint_kinematic_params['y']} ${joint_kinematic_params['z']}" rpy="${joint_kinematic_params['roll']} ${joint_kinematic_params['pitch']} ${joint_kinematic_params['yaw']}" />
+  </xacro:macro>
   <xacro:macro name="parse_link_inertial_filename" params="dof robot_type robot_sn model1300">
     <!-- default inertial params filename -->

File: xarm_description/urdf/dual_xarm_device.urdf.xacro (robot description, xacro)
@@ -58,4 +58,6 @@
   <xacro:arg name="default_gripper_baud_2" default="2000000"/>
   <xacro:arg name="mesh_suffix" default="stl"/>
+  <xacro:arg name="kinematics_suffix_1" default=""/>
+  <xacro:arg name="kinematics_suffix_2" default=""/>
   <!-- load xarm device -->
   <xacro:include filename="$(find xarm_description)/urdf/xarm_device_macro.xacro" />
@@ -77,5 +79,5 @@
     robot_ip="$(arg robot_ip_1)" report_type="$(arg report_type_1)"
     baud_checkset="$(arg baud_checkset_1)" default_gripper_baud="$(arg default_gripper_baud_1)"
-    model1300="$(arg model1300_1)" robot_sn="$(arg robot_sn_1)" mesh_suffix="$(arg mesh_suffix)" />
+    model1300="$(arg model1300_1)" robot_sn="$(arg robot_sn_1)" mesh_suffix="$(arg mesh_suffix)" kinematics_suffix="$(arg kinematics_suffix_1)" />
   <xacro:xarm_device prefix="$(arg prefix_2)" hw_ns="$(arg hw_ns)" limited="$(arg limited)"
     effort_control="$(arg effort_control)" velocity_control="$(arg velocity_control)"
@@ -95,4 +97,4 @@
     robot_ip="$(arg robot_ip_2)" report_type="$(arg report_type_2)"
     baud_checkset="$(arg baud_checkset_2)" default_gripper_baud="$(arg default_gripper_baud_2)"
-    model1300="$(arg model1300_2)" robot_sn="$(arg robot_sn_2)" mesh_suffix="$(arg mesh_suffix)" />
+    model1300="$(arg model1300_2)" robot_sn="$(arg robot_sn_2)" mesh_suffix="$(arg mesh_suffix)" kinematics_suffix="$(arg kinematics_suffix_2)" />
 </robot>

File: xarm_description/urdf/lite6/lite6.urdf.xacro (robot description, xacro)
@@ -8,5 +8,5 @@
     joint5_lower_limit:=${-2.1642}  joint5_upper_limit:=${2.1642}
     joint6_lower_limit:=${-2.0*pi}  joint6_upper_limit:=${2.0*pi}
-    inertial_params_filename:='' "
+    inertial_params_filename:='' kinematics_params_filename:='' "
     >
     <!-- load params and define property -->
@@ -20,8 +20,11 @@
     <xacro:if value="${use_xacro_load_yaml}">
       <xacro:property name="inertial_params" value="${xacro.load_yaml(link_inertial_params_file)}"/>
+      <xacro:property name="kinematics_config" value="${xacro.load_yaml(kinematics_params_filename)}"/>
     </xacro:if>
     <xacro:unless value="${use_xacro_load_yaml}">
       <xacro:property name="inertial_params" value="${load_yaml(link_inertial_params_file)}"/>
+      <xacro:property name="kinematics_config" value="${load_yaml(kinematics_params_filename)}"/>
     </xacro:unless>
+    <xacro:property name="kinematics_params" value="${kinematics_config['kinematics']}"/>
     <link name="${prefix}link_base">
       <inertial>
@@ -57,5 +60,6 @@
     </link>
     <joint name="${prefix}joint1" type="revolute">
-      <origin xyz="0 0 0.2435" rpy="0 0 0" />
+      <!-- <origin xyz="0 0 0.2435" rpy="0 0 0" /> -->
+      <xacro:common_joint_origin joint_kinematic_params="${kinematics_params['joint1']}" />
       <parent link="${prefix}link_base" />
       <child link="${prefix}link1" />
@@ -74,14 +78,15 @@
       <xacro:common_link_visual
         mesh_filename="lite6/visual/link2"
-        origin_xyz="0 0 0"
+        origin_xyz="0 0 ${-kinematics_params['joint2']['y']}"
         origin_rpy="0 0 0"
         material_name="${prefix}White" />
       <xacro:common_link_collision
         mesh_filename="lite6/collision/link2"
-        origin_xyz="0 0 0"
+        origin_xyz="0 0 ${-kinematics_params['joint2']['y']}"
         origin_rpy="0 0 0" />
     </link>
     <joint name="${prefix}joint2" type="revolute">
-      <origin xyz="0 0 0" rpy="1.5708 -1.5708 3.1416" />
+      <!-- <origin xyz="0 0 0" rpy="1.5708 -1.5708 3.1416" /> -->
+      <xacro:common_joint_origin joint_kinematic_params="${kinematics_params['joint2']}" />
       <parent link="${prefix}link1" />
       <child link="${prefix}link2" />
@@ -109,5 +114,6 @@
     </link>
     <joint name="${prefix}joint3" type="revolute">
-      <origin xyz="0.2002 0 0" rpy="-3.1416 0 1.5708" />
+      <!-- <origin xyz="0.2002 0 0" rpy="-3.1416 0 1.5708" /> -->
+      <xacro:common_joint_origin joint_kinematic_params="${kinematics_params['joint3']}" />
       <parent link="${prefix}link2" />
       <child link="${prefix}link3" />
@@ -135,5 +141,6 @@
     </link>
     <joint name="${prefix}joint4" type="revolute">
-      <origin xyz="0.087 -0.22761 0" rpy="1.5708 0 0" />
+      <!-- <origin xyz="0.087 -0.22761 0" rpy="1.5708 0 0" /> -->
+      <xacro:common_joint_origin joint_kinematic_params="${kinematics_params['joint4']}" />
       <parent link="${prefix}link3" />
       <child link="${prefix}link4" />
@@ -161,5 +168,6 @@
     </link>
     <joint name="${prefix}joint5" type="revolute">
-      <origin xyz="0 0 0" rpy="1.5708 0 0" />
+      <!-- <origin xyz="0 0 0" rpy="1.5708 0 0" /> -->
+      <xacro:common_joint_origin joint_kinematic_params="${kinematics_params['joint5']}" />
       <parent link="${prefix}link4" />
       <child link="${prefix}link5" />
@@ -187,5 +195,6 @@
     </link>
     <joint name="${prefix}joint6" type="revolute">
-      <origin xyz="0 0.0625 0" rpy="-1.5708 0 0" />
+      <!-- <origin xyz="0 0.0625 0" rpy="-1.5708 0 0" /> -->
+      <xacro:common_joint_origin joint_kinematic_params="${kinematics_params['joint6']}" />
       <parent link="${prefix}link5" />
       <child link="${prefix}link6" />

File: xarm_description/urdf/lite6/lite6_robot_macro.xacro (robot description, xacro)
@@ -13,4 +13,5 @@
     default_gripper_baud:=2000000
     inertial_params_filename:=''
+    kinematics_params_filename:=''
     hard_interface:='PositionJointInterface' "
     >
@@ -44,5 +45,7 @@
         joint5_lower_limit="${-2.1642}" joint5_upper_limit="${2.1642}"
         joint6_lower_limit="${-pi*0.99}" joint6_upper_limit="${pi*0.99}"
-        inertial_params_filename="${inertial_params_filename}" />
+        inertial_params_filename="${inertial_params_filename}"
+        kinematics_params_filename="${kinematics_params_filename}"
+        />
     </xacro:if>
     <xacro:unless value="${limited}">
@@ -54,5 +57,8 @@
           baud_checkset="${baud_checkset}" default_gripper_baud="${default_gripper_baud}" />
       </xacro:if>
-      <xacro:lite6_urdf prefix="${prefix}" inertial_params_filename="${inertial_params_filename}"/>
+      <xacro:lite6_urdf prefix="${prefix}"
+        inertial_params_filename="${inertial_params_filename}"
+        kinematics_params_filename="${kinematics_params_filename}"
+        />
     </xacro:unless>
     <xacro:lite6_transmission prefix="${prefix}" hard_interface="${hard_interface}" />

File: xarm_description/urdf/uf850/uf850.urdf.xacro (robot description, xacro)
@@ -9,5 +9,5 @@
     joint6_lower_limit:=${-2.0*pi}  joint6_upper_limit:=${2.0*pi}
     model1300:=false
-    inertial_params_filename:='' "
+    inertial_params_filename:='' kinematics_params_filename:='' "
     >
     <!-- load params and define property -->
@@ -21,8 +21,11 @@
     <xacro:if value="${use_xacro_load_yaml}">
       <xacro:property name="inertial_params" value="${xacro.load_yaml(link_inertial_params_file)}"/>
+      <xacro:property name="kinematics_config" value="${xacro.load_yaml(kinematics_params_filename)}"/>
     </xacro:if>
     <xacro:unless value="${use_xacro_load_yaml}">
       <xacro:property name="inertial_params" value="${load_yaml(link_inertial_params_file)}"/>
+      <xacro:property name="kinematics_config" value="${load_yaml(kinematics_params_filename)}"/>
     </xacro:unless>
+    <xacro:property name="kinematics_params" value="${kinematics_config['kinematics']}"/>
     <link name="${prefix}link_base">
       <inertial>
@@ -60,5 +63,6 @@
       <parent link="${prefix}link_base"/>
       <child link="${prefix}link1"/>
-      <origin xyz="0 0 0.364" rpy="0 0 0"/>
+      <!-- <origin xyz="0 0 0.364" rpy="0 0 0"/> -->
+      <xacro:common_joint_origin joint_kinematic_params="${kinematics_params['joint1']}" />
       <axis xyz="0 0 1"/>
       <limit
@@ -75,10 +79,10 @@
       <xacro:common_link_visual
         mesh_filename="uf850/visual/link2"
-        origin_xyz="0 0 0"
+        origin_xyz="0 0 ${kinematics_params['joint2']['y']}"
         origin_rpy="0 0 0"
         material_name="${prefix}White" />
       <xacro:common_link_collision
         mesh_filename="uf850/collision/link2"
-        origin_xyz="0 0 0"
+        origin_xyz="0 0 ${kinematics_params['joint2']['y']}"
         origin_rpy="0 0 0" />
     </link>
@@ -86,5 +90,6 @@
       <parent link="${prefix}link1"/>
       <child link="${prefix}link2"/>
-      <origin xyz="0 0 0" rpy="1.5708 -1.5708 0" />
+      <!-- <origin xyz="0 0 0" rpy="1.5708 -1.5708 0" /> -->
+      <xacro:common_joint_origin joint_kinematic_params="${kinematics_params['joint2']}" />
       <axis xyz="0 0 1"/>
       <limit
@@ -112,5 +117,6 @@
       <parent link="${prefix}link2"/>
       <child link="${prefix}link3"/>
-      <origin xyz="0.39 0 0" rpy="-3.1416 0 -1.5708"/>
+      <!-- <origin xyz="0.39 0 0" rpy="-3.1416 0 -1.5708"/> -->
+      <xacro:common_joint_origin joint_kinematic_params="${kinematics_params['joint3']}" />
       <axis xyz="0 0 1"/>
       <limit
@@ -138,5 +144,6 @@
       <parent link="${prefix}link3"/>
       <child link="${prefix}link4"/>
-      <origin xyz="0.15 0.426 0" rpy="-1.5708 0 0"/>
+      <!-- <origin xyz="0.15 0.426 0" rpy="-1.5708 0 0"/> -->
+      <xacro:common_joint_origin joint_kinematic_params="${kinematics_params['joint4']}" />
       <axis xyz="0 0 1"/>
       <limit
@@ -164,5 +171,6 @@
       <parent link="${prefix}link4"/>
       <child link="${prefix}link5"/>
-      <origin xyz="0 0 0" rpy="-1.5708 0 0"/>
+      <!-- <origin xyz="0 0 0" rpy="-1.5708 0 0"/> -->
+      <xacro:common_joint_origin joint_kinematic_params="${kinematics_params['joint5']}" />
       <axis xyz="0 0 1"/>
       <limit
@@ -190,5 +198,6 @@
       <parent link="${prefix}link5"/>
       <child link="${prefix}link6"/>
-      <origin xyz="0 -0.09 0" rpy="1.5708 0 0"/>
+      <!-- <origin xyz="0 -0.09 0" rpy="1.5708 0 0"/> -->
+      <xacro:common_joint_origin joint_kinematic_params="${kinematics_params['joint6']}" />
       <axis xyz="0 0 1"/>
       <limit

File: xarm_description/urdf/uf850/uf850_robot_macro.xacro (robot description, xacro)
@@ -14,4 +14,5 @@
     model1300:=false
     inertial_params_filename:=''
+    kinematics_params_filename:=''
     hard_interface:='PositionJointInterface' "
     >
@@ -46,5 +47,6 @@
         joint6_lower_limit="${-pi*0.99}" joint6_upper_limit="${pi*0.99}"
         model1300="${model1300}"
-        inertial_params_filename="${inertial_params_filename}"/>
+        inertial_params_filename="${inertial_params_filename}"
+        kinematics_params_filename="${kinematics_params_filename}"/>
     </xacro:if>
     <xacro:unless value="${limited}">
@@ -57,5 +59,6 @@
       </xacro:if>
       <xacro:uf850_urdf prefix="${prefix}" model1300="${model1300}"
-        inertial_params_filename="${inertial_params_filename}"/>
+        inertial_params_filename="${inertial_params_filename}"
+        kinematics_params_filename="${kinematics_params_filename}"/>
     </xacro:unless>
     <xacro:uf850_transmission prefix="${prefix}" hard_interface="${hard_interface}" />

File: xarm_description/urdf/xarm5/xarm5.urdf.xacro (robot description, xacro)
@@ -8,5 +8,5 @@
     joint5_lower_limit:=${-2.0*pi}  joint5_upper_limit:=${2.0*pi}
     model1300:=false
-    inertial_params_filename:='' "
+    inertial_params_filename:='' kinematics_params_filename:='' "
     >
     <!-- define property -->
@@ -29,8 +29,11 @@
     <xacro:if value="${use_xacro_load_yaml}">
       <xacro:property name="inertial_params" value="${xacro.load_yaml(link_inertial_params_file)}"/>
+      <xacro:property name="kinematics_config" value="${xacro.load_yaml(kinematics_params_filename)}"/>
     </xacro:if>
     <xacro:unless value="${use_xacro_load_yaml}">
       <xacro:property name="inertial_params" value="${load_yaml(link_inertial_params_file)}"/>
+      <xacro:property name="kinematics_config" value="${load_yaml(kinematics_params_filename)}"/>
     </xacro:unless>
+    <xacro:property name="kinematics_params" value="${kinematics_config['kinematics']}"/>
     <link name="${prefix}link_base">
       <inertial>
@@ -66,5 +69,6 @@
     </link>
     <joint name="${prefix}joint1" type="revolute">
-      <origin xyz="0 0 0.267" rpy="0 0 0" />
+      <!-- <origin xyz="0 0 0.267" rpy="0 0 0" /> -->
+      <xacro:common_joint_origin joint_kinematic_params="${kinematics_params['joint1']}" />
       <parent link="${prefix}link_base" />
       <child link="${prefix}link1" />
@@ -92,5 +96,6 @@
     </link>
     <joint name="${prefix}joint2" type="revolute">
-      <origin xyz="0 0 0" rpy="-1.5708 0 0" />
+      <!-- <origin xyz="0 0 0" rpy="-1.5708 0 0" /> -->
+      <xacro:common_joint_origin joint_kinematic_params="${kinematics_params['joint2']}" />
       <parent link="${prefix}link1" />
       <child link="${prefix}link2" />
@@ -118,5 +123,6 @@
     </link>
     <joint name="${prefix}joint3" type="revolute">
-      <origin xyz="0.0535 -0.2845 0" rpy="0 0 0" />
+      <!-- <origin xyz="0.0535 -0.2845 0" rpy="0 0 0" /> -->
+      <xacro:common_joint_origin joint_kinematic_params="${kinematics_params['joint3']}" />
       <parent link="${prefix}link2" />
       <child link="${prefix}link3" />
@@ -144,5 +150,6 @@
     </link>
     <joint name="${prefix}joint4" type="revolute">
-      <origin xyz="0.0775 0.3425 0" rpy="0 0 0" />
+      <!-- <origin xyz="0.0775 0.3425 0" rpy="0 0 0" /> -->
+      <xacro:common_joint_origin joint_kinematic_params="${kinematics_params['joint4']}" />
       <parent link="${prefix}link3" />
       <child link="${prefix}link4" />
@@ -170,5 +177,6 @@
     </link>
     <joint name="${prefix}joint5" type="revolute">
-      <origin xyz="0.076 0.097 0" rpy="-1.5708 0 0" />
+      <!-- <origin xyz="0.076 0.097 0" rpy="-1.5708 0 0" /> -->
+      <xacro:common_joint_origin joint_kinematic_params="${kinematics_params['joint5']}" />
       <parent link="${prefix}link4" />
       <child link="${prefix}link5" />

File: xarm_description/urdf/xarm5/xarm5_robot_macro.xacro (robot description, xacro)
@@ -14,4 +14,5 @@
     model1300:=false
     inertial_params_filename:=''
+    kinematics_params_filename:=''
     hard_interface:='PositionJointInterface' "
     >
@@ -44,5 +45,7 @@
         joint5_lower_limit="${-pi*0.99}" joint5_upper_limit="${pi*0.99}"
         model1300="${model1300}"
-        inertial_params_filename="${inertial_params_filename}"/>
+        inertial_params_filename="${inertial_params_filename}"
+        kinematics_params_filename="${kinematics_params_filename}"
+        />
     </xacro:if>
     <xacro:unless value="${limited}">
@@ -55,5 +58,7 @@
       </xacro:if>
       <xacro:xarm5_urdf prefix="${prefix}" model1300="${model1300}"
-        inertial_params_filename="${inertial_params_filename}"/>
+        inertial_params_filename="${inertial_params_filename}"
+        kinematics_params_filename="${kinematics_params_filename}"
+        />
     </xacro:unless>
     <xacro:xarm5_transmission prefix="${prefix}" hard_interface="${hard_interface}" />

File: xarm_description/urdf/xarm6/xarm6.urdf.xacro (robot description, xacro)
@@ -9,5 +9,5 @@
     joint6_lower_limit:=${-2.0*pi}  joint6_upper_limit:=${2.0*pi}
     model1300:=false
-    inertial_params_filename:='' "
+    inertial_params_filename:='' kinematics_params_filename:='' "
     >
     <!-- define property -->
@@ -30,8 +30,11 @@
     <xacro:if value="${use_xacro_load_yaml}">
       <xacro:property name="inertial_params" value="${xacro.load_yaml(link_inertial_params_file)}"/>
+      <xacro:property name="kinematics_config" value="${xacro.load_yaml(kinematics_params_filename)}"/>
     </xacro:if>
     <xacro:unless value="${use_xacro_load_yaml}">
       <xacro:property name="inertial_params" value="${load_yaml(link_inertial_params_file)}"/>
+      <xacro:property name="kinematics_config" value="${load_yaml(kinematics_params_filename)}"/>
     </xacro:unless>
+    <xacro:property name="kinematics_params" value="${kinematics_config['kinematics']}"/>
     <link name="${prefix}link_base">
       <inertial>
@@ -69,5 +72,6 @@
       <parent link="${prefix}link_base"/>
       <child link="${prefix}link1"/>
-      <origin xyz="0 0 0.267" rpy="0 0 0"/>
+      <!-- <origin xyz="0 0 0.267" rpy="0 0 0"/> -->
+      <xacro:common_joint_origin joint_kinematic_params="${kinematics_params['joint1']}" />
       <axis xyz="0 0 1"/>
       <limit
@@ -84,10 +88,10 @@
       <xacro:common_link_visual
         mesh_filename="xarm6/visual/link2"
-        origin_xyz="0 0 0"
+        origin_xyz="0 0 ${-kinematics_params['joint2']['y']}"
         origin_rpy="0 0 0"
         material_name="${prefix}White" />
       <xacro:common_link_collision
         mesh_filename="xarm6/visual/link2"
-        origin_xyz="0 0 0"
+        origin_xyz="0 0 ${-kinematics_params['joint2']['y']}"
         origin_rpy="0 0 0" />
     </link>
@@ -95,5 +99,6 @@
       <parent link="${prefix}link1"/>
       <child link="${prefix}link2"/>
-      <origin xyz="0 0 0" rpy="-1.5708 0 0" />
+      <!-- <origin xyz="0 0 0" rpy="-1.5708 0 0" /> -->
+      <xacro:common_joint_origin joint_kinematic_params="${kinematics_params['joint2']}" />
       <axis xyz="0 0 1"/>
       <limit
@@ -121,5 +126,6 @@
       <parent link="${prefix}link2"/>
       <child link="${prefix}link3"/>
-      <origin xyz="0.0535 -0.2845 0" rpy="0 0 0"/>
+      <!-- <origin xyz="0.0535 -0.2845 0" rpy="0 0 0"/> -->
+      <xacro:common_joint_origin joint_kinematic_params="${kinematics_params['joint3']}" />
       <axis xyz="0 0 1"/>
       <limit
@@ -147,5 +153,6 @@
       <parent link="${prefix}link3"/>
       <child link="${prefix}link4"/>
-      <origin xyz="0.0775 0.3425 0" rpy="-1.5708 0 0"/>
+      <!-- <origin xyz="0.0775 0.3425 0" rpy="-1.5708 0 0"/> -->
+      <xacro:common_joint_origin joint_kinematic_params="${kinematics_params['joint4']}" />
       <axis xyz="0 0 1"/>
       <limit
@@ -174,4 +181,5 @@
       <child link="${prefix}link5"/>
       <origin xyz="0 0 0" rpy="1.5708 0 0"/>
+      <xacro:common_joint_origin joint_kinematic_params="${kinematics_params['joint5']}" />
       <axis xyz="0 0 1"/>
       <limit
@@ -199,5 +207,6 @@
       <parent link="${prefix}link5"/>
       <child link="${prefix}link6"/>
-      <origin xyz="0.076 0.097 0" rpy="-1.5708 0 0"/>
+      <!-- <origin xyz="0.076 0.097 0" rpy="-1.5708 0 0"/> -->
+      <xacro:common_joint_origin joint_kinematic_params="${kinematics_params['joint6']}" />
       <axis xyz="0 0 1"/>
       <limit

File: xarm_description/urdf/xarm6/xarm6_robot_macro.xacro (robot description, xacro)
@@ -14,4 +14,5 @@
     model1300:=false
     inertial_params_filename:=''
+    kinematics_params_filename:=''
     hard_interface:='PositionJointInterface' "
     >
@@ -46,5 +47,7 @@
         joint6_lower_limit="${-pi*0.99}" joint6_upper_limit="${pi*0.99}"
         model1300="${model1300}"
-        inertial_params_filename="${inertial_params_filename}"/>
+        inertial_params_filename="${inertial_params_filename}"
+        kinematics_params_filename="${kinematics_params_filename}"
+        />
     </xacro:if>
     <xacro:unless value="${limited}">
@@ -57,5 +60,7 @@
       </xacro:if>
       <xacro:xarm6_urdf prefix="${prefix}" model1300="${model1300}"
-        inertial_params_filename="${inertial_params_filename}"/>
+        inertial_params_filename="${inertial_params_filename}"
+        kinematics_params_filename="${kinematics_params_filename}"
+        />
     </xacro:unless>
     <xacro:xarm6_transmission prefix="${prefix}" hard_interface="${hard_interface}" />
