Commit message: [feat] add kinematics_suffix parameter

File: xarm_description/urdf/xarm7/xarm7.urdf.xacro (robot description, xacro)
@@ -10,5 +10,5 @@
     joint7_lower_limit:=${-2.0*pi}  joint7_upper_limit:=${2.0*pi}
     model1300:=false
-    inertial_params_filename:='' "
+    inertial_params_filename:='' kinematics_params_filename:='' "
     >
     <!-- define property -->
@@ -31,8 +31,11 @@
     <xacro:if value="${use_xacro_load_yaml}">
       <xacro:property name="inertial_params" value="${xacro.load_yaml(link_inertial_params_file)}"/>
+      <xacro:property name="kinematics_config" value="${xacro.load_yaml(kinematics_params_filename)}"/>
     </xacro:if>
     <xacro:unless value="${use_xacro_load_yaml}">
       <xacro:property name="inertial_params" value="${load_yaml(link_inertial_params_file)}"/>
+      <xacro:property name="kinematics_config" value="${load_yaml(kinematics_params_filename)}"/>
     </xacro:unless>
+    <xacro:property name="kinematics_params" value="${kinematics_config['kinematics']}"/>
     <link name="${prefix}link_base">
       <inertial>
@@ -68,5 +71,6 @@
     </link>
     <joint name="${prefix}joint1" type="revolute">
-      <origin xyz="0 0 0.267" rpy="0 0 0" />
+      <!-- <origin xyz="0 0 0.267" rpy="0 0 0" /> -->
+      <xacro:common_joint_origin joint_kinematic_params="${kinematics_params['joint1']}" />
       <parent link="${prefix}link_base" />
       <child link="${prefix}link1" />
@@ -94,5 +98,6 @@
     </link>
     <joint name="${prefix}joint2" type="revolute">
-      <origin xyz="0 0 0" rpy="-1.5708 0 0" />
+      <!-- <origin xyz="0 0 0" rpy="-1.5708 0 0" /> -->
+      <xacro:common_joint_origin joint_kinematic_params="${kinematics_params['joint2']}" />
       <parent link="${prefix}link1" />
       <child link="${prefix}link2" />
@@ -120,5 +125,6 @@
     </link>
     <joint name="${prefix}joint3" type="revolute">
-      <origin xyz="0 -0.293 0" rpy="1.5708 0 0" />
+      <!-- <origin xyz="0 -0.293 0" rpy="1.5708 0 0" /> -->
+      <xacro:common_joint_origin joint_kinematic_params="${kinematics_params['joint3']}" />
       <parent link="${prefix}link2" />
       <child link="${prefix}link3" />
@@ -146,5 +152,6 @@
     </link>
     <joint name="${prefix}joint4" type="revolute">
-      <origin xyz="0.0525 0 0" rpy="1.5708 0 0" />
+      <!-- <origin xyz="0.0525 0 0" rpy="1.5708 0 0" /> -->
+      <xacro:common_joint_origin joint_kinematic_params="${kinematics_params['joint4']}" />
       <parent link="${prefix}link3" />
       <child link="${prefix}link4" />
@@ -172,5 +179,6 @@
     </link>
     <joint name="${prefix}joint5" type="revolute">
-      <origin xyz="0.0775 -0.3425 0" rpy="1.5708 0 0" />
+      <!-- <origin xyz="0.0775 -0.3425 0" rpy="1.5708 0 0" /> -->
+      <xacro:common_joint_origin joint_kinematic_params="${kinematics_params['joint5']}" />
       <parent link="${prefix}link4" />
       <child link="${prefix}link5" />
@@ -198,5 +206,6 @@
     </link>
     <joint name="${prefix}joint6" type="revolute">
-      <origin xyz="0 0 0" rpy="1.5708 0 0" />
+      <!-- <origin xyz="0 0 0" rpy="1.5708 0 0" /> -->
+      <xacro:common_joint_origin joint_kinematic_params="${kinematics_params['joint6']}" />
       <parent link="${prefix}link5" />
       <child link="${prefix}link6" />
@@ -224,5 +233,6 @@
     </link>
     <joint name="${prefix}joint7" type="revolute">
-      <origin xyz="0.076 0.097 0" rpy="-1.5708 0 0" />
+      <!-- <origin xyz="0.076 0.097 0" rpy="-1.5708 0 0" /> -->
+      <xacro:common_joint_origin joint_kinematic_params="${kinematics_params['joint7']}" />
       <parent link="${prefix}link6" />
       <child link="${prefix}link7" />

File: xarm_description/urdf/xarm7/xarm7_robot_macro.xacro (robot description, xacro)
@@ -14,4 +14,5 @@
     model1300:=false
     inertial_params_filename:=''
+    kinematics_params_filename:=''
     hard_interface:='PositionJointInterface' "
     >
@@ -48,5 +49,7 @@
         joint7_lower_limit="${-pi*0.99}" joint7_upper_limit="${pi*0.99}"
         model1300="${model1300}"
-        inertial_params_filename="${inertial_params_filename}"/>
+        inertial_params_filename="${inertial_params_filename}"
+        kinematics_params_filename="${kinematics_params_filename}"
+        />
     </xacro:if>
     <xacro:unless value="${limited}">
@@ -59,5 +62,7 @@
       </xacro:if>
       <xacro:xarm7_urdf prefix="${prefix}" model1300="${model1300}"
-        inertial_params_filename="${inertial_params_filename}"/>
+        inertial_params_filename="${inertial_params_filename}"
+        kinematics_params_filename="${kinematics_params_filename}"
+        />
     </xacro:unless>
     <xacro:xarm7_transmission prefix="${prefix}" hard_interface="${hard_interface}" />

File: xarm_description/urdf/xarm_device.urdf.xacro (robot description, xacro)
@@ -37,4 +37,5 @@
   <xacro:arg name="attach_rpy" default="0 0 0"/>
   <xacro:arg name="mesh_suffix" default="stl"/>
+  <xacro:arg name="kinematics_suffix" default=""/>
   <!-- load xarm device -->
   <xacro:include filename="$(find xarm_description)/urdf/xarm_device_macro.xacro" />
@@ -56,4 +57,4 @@
     baud_checkset="$(arg baud_checkset)" default_gripper_baud="$(arg default_gripper_baud)"
     model1300="$(arg model1300)" attach_to="$(arg attach_to)" attach_xyz="$(arg attach_xyz)" attach_rpy="$(arg attach_rpy)"
-    robot_sn="$(arg robot_sn)" use_gazebo_camera="$(arg use_gazebo_camera)" mesh_suffix="$(arg mesh_suffix)" />
+    robot_sn="$(arg robot_sn)" use_gazebo_camera="$(arg use_gazebo_camera)" mesh_suffix="$(arg mesh_suffix)" kinematics_suffix="$(arg kinematics_suffix)" />
 </robot>

File: xarm_description/urdf/xarm_device_macro.xacro (robot description, xacro)
@@ -39,5 +39,7 @@
     model1300:=false
     robot_sn:=''
-    mesh_suffix:='stl' "
+    mesh_suffix:='stl'
+    kinematics_suffix:=''
+    "
     >
     <!-- Load Common Material -->
@@ -67,5 +69,5 @@
     <joint name="${prefix}world_joint" type="fixed">
       <parent link="${attach_to}" />
-      <child link = "${prefix}link_base" />
+      <child link="${prefix}link_base" />
       <origin xyz="${attach_xyz}" rpy="${attach_rpy}" />
     </joint>
@@ -80,4 +82,16 @@
         <xacro:property name="hard_interface" value="PositionJointInterface" />
       </xacro:unless>
+    </xacro:unless>
+    <xacro:if value="${robot_type == 'uf850'}">
+      <xacro:property name="robot_name" value="${robot_type}" />
+    </xacro:if>
+    <xacro:unless value="${robot_type == 'uf850'}">
+      <xacro:property name="robot_name" value="${robot_type}${dof}" />
+    </xacro:unless>
+    <xacro:if value="${kinematics_suffix != ''}">
+      <xacro:property name="kinematics_params_filename" value="$(find xarm_description)/config/kinematics/user/${robot_name}_kinematics_${kinematics_suffix}.yaml"/>
+    </xacro:if>
+    <xacro:unless value="${kinematics_suffix != ''}">
+      <xacro:property name="kinematics_params_filename" value="$(find xarm_description)/config/kinematics/default/${robot_name}_default_kinematics.yaml"/>
     </xacro:unless>
     <xacro:if value="${dof == 5}">
@@ -94,4 +108,5 @@
         model1300="${new_model1300}"
         inertial_params_filename="${inertial_params_filename}"
+        kinematics_params_filename="${kinematics_params_filename}"
         hard_interface="${hard_interface}" />
     </xacro:if>
@@ -110,4 +125,5 @@
           model1300="${new_model1300}"
           inertial_params_filename="${inertial_params_filename}"
+          kinematics_params_filename="${kinematics_params_filename}"
           hard_interface="${hard_interface}" />
       </xacro:if>
@@ -124,4 +140,5 @@
           default_gripper_baud="${default_gripper_baud}"
           inertial_params_filename="${inertial_params_filename}"
+          kinematics_params_filename="${kinematics_params_filename}"
           hard_interface="${hard_interface}" />
       </xacro:if>
@@ -139,4 +156,5 @@
           model1300="${new_model1300}"
           inertial_params_filename="${inertial_params_filename}"
+          kinematics_params_filename="${kinematics_params_filename}"
           hard_interface="${hard_interface}" />
       </xacro:unless>
@@ -155,4 +173,5 @@
         model1300="${new_model1300}"
         inertial_params_filename="${inertial_params_filename}"
+        kinematics_params_filename="${kinematics_params_filename}"
         hard_interface="${hard_interface}" />
     </xacro:unless>
